Commit message: Define default values for some parameters
Added default values for effort_limit, velocity_limit, mu, mu2, slip1,
slip2, ,max_contacts

Regarding the default value for the paramters 'velocity_limit' and 'effor_limit'.

    effort_limit = 100000 Newton-meters, is a huge value.
    This represents the maximum torque the joint can apply. To put this into perspective, a high-performance
    passenger car engine produces between 200-500 N·m of torque. A value of 100000 N·m is more in the realm of
    industrial cranes or ship engines. It is an astronomically high value for a robot wheel.

    velocity_limit = 100 rad/s translates to approximately 955 rpm, which is extremely fast.

    By setting such a high values, we are declaring the actuator is ideal and can achieve very high torque and
    speeds without physical constraints. This is useful in simulation environments where we want to test the
    control algorithms (like velocity control, path planning, or trajectory following) without being constrained by
    the physical limitations of real-world motors.
    In essence, we are testing the software logic in isolation.

Default values for max_contacts, mu, mu2, slip1, and slip2 obtained from:
    http://sdformat.org/spec?ver=1.10&elem=collision
    SDFormat 1.10 is valid for library sdformat14.

File: urdf/wheels/set_wheel_props_macro.xacro (robot description, xacro)
@@ -2,5 +2,7 @@
 <robot name="set_wheel_props" xmlns:xacro="http://ros.org/wiki/xacro" xmlns:gz="http://gazebosim.org/schema">
   <xacro:macro name="set_wheel_props" params="desc_cfg prop_prefix">
-    <xacro:property name="${prop_prefix}_mass"        value="${desc_cfg['mass']}"  scope="parent"/>
+    <xacro:property name="${prop_prefix}_mass"
+                    value="${desc_cfg.get('mass', 0.1)}"
+                    scope="parent"/>
     <!--
     A wheel is either a cylinder (c) with its rotation axis along the y-axis or a sphere (s), no more geometries are
@@ -40,11 +42,45 @@
     -->
     <xacro:property name="${prop_prefix}_radius"         value="${0.5 * _wheel_size_x}"        scope="parent"/>
-    <xacro:property name="${prop_prefix}_velocity_limit" value="${desc_cfg['velocity_limit']}" scope="parent"/>
-    <xacro:property name="${prop_prefix}_effort_limit"   value="${desc_cfg['effort_limit']}"   scope="parent"/>
-    <xacro:property name="${prop_prefix}_max_contacts"   value="${desc_cfg.get('max_contacts', 10)}" scope="parent"/>
-    <xacro:property name="${prop_prefix}_mu"             value="${desc_cfg['mu']}"             scope="parent"/>
-    <xacro:property name="${prop_prefix}_mu2"            value="${desc_cfg['mu2']}"            scope="parent"/>
-    <xacro:property name="${prop_prefix}_slip1"          value="${desc_cfg['slip1']}"          scope="parent"/>
-    <xacro:property name="${prop_prefix}_slip2"          value="${desc_cfg['slip2']}"          scope="parent"/>
+    <!--
+    Regarding the default value for the paramters 'velocity_limit' and 'effor_limit'.
+    effort_limit = 100000 Newton-meters, is a huge value.
+    This represents the maximum torque the joint can apply. To put this into perspective, a high-performance
+    passenger car engine produces between 200-500 N·m of torque. A value of 100000 N·m is more in the realm of
+    industrial cranes or ship engines. It is an astronomically high value for a robot wheel.
+    velocity_limit = 100 rad/s translates to approximately 955 rpm, which is extremely fast.
+    By setting such a high values, we are declaring the actuator is ideal and can achieve very high torque and
+    speeds without physical constraints. This is useful in simulation environments where we want to test the
+    control algorithms (like velocity control, path planning, or trajectory following) without being constrained by
+    the physical limitations of real-world motors.
+    In essence, we are testing the software logic in isolation.
+    -->
+    <xacro:property name="${prop_prefix}_velocity_limit"
+                    value="${desc_cfg.get('velocity_limit', 100)}"
+                    scope="parent"/>
+    <xacro:property name="${prop_prefix}_effort_limit"
+                    value="${desc_cfg.get('effort_limit', 100000)}"
+                    scope="parent"/>
+    <!--
+    Default values for max_contacts, mu, mu2, slip1, and slip2 obtained from:
+    http://sdformat.org/spec?ver=1.10&elem=collision
+    SDFormat 1.10 is valid for library sdformat14.
+    -->
+    <xacro:property name="${prop_prefix}_max_contacts"
+                    value="${desc_cfg.get('max_contacts', 10)}"
+                    scope="parent"/>
+    <!--
+    -->
+    <xacro:property name="${prop_prefix}_mu"
+                    value="${desc_cfg.get('mu', 1)}"
+                    scope="parent"/>
+    <xacro:property name="${prop_prefix}_mu2"
+                    value="${desc_cfg.get('mu2', 1)}"
+                    scope="parent"/>
+    <xacro:property name="${prop_prefix}_slip1"
+                    value="${desc_cfg.get('slip1', 0)}"
+                    scope="parent"/>
+    <xacro:property name="${prop_prefix}_slip2"
+                    value="${desc_cfg.get('slip2', 0)}"
+                    scope="parent"/>
     <xacro:property name="${prop_prefix}_mesh_visual"
                     value="${mesh_dir + '/' + _wheel_mesh_visual if _wheel_mesh_visual else ''}"
@@ -53,9 +89,9 @@
                     value="${desc_cfg['mesh_visual_has_color']}"
                     scope="parent"/>
-    <xacro:property name="_wheel_color" value="${desc_cfg['color']}"/>
+    <xacro:property name="_wheel_color" value="${desc_cfg.get('color', dict(r = 0, g = 0, b = 0, a = 1))}"/>
     <xacro:property name="${prop_prefix}_color"
                     value="${_wheel_color['r']} ${_wheel_color['g']} ${_wheel_color['b']} ${_wheel_color['a']}"
                     scope="parent"/>
-    <xacro:property name="_wheel_scale" value="${desc_cfg['scale']}"/>
+    <xacro:property name="_wheel_scale" value="${desc_cfg.get('scale', dict(x = 1, y = 1, z = 1))}"/>
     <xacro:property name="${prop_prefix}_scale"
                     value="${_wheel_scale['x']} ${_wheel_scale['y']} ${_wheel_scale['z']}"

Commit message: Wheel can be configured as fixed or continuous

File: urdf/wheels/set_wheel_props_macro.xacro (robot description, xacro)
@@ -41,5 +41,10 @@
     size_x = 2*radius, radius = 0.5*size_x
     -->
-    <xacro:property name="${prop_prefix}_radius"         value="${0.5 * _wheel_size_x}"        scope="parent"/>
+    <xacro:property name="${prop_prefix}_radius"
+                    value="${0.5 * _wheel_size_x}"
+                    scope="parent"/>
+    <xacro:property name="${prop_prefix}_joint_type"
+                    value="${desc_cfg.get('joint_type', 'continuous')}"
+                    scope="parent"/>
     <!--
     Regarding the default value for the paramters 'velocity_limit' and 'effor_limit'.

File: urdf/wheels/wheel_macro.xacro (robot description, xacro)
@@ -9,4 +9,25 @@
 size_x = size_y = size_z = 2*radius
 shape='s 2*radius  2*radius  2*radius'  -> sphere.
+'joint_type' must be either 'continuous' or 'fixed'.
+'effort_limit' and 'velocity_limit' are considered only if 'joint_type' is 'continuous'.
+Explanation of the default values for the fields 'effort_limit' and 'velocity_limit'
+================================================================================================
+The 'effort' and 'velocity' limits for this joint are intentionally set to extremely high, non-physical values.
+This is a common and deliberate practice in simulation for the specific reason of modeling an 'ideal' actuator.
+By setting virtually infinite limits, we ensure that the simulator's physics engine will never be the limiting
+factor in the joint's performance. This allows developers to test high-level control algorithms (e.g., navigation,
+trajectory following) without being constrained by the physical limitations of real-world motors.
+In essence, we are testing the software logic in isolation.
+effort_limit = "100000" (Newton-meters).
+This represents the maximum torque the joint can apply. To put this into perspective, a high-performance
+passenger car engine produces between 200-500 N·m of torque. A value of 100000 N·m is more in the realm of
+industrial cranes or ship engines. It is an astronomically high value for a robot wheel.
+velocity_limit = "100" (radians/second).
+This translates to approximately 955 rpm. For context, a typical educational robot wheel (like a TurtleBot) spins
+at around 70-100 rpm. So, 955 rpm is extremely fast.
+If you need a realistic simulation of a physical robot, you should replace these values with the specifications
+from your wheel. For a typical medium-sized wheel, realistic values would be in the range of:
+Effort:   10 to 100 N·m
+Velocity: 10 to 30 rad/s
 -->
 <robot name="wheel" xmlns:xacro="http://ros.org/wiki/xacro" xmlns:gz="http://gazebosim.org/schema">
@@ -17,4 +38,5 @@
                        mass:=0.1
                        shape
+                       joint_type:=continuous
                        velocity_limit:=100
                        effort_limit:=100000
@@ -29,27 +51,7 @@
                        scale:='1 1 1'
                        joint_parent_fr_wheel_fr
-                       base_root_fr
-                       fdir1_base_root_fr">
+                       fdir1_fr
+                       fdir1">
     <!--
-    ================================================================================================
-    Explanation of the default values for the fields 'effort_limit' and 'velocity_limit'
-    ================================================================================================
-    The 'effort' and 'velocity' limits for this joint are intentionally set to extremely high, non-physical values.
-    This is a common and deliberate practice in simulation for the specific reason of modeling an 'ideal' actuator.
-    By setting virtually infinite limits, we ensure that the simulator's physics engine will never be the limiting
-    factor in the joint's performance. This allows developers to test high-level control algorithms (e.g., navigation,
-    trajectory following) without being constrained by the physical limitations of real-world motors.
-    In essence, we are testing the software logic in isolation.
-    effort_limit = "100000" (Newton-meters).
-    This represents the maximum torque the joint can apply. To put this into perspective, a high-performance
-    passenger car engine produces between 200-500 N·m of torque. A value of 100000 N·m is more in the realm of
-    industrial cranes or ship engines. It is an astronomically high value for a robot wheel.
-    velocity_limit = "100" (radians/second).
-    This translates to approximately 955 rpm. For context, a typical educational robot wheel (like a TurtleBot) spins
-    at around 70-100 rpm. So, 955 rpm is extremely fast.
-    If you need a realistic simulation of a physical robot, you should replace these values with the specifications
-    from your wheel. For a typical medium-sized wheel, realistic values would be in the range of:
-    Effort:   10 to 100 N·m
-    Velocity: 10 to 30 rad/s
     -->
     <xacro:include filename="$(find eut_robotics_description)/urdf/common/all_commons.xacro"/>
@@ -107,10 +109,15 @@
       vci_pose="0 0 0 0 0 0"/>
     <xacro:property name="j_wheel" value="${joint_parent_fr_wheel_fr.split()}"/>
-    <joint name="${prefix}${name}_joint" type="continuous">
+    <xacro:if value="${joint_type not in ('continuous', 'fixed')}">
+      ${xacro.fatal("The field 'joint_type' must be either 'continuous' or 'fixed'")}
+    </xacro:if>
+    <joint name="${prefix}${name}_joint" type="${joint_type}">
       <parent link="${parent_frame}"/>
       <child link="${prefix}${name}_link"/>
       <origin rpy="${j_wheel[3]} ${j_wheel[4]} ${j_wheel[5]}" xyz="${j_wheel[0]} ${j_wheel[1]} ${j_wheel[2]}"/>
-      <axis xyz="0 1 0"/>
-      <limit effort="${effort_limit}" velocity="${velocity_limit}"/>
+      <xacro:if value="${joint_type == 'continuous'}">
+        <axis xyz="0 1 0"/>
+        <limit effort="${effort_limit}" velocity="${velocity_limit}"/>
+      </xacro:if>
     </joint>
     <gazebo reference="${prefix}${name}_link">
@@ -123,5 +130,5 @@
               Read the explanation at the end of this file about how to set fdir1 for mecanum wheels.
               -->
-              <fdir1 gz:expressed_in="${base_root_fr}">${fdir1_base_root_fr}</fdir1>
+              <fdir1 gz:expressed_in="${fdir1_fr}">${fdir1}</fdir1>
               <!--
               Reference 'http://sdformat.org/tutorials?tut=sdformat_urdf_extensions&cat=specification#gazebo-elements-for-links'
