Commit message: Clarify wheel macro docs and use primitive wheel collisions

File: urdf/wheels/steerable_wheel_macro.xacro (robot description, xacro)
@@ -1,9 +1,10 @@
 <?xml version="1.0"?>
 <!--
+This macro models one steerable wheel assembly: a steering joint/link plus a rotating wheel link/joint.
 Convention for parameter types:
-R means real number (float or double)
-I means integer
-S means string
-B means boolean
+R means real number (with decimal point)
+I means integer (without decimal point)
+S means string (any sequence of characters)
+B means boolean (true or false)
 name (S): name of the wheel, used to name the links and joints.
 prefix (S): optional prefix for the names of the links and joints.
@@ -11,17 +12,17 @@
 use_visual (B): if true, include visual element.
 use_inertial (B): if true, include inertial element.
-v_mesh (S): mesh filename for the visual element of the main link, '${prefix}${name}_rotation_link'. If empty string,
-            a cylinder shape is used with size defined by 'radius' and 'length'.
-            Used only if use_visual is true.
+v_mesh (S): package-relative mesh path used only by the visual element of '${prefix}${name}_rotation_link'
+            (for example: 'robotics_description/meshes/.../wheel.dae').
+            If empty, the visual element falls back to a primitive cylinder defined by 'radius' and 'length'.
+            Ignored when use_visual is false.
 v_mesh_scale (S): Scale of the visual mesh, if use_visual is true and v_mesh is provided.
     v_mesh_scale (S) = 'sx (R) sy (R) sz (R)'.
 v_mesh_origin (S): String of the form 'x (R) y (R) z (R) roll (R) pitch (R) yaw (R)' used to place the visual mesh
-                   w.r.t the frame of the wheel's link (${prefix}${name}_rotation_link).
-                   Used only if use_visual is true and v_mesh is provided.
-                   IMPORTANT: A WHEEL IS CONSIDERED TO BE A CYLINDER WITH ITS ROTATION AXIS ALONG THE Y-AXIS.
-                   THEREFORE, A PROPER ORIGIN MUST BE PROVIDED TO ALIGN THE MESH W.R.T THE WHEEL'S FRAME,
-                   '${prefix}${name}_rotation_link', SO THAT THE Y-AXIS OF THE WHEEL'S FRAME IS THE ROTATION AXIS OF THE
-                   WHEEL MESH, THE X-AXIS OF THE WHEEL'S FRAME IS ALONG THE ROLLING DIRECTION OF THE WHEEL MESH,
-                   AND THE Z-AXIS OF THE WHEEL'S FRAME POINTS UPWARDS.
+                   w.r.t the frame '${prefix}${name}_rotation_link'. Used only if use_visual is true and v_mesh is provided.
+                   IMPORTANT: The wheel frame convention is fixed:
+                     - +Y is the wheel spin axis.
+                     - +X is the rolling direction.
+                     - +Z points upward.
+                   v_mesh_origin must align the mesh to that convention.
 color (S): String of the form 'r (R) g (R) b (R) a (R)'. Used only if use_visual is true.
            If color is not empty, the provided color is applied to the object used in the visual element, either
@@ -31,8 +32,8 @@
                If a mesh is used with no color data associated or a cylinder shape is used, a whitish default color is used
                to display the visual element.
-radius (R): radius of the wheel. Used if v_mesh is an empty string or use_inertial is true (even if a mesh is used,
-               the radius is used to compute the inertia).
-length (R): length of the wheel along its rotation axis (y-axis). Used if v_mesh is an empty string or use_inertial
-               is true (even if a mesh is used, the length is used to compute the inertia).
+radius (R): wheel radius. Used for primitive visual (when v_mesh is empty), always used for collision
+            (collision is always a primitive cylinder), and used for inertia if use_inertial is true.
+length (R): wheel length along the rotation axis (+Y). Used for primitive visual (when v_mesh is empty), always used
+            for collision, and used for inertia if use_inertial is true.
 mass (R): mass of the wheel. Used only if use_inertial is true.
 steerable_joint_type (S): type of the joint connecting the wheel's steerable link to the parent frame.
@@ -68,6 +69,13 @@
 slip2 (R): slip parameter along the secondary direction of motion of the wheel (y-axis of the wheel's frame).
            This parameter should be very low, typically between 0 and 0.01, to prevent the wheel from slipping sideways.
-joint_parent_fr_wheel_fr (S): Pose of the wheel's steerable link frame w.r.t the parent's frame
+joint_parent_fr_wheel_fr (S): Pose of '${prefix}${name}_steerable_link' w.r.t the parent frame.
     joint_parent_fr_wheel_fr (S) = 'x (R) y (R) z (R) roll (R) pitch (R) yaw (R)'.
+    IMPORTANT:
+    This value positions '${prefix}${name}_steerable_link' with respect to the parent frame.
+    The rotation frame '${prefix}${name}_rotation_link' is coincident with the steerable frame, in position, and
+    initially in orientation.
+    The steerable frame changes its orientation with respect to the parent when the wheel is steered.
+    The rotation frame changes its orientation with respect to the steerable frame when the wheel spins.
+    This parameter does not define any offset between steerable and rotation frames.
 Explanation of the default values for the field 'steerable_joint_steerable_limits: "-3.14159265 3.14159265 100 100000"'
 and 'rotation_joint_limits: "100 100000"':
@@ -128,31 +136,22 @@
     <xacro:include filename="$(find robotics_description)/urdf/common/all_commons.xacro"/>
     <!--
-    When the v_mesh_origin parameter was explained above, it was mentioned:
-    IMPORTANT: A WHEEL IS CONSIDERED TO BE A CYLINDER WITH ITS ROTATION AXIS ALONG THE Y-AXIS.
-    THEREFORE, A PROPER ORIGIN MUST BE PROVIDED TO ALIGN THE MESH W.R.T THE WHEEL'S FRAME,
-    '${prefix}${name}_rotation_link', SO THAT THE Y-AXIS OF THE WHEEL'S FRAME IS THE ROTATION AXIS OF THE WHEEL MESH,
-    THE X-AXIS OF THE WHEEL'S FRAME IS ALONG THE ROLLING DIRECTION OF THE WHEEL MESH, AND THE Z-AXIS OF THE WHEEL'S
-    FRAME POINTS UPWARDS.
-    If v_mesh is an empty string, a cylinder shape is used for the visual element. A cylinder shape has its symmetry
-    axis along the z-axis by default. Therefore, the cylinder shape must be rotated along its x-axis (roll = 0.5 * pi),
-    so that its symmetry axis aligns with the y-axis of the wheel's frame.
-    Besides, some friction properties must be modeled for the wheel, because the wheel will interact with the ground.
-    therefore, a wheel always uses a collision element.
-    The collision element is always a cylinder shape (no mesh), also with its symmetry axis (rotation axis) along the
-    y-axis, regardless if the visual element is a mesh or a cylinder shape.
-    The use a basic cylinder shape for the collision element improves the simulation performance.
-    Therefore, a property 'shape_origin = "0.0 0.0 0.0 0.5*pi 0.0 0.0"' is created, which is used as the origin
-    for a cylinder shape, that could be used for the visual element, if no mesh is provided, and is always used for the
-    collision element and for the inertia computation.
+    Frame convention for '${prefix}${name}_rotation_link':
+      - +Y is wheel spin axis.
+      - +X is rolling direction.
+      - +Z points upward.
+    If v_mesh is provided, v_mesh_origin must align the mesh to that convention.
+    If v_mesh is empty, a primitive cylinder is used for visual.
+    Collision is always enabled and always represented as a primitive cylinder (no collision mesh), to keep contacts
+    stable and fast.
+    Primitive cylinders are Z-axis aligned by default in URDF, so they are rotated by +pi/2 around X using:
+      shape_origin = "0.0 0.0 0.0 0.5*pi 0.0 0.0"
+    The same shape_origin is used by visual primitives and collision primitives.
     -->
     <xacro:property name="shape_origin" value="0.0 0.0 0.0 ${0.5 * pi} 0.0 0.0"/>
     <link name="${prefix}${name}_steerable_link">
-      <xacro:if value="${use_visual}">
-        <xacro:property name="v_color" value="${(prefix + name + '_color_steer 1.0 0.0 0.0 1.0')}"/>
-        <xacro:visual_cylinder radius="0.025"
-                               length="${radius}"
-                               shape_origin="${0.5 * radius} 0.0 0.0 0.0 ${pi * 0.5} 0.0"
-                               color="${v_color}"/>
-      </xacro:if>
+      <!--
+      Steerable link is an articulation frame only.
+      Geometry and wheel mass are defined in rotation_link to avoid duplicated visuals/collisions/inertia.
+      -->
       <xacro:null_inertia/>
     </link>
@@ -160,4 +159,5 @@
       ${xacro.fatal("The field 'steerable_joint_type' must be either 'revolute' or 'fixed'")}
     </xacro:if>
+    <!-- Parsed as [x, y, z, roll, pitch, yaw]. -->
     <xacro:property name="j" value="${joint_parent_fr_wheel_fr.split()}"/>
     <joint name="${prefix}${name}_steerable_joint" type="${steerable_joint_type}">
@@ -189,11 +189,11 @@
                                color="${v_color}"/>
       </xacro:if>
-      <!-- The collision element is always used -->
-      <xacro:visual_cylinder mesh="${v_mesh}"
-                             scale="${v_mesh_scale}"
-                             mesh_origin="${v_mesh_origin}"
-                             radius="${radius}"
-                             length="${length}"
-                             shape_origin="${shape_origin}"/>
+      <!--
+      Collision is always enabled for wheel-ground contact and is always represented as
+      a primitive cylinder (no collision mesh), for stable and fast simulation.
+      -->
+      <xacro:collision_cylinder radius="${radius}"
+                                length="${length}"
+                                shape_origin="${shape_origin}"/>
       <xacro:if value="${use_inertial}">
       <!--
@@ -222,7 +222,7 @@
       <child link="${prefix}${name}_rotation_link"/>
       <!--
-      The rotation link frame coincides with the steerable link frame.
-      Initially, there is no rotation between both frames.
-      Once the wheel starts rotating its frame will rotate around the y-axis of the steerable link.
+      rotation_link and steerable_link start coincident (same position and orientation).
+      The zero origin below enforces that rule.
+      This joint adds only wheel spin around +Y of steerable_link.
       -->
       <origin rpy="0.0 0.0 0.0" xyz="0.0 0.0 0.0"/>
@@ -237,4 +237,8 @@
     </joint>
     <gazebo reference="${prefix}${name}_rotation_link">
+      <!--
+      This block configures contact/friction for the URDF collision already defined in rotation_link.
+      It does not create a second collision shape.
+      -->
       <collision>
         <max_contacts>${max_contacts}</max_contacts>

File: urdf/wheels/wheel_macro.xacro (robot description, xacro)
@@ -1,28 +1,28 @@
 <?xml version="1.0"?>
 <!--
+This macro models one non-steerable wheel assembly: a rotating wheel link with its rotation joint.
 Convention for parameter types:
-R means real number (float or double)
-I means integer
-S means string
-B means boolean
+R means real number (with decimal point)
+I means integer (without decimal point)
+S means string (any sequence of characters)
+B means boolean (true or false)
 name (S): name of the wheel, used to name the links and joints.
 prefix (S): optional prefix for the names of the links and joints.
 parent_frame (S): name of the parent frame to which the wheel's root link is attached.
 use_visual (B): if true, include visual element.
-use_collision (B): if true, include collision element.
 use_inertial (B): if true, include inertial element.
-v_mesh (S): mesh filename for the visual element of the main link, '${prefix}${name}_rotation_link'. If empty string,
-            a cylinder shape is used with size defined by 'radius' and 'length'.
-            Used only if use_visual is true.
+v_mesh (S): package-relative mesh path used only by the visual element of '${prefix}${name}_rotation_link'
+            (for example: 'robotics_description/meshes/.../wheel.dae').
+            If empty, the visual element falls back to a primitive cylinder defined by 'radius' and 'length'.
+            Ignored when use_visual is false.
 v_mesh_scale (S): Scale of the visual mesh, if use_visual is true and v_mesh is provided.
     v_mesh_scale (S) = 'sx (R) sy (R) sz (R)'.
 v_mesh_origin (S): String of the form 'x (R) y (R) z (R) roll (R) pitch (R) yaw (R)' used to place the visual mesh
-                   w.r.t the frame of the wheel's link (${prefix}${name}_rotation_link).
-                   Used only if use_visual is true and v_mesh is provided.
-                   IMPORTANT: A WHEEL IS CONSIDERED TO BE A CYLINDER WITH ITS ROTATION AXIS ALONG THE Y-AXIS.
-                   THEREFORE, A PROPER ORIGIN MUST BE PROVIDED TO ALIGN THE MESH W.R.T THE WHEEL'S FRAME,
-                   '${prefix}${name}_rotation_link', SO THAT THE Y-AXIS OF THE WHEEL'S FRAME IS THE ROTATION AXIS OF THE
-                   WHEEL MESH, THE X-AXIS OF THE WHEEL'S FRAME IS ALONG THE ROLLING DIRECTION OF THE WHEEL MESH,
-                   AND THE Z-AXIS OF THE WHEEL'S FRAME POINTS UPWARDS.
+                   w.r.t the frame '${prefix}${name}_rotation_link'. Used only if use_visual is true and v_mesh is provided.
+                   IMPORTANT: The wheel frame convention is fixed:
+                     - +Y is the wheel spin axis.
+                     - +X is the rolling direction.
+                     - +Z points upward.
+                   v_mesh_origin must align the mesh to that convention.
 color (S): String of the form 'r (R) g (R) b (R) a (R)'. Used only if use_visual is true.
            If color is not empty, the provided color is applied to the object used in the visual element, either
@@ -32,8 +32,8 @@
                If a mesh is used with no color data associated or a cylinder shape is used, a whitish default color is used
                to display the visual element.
-radius (R): radius of the wheel. Used if v_mesh is an empty string or use_inertial is true (even if a mesh is used,
-               the radius is used to compute the inertia).
-length (R): length of the wheel along its rotation axis (y-axis). Used if v_mesh is an empty string or use_inertial
-               is true (even if a mesh is used, the length is used to compute the inertia).
+radius (R): wheel radius. Used for primitive visual (when v_mesh is empty), always used for collision
+            (collision is always a primitive cylinder), and used for inertia if use_inertial is true.
+length (R): wheel length along the rotation axis (+Y). Used for primitive visual (when v_mesh is empty), always used
+            for collision, and used for inertia if use_inertial is true.
 mass (R): mass of the wheel. Used only if use_inertial is true.
 rotation_joint_type (S): type of the joint connecting the wheel to the parent frame.
@@ -112,21 +112,15 @@
     <xacro:include filename="$(find robotics_description)/urdf/common/all_commons.xacro"/>
     <!--
-    When the v_mesh_origin parameter was explained above, it was mentioned:
-    IMPORTANT: A WHEEL IS CONSIDERED TO BE A CYLINDER WITH ITS ROTATION AXIS ALONG THE Y-AXIS.
-    THEREFORE, A PROPER ORIGIN MUST BE PROVIDED TO ALIGN THE MESH W.R.T THE WHEEL'S FRAME,
-    '${prefix}${name}_rotation_link', SO THAT THE Y-AXIS OF THE WHEEL'S FRAME IS THE ROTATION AXIS OF THE WHEEL MESH,
-    THE X-AXIS OF THE WHEEL'S FRAME IS ALONG THE ROLLING DIRECTION OF THE WHEEL MESH, AND THE Z-AXIS OF THE WHEEL'S
-    FRAME POINTS UPWARDS.
-    If v_mesh is an empty string, a cylinder shape is used for the visual element. A cylinder shape has its symmetry
-    axis along the z-axis by default. Therefore, the cylinder shape must be rotated along its x-axis (roll = 0.5 * pi),
-    so that its symmetry axis aligns with the y-axis of the wheel's frame.
-    Besides, some friction properties must be modeled for the wheel, because the wheel will interact with the ground.
-    therefore, a wheel always uses a collision element.
-    The collision element is always a cylinder shape (no mesh), also with its symmetry axis (rotation axis) along the
-    y-axis, regardless if the visual element is a mesh or a cylinder shape.
-    The use a basic cylinder shape for the collision element improves the simulation performance.
-    Therefore, a property 'shape_origin = "0.0 0.0 0.0 0.5*pi 0.0 0.0"' is created, which is used as the origin
-    for a cylinder shape, that could be used for the visual element, if no mesh is provided, and is always used for the
-    collision element and for the inertia computation.
+    Frame convention for '${prefix}${name}_rotation_link':
+      - +Y is wheel spin axis.
+      - +X is rolling direction.
+      - +Z points upward.
+    If v_mesh is provided, v_mesh_origin must align the mesh to that convention.
+    If v_mesh is empty, a primitive cylinder is used for visual.
+    Collision is always enabled and always represented as a primitive cylinder (no collision mesh), to keep contacts
+    stable and fast.
+    Primitive cylinders are Z-axis aligned by default in URDF, so they are rotated by +pi/2 around X using:
+      shape_origin = "0.0 0.0 0.0 0.5*pi 0.0 0.0"
+    The same shape_origin is used by visual primitives and collision primitives.
     -->
     <xacro:property name="shape_origin" value="0.0 0.0 0.0 ${0.5 * pi} 0.0 0.0"/>
@@ -143,11 +137,11 @@
                                color="${v_color}"/>
       </xacro:if>
-      <!-- The collision element is always used -->
-      <xacro:visual_cylinder mesh="${v_mesh}"
-                             scale="${v_mesh_scale}"
-                             mesh_origin="${v_mesh_origin}"
-                             radius="${radius}"
-                             length="${length}"
-                             shape_origin="${shape_origin}"/>
+      <!--
+      Collision is always enabled for wheel-ground contact and is always represented as
+      a primitive cylinder (no collision mesh), for stable and fast simulation.
+      -->
+      <xacro:collision_cylinder radius="${radius}"
+                                length="${length}"
+                                shape_origin="${shape_origin}"/>
       <xacro:if value="${use_inertial}">
       <!--
@@ -172,4 +166,5 @@
       ${xacro.fatal("the field 'rotation_joint_type' must be either 'continuous' or 'fixed'")}
     </xacro:if>
+    <!-- Parsed as [x, y, z, roll, pitch, yaw]. -->
     <xacro:property name="j" value="${joint_parent_fr_wheel_fr.split()}"/>
     <joint name="${prefix}${name}_rotation_joint" type="${rotation_joint_type}">
@@ -187,4 +182,8 @@
     </joint>
     <gazebo reference="${prefix}${name}_rotation_link">
+      <!--
+      This block configures contact/friction for the URDF collision already defined in rotation_link.
+      It does not create a second collision shape.
+      -->
       <collision>
         <max_contacts>${max_contacts}</max_contacts>
