Commit message: feat(gz-system-plugins): add reusable Gazebo control wrappers
Add reusable wrappers for the Gazebo system plugins used to control
joints and publish simulation state.

This groups the shared JointController, JointPositionController,
VelocityControl, OdometryPublisher, and JointStatePublisher wrappers,
along with the wheel and fork helper macros that now delegate to them.

Also add a focused xacro regression test for the new wrapper set.

File: urdf/wheels/steerable_wheel_macro.xacro (robot description, xacro)
@@ -1,5 +1,5 @@
 <?xml version="1.0"?>
 <!--
-This macro models one steerable wheel assembly: a steering joint/link plus a rotating wheel link/joint.
+This macro models one steerable wheel assembly: a steering joint plus a rotating wheel link/joint.
 Convention for parameter types:
 R means real number (with decimal point)
@@ -37,14 +37,14 @@
             for collision, and used for inertia if use_inertial is true.
 mass (R): mass of the wheel. Used only if use_inertial is true.
-steerable_joint_type (S): type of the joint connecting the wheel's steerable link to the parent frame.
-    steerable_joint_type (S) = 'revolute' | 'fixed'.
+steering_joint_type (S): type of the joint connecting the wheel's steerable link to the parent frame.
+    steering_joint_type (S) = 'revolute' | 'fixed'.
     If 'fixed' is used, the wheel will not be able to steer in simulation.
-steerable_joint_steerable_limits (S): limits of the steerable joint.
-    steerable_joint_steerable_limits (S) = 'lower_limit (R) upper_limit (R) velocity (R) effort (R)'.
-    lower_limit (R): lower position limit of the steerable joint (radians).
-    upper_limit (R): upper position limit of the steerable joint (radians).
-    velocity (R): velocity limit of the steerable joint (radians/second).
-    effort (R): effort limit of the steerable joint (newton-meters).
-    Used only if steerable_joint_type is 'revolute'.
+steering_joint_limits (S): limits of the steering joint.
+    steering_joint_limits (S) = 'lower_limit (R) upper_limit (R) velocity (R) effort (R)'.
+    lower_limit (R): lower position limit of the steering joint (radians).
+    upper_limit (R): upper position limit of the steering joint (radians).
+    velocity (R): velocity limit of the steering joint (radians/second).
+    effort (R): effort limit of the steering joint (newton-meters).
+    Used only if steering_joint_type is 'revolute'.
 rotation_joint_type (S): type of the joint connecting the wheel to the parent frame.
     rotation_joint_type (S) = 'continuous' | 'fixed'.
@@ -78,5 +78,5 @@
     The rotation frame changes its orientation with respect to the steerable frame when the wheel spins.
     This parameter does not define any offset between steerable and rotation frames.
-Explanation of the default values for the field 'steerable_joint_steerable_limits: "-3.14159265 3.14159265 100 100000"'
+Explanation of the default values for the field 'steering_joint_limits: "-3.14159265 3.14159265 100 100000"'
 and 'rotation_joint_limits: "100 100000"':
 ======================================================================================================================
@@ -87,12 +87,12 @@
 trajectory following) without being constrained by the physical limitations of real-world motors.
 in essence, the software logic is tested in isolation.
-steerable_joint_steerable_limits.lower_limit = "-3.14159265" (radians).
+steering_joint_limits.lower_limit = "-3.14159265" (radians).
 This allows the wheel to steer a full -180 degrees.
-steerable_joint_steerable_limits.upper_limit = "3.14159265" (radians).
+steering_joint_limits.upper_limit = "3.14159265" (radians).
 This allows the wheel to steer a full +180 degrees.
-steerable_joint_steerable_limits.velocity = "100" (radians/second).
+steering_joint_limits.velocity = "100" (radians/second).
 This means the wheel can orient itself extremely quickly.
-steerable_joint_steerable_limits.effort = "100000" (newton-meters).
-For a steerable joint, this represents the maximum torque the joint can apply to change its orientation. It is not
+steering_joint_limits.effort = "100000" (newton-meters).
+For a steering joint, this represents the maximum torque the joint can apply to change its orientation. It is not
 an important value for most robot applications, as steering usually requires much less torque than driving. However,
 setting it to a very high value ensures that the steering action is not limited by the simulator.
@@ -123,6 +123,6 @@
                        length
                        mass
-                       steerable_joint_type:=revolute
-                       steerable_joint_steerable_limits:='-3.14159265 3.14159265 100.0 100000.0'
+                       steering_joint_type:=revolute
+                       steering_joint_limits:='-3.14159265 3.14159265 100.0 100000.0'
                        rotation_joint_type:=continuous
                        rotation_joint_limits:='100.0 100000.0'
@@ -156,23 +156,23 @@
       <xacro:null_inertia/>
     </link>
-    <xacro:if value="${steerable_joint_type not in ('revolute', 'fixed')}">
-      ${xacro.fatal("The field 'steerable_joint_type' must be either 'revolute' or 'fixed'")}
+    <xacro:if value="${steering_joint_type not in ('revolute', 'fixed')}">
+      ${xacro.fatal("The field 'steering_joint_type' must be either 'revolute' or 'fixed'")}
     </xacro:if>
     <!-- Parsed as [x, y, z, roll, pitch, yaw]. -->
     <xacro:property name="j" value="${joint_parent_fr_wheel_fr.split()}"/>
-    <joint name="${prefix}${name}_steerable_joint" type="${steerable_joint_type}">
+    <joint name="${prefix}${name}_steering_joint" type="${steering_joint_type}">
       <parent link="${parent_frame}"/>
       <child link="${prefix}${name}_steerable_link"/>
       <origin rpy="${j[3]} ${j[4]} ${j[5]}" xyz="${j[0]} ${j[1]} ${j[2]}"/>
-      <xacro:if value="${steerable_joint_type == 'revolute'}">
-        <xacro:property name="sj_limits_seq" value="${steerable_joint_steerable_limits.split()}"/>
-        <xacro:if value="${len(sj_limits_seq) != 4}">
-            ${xacro.fatal("steerable_wheel: steerable_joint_steerable_limits must have 4 elements: 'lower_limit (R) upper_limit (R) velocity (R) effort (R)'")}
+      <xacro:if value="${steering_joint_type == 'revolute'}">
+        <xacro:property name="steering_joint_limits_seq" value="${steering_joint_limits.split()}"/>
+        <xacro:if value="${len(steering_joint_limits_seq) != 4}">
+            ${xacro.fatal("steerable_wheel: steering_joint_limits must have 4 elements: 'lower_limit (R) upper_limit (R) velocity (R) effort (R)'")}
         </xacro:if>
         <axis xyz="0 0 1"/>
-        <limit lower="${sj_limits_seq[0]}"
-               upper="${sj_limits_seq[1]}"
-               velocity="${sj_limits_seq[2]}"
-               effort="${sj_limits_seq[3]}"/>
+        <limit lower="${steering_joint_limits_seq[0]}"
+               upper="${steering_joint_limits_seq[1]}"
+               velocity="${steering_joint_limits_seq[2]}"
+               effort="${steering_joint_limits_seq[3]}"/>
       </xacro:if>
     </joint>

Commit message: feat(wheels): [0520-01] Add joint dynamics parameters
Add wheel and steerable wheel joint dynamics parameters with default zero damping and friction so existing macro call sites remain compatible while callers can configure damping and friction explicitly.

File: urdf/wheels/steerable_wheel_macro.xacro (robot description, xacro)
@@ -117,6 +117,8 @@
                        steering_joint_type:=revolute
                        steering_joint_limits:='-3.14159265 3.14159265 100.0 100000.0'
+                       steering_joint_dynamics:='0.0 0.0'
                        rotation_joint_type:=continuous
                        rotation_joint_limits:='100.0 100000.0'
+                       rotation_joint_dynamics:='0.0 0.0'
                        max_contacts:=10
                        mu:=0.5
@@ -163,4 +165,12 @@
       )}
     </xacro:if>
+    <xacro:property name="steering_joint_limits_seq"   value="${str(steering_joint_limits).split()}"/>
+    <xacro:property name="steering_joint_dynamics_seq" value="${str(steering_joint_dynamics).split()}"/>
+    <xacro:if value="${steering_joint_type == 'revolute' and len(steering_joint_limits_seq) != 4}">
+      ${xacro.fatal("steerable_wheel: steering_joint_limits must have 4 elements: 'lower_limit (R) upper_limit (R) velocity (R) effort (R)'")}
+    </xacro:if>
+    <xacro:if value="${steering_joint_type == 'revolute' and len(steering_joint_dynamics_seq) != 2}">
+      ${xacro.fatal("steerable_wheel: steering_joint_dynamics must have 2 elements: 'damping friction'")}
+    </xacro:if>
     <joint name="${prefix}${name}_steering_joint" type="${steering_joint_type}">
       <parent link="${parent_frame}"/>
@@ -168,9 +178,6 @@
       <origin rpy="${j[3]} ${j[4]} ${j[5]}" xyz="${j[0]} ${j[1]} ${j[2]}"/>
       <xacro:if value="${steering_joint_type == 'revolute'}">
-        <xacro:property name="steering_joint_limits_seq" value="${steering_joint_limits.split()}"/>
-        <xacro:if value="${len(steering_joint_limits_seq) != 4}">
-            ${xacro.fatal("steerable_wheel: steering_joint_limits must have 4 elements: 'lower_limit (R) upper_limit (R) velocity (R) effort (R)'")}
-        </xacro:if>
         <axis xyz="0 0 1"/>
+        <dynamics damping="${steering_joint_dynamics_seq[0]}" friction="${steering_joint_dynamics_seq[1]}"/>
         <limit lower="${steering_joint_limits_seq[0]}"
                upper="${steering_joint_limits_seq[1]}"
@@ -220,4 +227,12 @@
       ${xacro.fatal("The field 'rotation_joint_type' must be either 'continuous' or 'fixed'")}
     </xacro:if>
+    <xacro:property name="rj_limits_seq"   value="${str(rotation_joint_limits).split()}"/>
+    <xacro:property name="rj_dynamics_seq" value="${str(rotation_joint_dynamics).split()}"/>
+    <xacro:if value="${rotation_joint_type == 'continuous' and len(rj_limits_seq) != 2}">
+      ${xacro.fatal("steerable_wheel: rotation_joint_limits must have 2 elements: 'velocity (R) effort (R)'")}
+    </xacro:if>
+    <xacro:if value="${rotation_joint_type == 'continuous' and len(rj_dynamics_seq) != 2}">
+      ${xacro.fatal("steerable_wheel: rotation_joint_dynamics must have 2 elements: 'damping friction'")}
+    </xacro:if>
     <joint name="${prefix}${name}_rotation_joint" type="${rotation_joint_type}">
       <parent link="${prefix}${name}_steerable_link"/>
@@ -230,9 +245,6 @@
       <origin rpy="0.0 0.0 0.0" xyz="0.0 0.0 0.0"/>
       <xacro:if value="${rotation_joint_type == 'continuous'}">
-        <xacro:property name="rj_limits_seq" value="${rotation_joint_limits.split()}"/>
-        <xacro:if value="${len(rj_limits_seq) != 2}">
-            ${xacro.fatal("steerable_wheel: rotation_joint_limits must have 2 elements: 'velocity (R) effort (R)'")}
-        </xacro:if>
         <axis xyz="0 1 0"/>
+        <dynamics damping="${rj_dynamics_seq[0]}" friction="${rj_dynamics_seq[1]}"/>
         <limit velocity="${rj_limits_seq[0]}" effort="${rj_limits_seq[1]}"/>
       </xacro:if>

File: urdf/wheels/wheel_macro.xacro (robot description, xacro)
@@ -94,4 +94,5 @@
                        rotation_joint_type:=continuous
                        rotation_joint_limits:='100.0 100000.0'
+                       rotation_joint_dynamics:='0.0 0.0'
                        max_contacts:=10
                        mu:=0.5
@@ -171,4 +172,12 @@
       ${xacro.fatal("wheel: joint_parent_fr_wheel_fr must have 6 elements: 'x y z roll pitch yaw'")}
     </xacro:if>
+    <xacro:property name="rj_limits_seq"   value="${str(rotation_joint_limits).split()}"/>
+    <xacro:property name="rj_dynamics_seq" value="${str(rotation_joint_dynamics).split()}"/>
+    <xacro:if value="${rotation_joint_type == 'continuous' and len(rj_limits_seq) != 2}">
+      ${xacro.fatal("wheel: rotation_joint_limits must have 2 elements: 'velocity (R) effort (R)'")}
+    </xacro:if>
+    <xacro:if value="${rotation_joint_type == 'continuous' and len(rj_dynamics_seq) != 2}">
+      ${xacro.fatal("wheel: rotation_joint_dynamics must have 2 elements: 'damping friction'")}
+    </xacro:if>
     <joint name="${prefix}${name}_rotation_joint" type="${rotation_joint_type}">
       <parent link="${parent_frame}"/>
@@ -176,9 +185,6 @@
       <origin rpy="${j[3]} ${j[4]} ${j[5]}" xyz="${j[0]} ${j[1]} ${j[2]}"/>
       <xacro:if value="${rotation_joint_type == 'continuous'}">
-        <xacro:property name="rj_limits_seq" value="${rotation_joint_limits.split()}"/>
-        <xacro:if value="${len(rj_limits_seq) != 2}">
-            ${xacro.fatal("wheel: rotation_joint_limits must have 2 elements: 'velocity (R) effort (R)'")}
-        </xacro:if>
         <axis xyz="0 1 0"/>
+        <dynamics damping="${rj_dynamics_seq[0]}" friction="${rj_dynamics_seq[1]}"/>
         <limit velocity="${rj_limits_seq[0]}" effort="${rj_limits_seq[1]}"/>
       </xacro:if>
