Commit message: Added ballast to the base, to lower the center of mass of the base, so the base is stable when moving.

File: urdf/bases/rectangular_body_macro.xacro (robot description, xacro)
@@ -36,4 +36,6 @@
                         size
                         ground_clearance
+                        ballast_mass_ratio:=0.95
+                        ballast_height_ratio:=0.1
                         mesh_visual:=''
                         mesh_visual_has_color:=False
@@ -48,7 +50,7 @@
     -->
     <xacro:property name="body_size_lst" value="${size.split()}"/>
-    <xacro:property name="body_size_x"   value="${body_size_lst[0]}"/>
-    <xacro:property name="body_size_y"   value="${body_size_lst[1]}"/>
-    <xacro:property name="body_size_z"   value="${body_size_lst[2]}"/>
+    <xacro:property name="body_size_x"   value="${float(body_size_lst[0])}"/>
+    <xacro:property name="body_size_y"   value="${float(body_size_lst[1])}"/>
+    <xacro:property name="body_size_z"   value="${float(body_size_lst[2])}"/>
     <!--
     Definition of the link ${prefix}${name}_footprint_link.
@@ -58,4 +60,5 @@
     <!--
     Definition of the link '${prefix}${name}_link'.
+    The proportion of the mass that is not ballast is considered to be uniformly distributed in the box.
     -->
     <xacro:link_r
@@ -65,5 +68,5 @@
       use_collision="True"
       use_inertia="True"
-      mass="${mass}"
+      mass="${(1.0 - ballast_mass_ratio) * mass}"
       size="${size}"
       mesh_visual="${mesh_visual}"
@@ -82,4 +85,47 @@
       <origin rpy="0 0 0" xyz="0 0 ${ground_clearance}"/>
     </joint>
+    <!--
+    Ballast to adjust the center of mass of the base.
+    The ballast is modeled as a box of the same size as the base in the X and Y directions, but with a height equal to
+    'ballast_height_ratio * body_size_z'.
+    'ballast_height_ratio' must be in the range [0, 1], and represents the proportion of the base height that the
+    ballast occupies. It should be a small value, e.g., 0.1 (10% of the base height), so that the center of mass of the
+    base is lowered.
+    The ballast mass is equal to 'ballast_mass_ratio * mass'.
+    'ballast_mass_ratio' must be in the range [0, 1], and represents the proportion of the total mass of the base that
+    the ballast occupies. It should be a large value, e.g., 0.9 (90% of the total mass), so that the center of mass of
+    the base is lowered.
+    The ballast is positioned at the bottom of the base, so its center is at a height of
+    '0.5 * ballast_height_ratio * body_size_z'.
+    -->
+    <!--
+    The value of attribute 'value' must not contain the '<' character.
+    &lt; is equivalent to '<'.
+    -->
+    <xacro:if value="${ballast_mass_ratio &lt; 0.0 or ballast_mass_ratio > 1.0}">
+      ${xacro.fatal("The 'ballast_mass_ratio' parameter must be in the range [0, 1].")}
+    </xacro:if>
+    <xacro:if value="${ballast_height_ratio &lt; 0.0 or ballast_height_ratio > 1.0}">
+      ${xacro.fatal("The 'ballast_height_ratio' parameter must be in the range [0, 1].")}
+    </xacro:if>
+    <xacro:property name="ballast_size_z" value="${ballast_height_ratio * body_size_z}"/>
+    <xacro:link_r
+      name="${name}_ballast"
+      prefix="${prefix}"
+      use_visual="False"
+      use_collision="False"
+      use_inertia="True"
+      mass="${ballast_mass_ratio * mass}"
+      size="${body_size_x} ${body_size_y} ${ballast_size_z}"
+      vci_pose="0 0 0 0 0 0"/>
+    <!--
+    Joint '${prefix}${name}_ballast_joint' connects the link '${prefix}${name}_link'
+    with the link '${prefix}${name}_ballast_link'.
+    -->
+    <joint name="${prefix}${name}_ballast_joint" type="fixed">
+      <parent link="${prefix}${name}_link"/>
+      <child link="${prefix}${name}_ballast_link"/>
+      <origin rpy="0 0 0" xyz="0 0 ${0.5 * ballast_size_z}"/>
+    </joint>
   </xacro:macro>
 </robot>

File: urdf/robots/flart/description.xacro (robot description, xacro)
@@ -80,16 +80,19 @@
   <xacro:property name="robot_size_z" value="${desc_cfg['size']['z']}"/>
   <!-- ===================================================================== -->
-  <!-- MECANUM RECTANGULAR BASE -->
-  <!-- ===================================================================== -->
-  <!--
-  A base is composed of a body and wheels.
-  In this case, the base is rectangular with mecanum wheels.
+  <!-- RECTANGULAR BASE -->
+  <!-- ===================================================================== -->
+  <!--
+  base = body + wheels.
+  In this case, the base is rectangular with 3 wheels, one in the front and two in the back.
   The rectangular_body macro defines the following links and joints:
   - Links:
     * ${prefix}${name}_footprint_link = ${robot_prefix}${base_name}_footprint_link
     * ${prefix}${name}_link = ${robot_prefix}${base_name}_link
+    * ${prefix}${name}_ballast_link = ${robot_prefix}${base_name}_ballast_link
   - Joints:
     * ${prefix}${name}_joint = ${robot_prefix}${base_name}_joint, joining the links
       ${robot_prefix}${base_name}_footprint_link and ${robot_prefix}${base_name}_link.
+    * ${prefix}${name}_ballast_joint = ${robot_prefix}${base_name}_ballast_joint, joining the links
+      ${robot_prefix}${base_name}_link and ${robot_prefix}${base_name}_ballast_link.
   THE LINK '${robot_prefix}${base_name}_link' IS LOCATED AT THE CENTER OF THE BOTTOM FACE OF THE BASE BODY.
   THE LINK '${robot_prefix}${base_name}_footprint_link' IS LOCATED ON THE GROUND, JUST BELOW THE LINK
@@ -112,4 +115,6 @@
     size="${base_body_size_x} ${base_body_size_y} ${base_body_size_z}"
     ground_clearance="${base_body_ground_clearance}"
+    ballast_mass_ratio="0.95"
+    ballast_height_ratio="0.1"
     mesh_visual="${base_body_mesh_visual if use_visual_meshes else ''}"
     mesh_visual_has_color="${base_body_mesh_visual_has_color}"
