Commit message: Extract files regarding flart robot
Created a new package and dedicated package for the flart robot

File: urdf/bases/set_rectangular_body_props_macro.xacro (robot description, xacro)
@@ -10,10 +10,16 @@
     <xacro:property name="${prop_prefix}_track_width"      value="${desc_cfg['track_width']}"      scope="parent"/>
     <xacro:property name="${prop_prefix}_ground_clearance" value="${desc_cfg['ground_clearance']}" scope="parent"/>
-    <xacro:property name="mesh_dir"                  value="$(find eut_robotics_description)/meshes"/>
-    <xacro:property name="_base_body_mesh_visual"    value="${desc_cfg['mesh_visual']}"/>
-    <xacro:property name="_base_body_mesh_collision" value="${desc_cfg['mesh_collision']}"/>
-    <xacro:property name="${prop_prefix}_mesh_visual"
-                    value="${mesh_dir + '/' + _base_body_mesh_visual if _base_body_mesh_visual else ''}"
-                    scope="parent"/>
+    <xacro:property name="_base_body_mesh_visual"    value="${desc_cfg.get('mesh_visual', '')}"/>
+    <xacro:property name="_base_body_mesh_collision" value="${desc_cfg.get('mesh_collision', '')}"/>
+    <xacro:if value="${_base_body_mesh_visual is not None and _base_body_mesh_visual != ''}">
+      <xacro:property name="${prop_prefix}_mesh_visual"
+                      value="${_base_body_mesh_visual}"
+                      scope="parent"/>
+    </xacro:if>
+    <xacro:if value="${_base_body_mesh_visual is None or _base_body_mesh_visual == ''}">
+      <xacro:property name="${prop_prefix}_mesh_visual"
+                      value=""
+                      scope="parent"/>
+    </xacro:if>
     <xacro:property name="${prop_prefix}_mesh_visual_has_color"
                     value="${desc_cfg['mesh_visual_has_color']}"
@@ -23,7 +29,14 @@
                     value="${_base_body_color['r']} ${_base_body_color['g']} ${_base_body_color['b']} ${_base_body_color['a']}"
                     scope="parent"/>
-    <xacro:property name="${prop_prefix}_mesh_collision"
-                    value="${mesh_dir + '/' + _base_body_mesh_collision if _base_body_mesh_collision else ''}"
-                    scope="parent"/>
+    <xacro:if value="${_base_body_mesh_collision is not None and _base_body_mesh_collision != ''}">
+      <xacro:property name="${prop_prefix}_mesh_collision"
+                      value="${_base_body_mesh_collision}"
+                      scope="parent"/>
+    </xacro:if>
+    <xacro:unless value="${_base_body_mesh_collision is None or _base_body_mesh_collision == ''}">
+      <xacro:property name="${prop_prefix}_mesh_collision"
+                      value=""
+                      scope="parent"/>
+    </xacro:unless>
     <xacro:property name="_base_body_scale" value="${desc_cfg['scale']}"/>
     <xacro:property name="${prop_prefix}_scale"

File: urdf/common/all_commons.xacro (robot description, xacro)
@@ -6,3 +6,5 @@
   <xacro:include filename="$(find eut_robotics_description)/urdf/common/link_s_macro.xacro"/>
   <xacro:include filename="$(find eut_robotics_description)/urdf/common/link_w_shape_macro.xacro"/>
+  <xacro:include filename="$(find eut_robotics_description)/urdf/common/make_robot_namespace_macro.xacro"/>
+  <xacro:include filename="$(find eut_robotics_description)/urdf/common/make_robot_prefix_macro.xacro"/>
 </robot>

File: urdf/common/link_c_macro.xacro (robot description, xacro)
@@ -107,8 +107,5 @@
           <xacro:if value="${mesh_visual != ''}"> <!-- There is mesh for visual -->
             <geometry>
-              <!--
               <mesh filename="package://${mesh_visual}" scale="${scale}"/>
-              -->
-              <mesh filename="file://${mesh_visual}" scale="${scale}"/>
             </geometry>
             <xacro:unless value="${mesh_visual_has_color}"> <!-- Check if mesh_visual must be colored -->
@@ -130,8 +127,5 @@
           <xacro:if value="${mesh_collision != ''}"> <!-- There is mesh for collision -->
             <geometry>
-              <!--
               <mesh filename="package://${mesh_collision}" scale="${scale}"/>
-              -->
-              <mesh filename="file://${mesh_collision}" scale="${scale}"/>
             </geometry>
           </xacro:if>

File: urdf/common/link_r_macro.xacro (robot description, xacro)
@@ -55,8 +55,5 @@
           <xacro:if value="${mesh_visual != ''}"> <!-- There is mesh for visual -->
             <geometry>
-              <!--
               <mesh filename="package://${mesh_visual}" scale="${scale}"/>
-              -->
-              <mesh filename="file://${mesh_visual}" scale="${scale}"/>
             </geometry>
             <xacro:unless value="${mesh_visual_has_color}"> <!-- Check if mesh_visual must be colored -->
@@ -78,8 +75,5 @@
           <xacro:if value="${mesh_collision != ''}"> <!-- There is mesh for collision -->
             <geometry>
-              <!--
               <mesh filename="package://${mesh_collision}" scale="${scale}"/>
-              -->
-              <mesh filename="file://${mesh_collision}" scale="${scale}"/>
             </geometry>
           </xacro:if>

File: urdf/common/link_s_macro.xacro (robot description, xacro)
@@ -38,8 +38,5 @@
           <xacro:if value="${mesh_visual != ''}"> <!-- There is mesh for visual -->
             <geometry>
-              <!--
               <mesh filename="package://${mesh_visual}" scale="${scale}"/>
-              -->
-              <mesh filename="file://${mesh_visual}" scale="${scale}"/>
             </geometry>
             <xacro:unless value="${mesh_visual_has_color}"> <!-- Check if mesh_visual must be colored -->
@@ -61,8 +58,5 @@
           <xacro:if value="${mesh_collision != ''}"> <!-- There is mesh for collision -->
             <geometry>
-              <!--
               <mesh filename="package://${mesh_collision}" scale="${scale}"/>
-              -->
-              <mesh filename="file://${mesh_collision}" scale="${scale}"/>
             </geometry>
           </xacro:if>

File: urdf/extras/set_fork_props_macro.xacro (robot description, xacro)
@@ -11,51 +11,70 @@
                     value="${tine_cfg['size']['x']} ${tine_cfg['size']['y']} ${tine_cfg['size']['z']}"
                     scope="parent"/>
-    <!--
-    The property 'mesh' is local to this macro, so no need to use scope="parent". This property is used to set
-    another property in the parent scope, which is '${prop_prefix}_mesh'.
-    -->
-    <!--
-    The property 'mesh' is local to this macro, so no need to use scope="parent". This property is used to set
-    another property in the parent scope, which is '${prop_prefix}_mesh'.
-    -->
-    <xacro:property name="mesh_dir" value="$(find eut_robotics_description)/meshes"/>
-    <xacro:property name="${prop_prefix}_tine_mesh_visual"
-                    value="${mesh_dir + '/' + tine_cfg['mesh_visual'] if tine_cfg['mesh_visual'] else ''}"
-                    scope="parent"/>
+    <xacro:property name="_tine_mesh_visual"    value="${tine_cfg.get('mesh_visual', '')}"/>
+    <xacro:property name="_tine_mesh_collision" value="${tine_cfg.get('mesh_collision', '')}"/>
+    <xacro:if value="${_tine_mesh_visual is not None and _tine_mesh_visual != ''}">
+      <xacro:property name="${prop_prefix}_tine_mesh_visual"
+                      value="${_tine_mesh_visual}"
+                      scope="parent"/>
+    </xacro:if>
+    <xacro:if value="${_tine_mesh_visual is None or _tine_mesh_visual == ''}">
+      <xacro:property name="${prop_prefix}_mesh_visual"
+                      value=""
+                      scope="parent"/>
+    </xacro:if>
     <xacro:property name="${prop_prefix}_tine_mesh_visual_has_color"
                     value="${tine_cfg['mesh_visual_has_color']}"
                     scope="parent"/>
-    <xacro:property name="${prop_prefix}_tine_mesh_collision"
-                    value="${mesh_dir + '/' + tine_cfg['mesh_collision'] if tine_cfg['mesh_collision'] else ''}"
+    <xacro:property name="_fork_color" value="${desc_cfg.get('color', dict(r = 0, g = 0, b = 0, a = 1))}"/>
+    <xacro:property name="${prop_prefix}_color"
+                    value="${_fork_color['r']} ${_fork_color['g']} ${_fork_color['b']} ${_fork_color['a']}"
                     scope="parent"/>
-      <!--
-      If you can accommodate all the values that constitute the string in a single line in the 'value' field, you can do
-      it directly as:
-      <xacro:property name="${prop_prefix}_tine_mass"
-                      value="${tine_cfg['mass']}"
+    <xacro:if value="${_tine_mesh_collision is not None and _tine_mesh_collision != ''}">
+      <xacro:property name="${prop_prefix}_mesh_collision"
+                      value="${_tine_mesh_collision}"
                       scope="parent"/>
-      But if you need to split the line that you assign to the 'value' field, because the line is too long to fit in a
-      single with a resonable length, then you have to use the 'join' method as done below to avoid sevaral whitespaces
-      in the resulting string separating the values when the macro is expanded.
-      -->
+    </xacro:if>
+    <xacro:unless value="${_tine_mesh_collision is None or _tine_mesh_collision == ''}">
+      <xacro:property name="${prop_prefix}_mesh_collision"
+                      value=""
+                      scope="parent"/>
+    </xacro:unless>
+    <xacro:property name="_tine_scale" value="${tine_cfg['scale']}"/>
     <xacro:property name="${prop_prefix}_tine_scale"
-                    value="${' '.join([str(tine_cfg['scale']['x']),
-                                       str(tine_cfg['scale']['y']),
-                                       str(tine_cfg['scale']['z'])])
-                            if tine_cfg['scale'] else ''}"
+                    value="${_tine_scale['x']} ${_tine_scale['y']} ${_tine_scale['z']}"
                     scope="parent"/>
-    <xacro:property name="${prop_prefix}_base_mass"   value="${base_cfg['mass']}"      scope="parent"/>
-    <xacro:property name="${prop_prefix}_base_size_x" value="${base_cfg['size']['x']}" scope="parent"/>
-    <xacro:property name="${prop_prefix}_base_size_y" value="${base_cfg['size']['y']}" scope="parent"/>
-    <xacro:property name="${prop_prefix}_base_size_z" value="${base_cfg['size']['z']}" scope="parent"/>
+    <xacro:property name="${prop_prefix}_base_mass"
+                    value="${base_cfg['mass']}"
+                    scope="parent"/>
+    <xacro:property name="${prop_prefix}_base_size_x"
+                    value="${base_cfg['size']['x']}"
+                    scope="parent"/>
+    <xacro:property name="${prop_prefix}_base_size_y"
+                    value="${base_cfg['size']['y']}"
+                    scope="parent"/>
+    <xacro:property name="${prop_prefix}_base_size_z"
+                    value="${base_cfg['size']['z']}"
+                    scope="parent"/>
     <xacro:property name="${prop_prefix}_base_size"
                     value="${base_cfg['size']['x']} ${base_cfg['size']['y']} ${base_cfg['size']['z']}"
                     scope="parent"/>
-    <xacro:property name="${prop_prefix}_use_inertia"     value="${desc_cfg['use_inertia']}"      scope="parent"/>
-    <xacro:property name="${prop_prefix}_tine_separation" value="${desc_cfg['tine_separation']}"  scope="parent"/>
-    <xacro:property name="${prop_prefix}_lower_limit"     value="${desc_cfg['lower_limit']}"      scope="parent"/>
-    <xacro:property name="${prop_prefix}_upper_limit"     value="${desc_cfg['upper_limit']}"      scope="parent"/>
-    <xacro:property name="${prop_prefix}_brake_distance"  value="${desc_cfg['brake_distance']}"   scope="parent"/>
-    <xacro:property name="${prop_prefix}_velocity_limit"  value="${desc_cfg['velocity_limit']}"   scope="parent"/>
+    <xacro:property name="${prop_prefix}_use_inertia"
+                    value="${desc_cfg['use_inertia']}"
+                    scope="parent"/>
+    <xacro:property name="${prop_prefix}_tine_separation"
+                    value="${desc_cfg['tine_separation']}"
+                    scope="parent"/>
+    <xacro:property name="${prop_prefix}_lower_limit"
+                    value="${desc_cfg['lower_limit']}"
+                    scope="parent"/>
+    <xacro:property name="${prop_prefix}_upper_limit"
+                    value="${desc_cfg['upper_limit']}"
+                    scope="parent"/>
+    <xacro:property name="${prop_prefix}_brake_distance"
+                    value="${desc_cfg['brake_distance']}"
+                    scope="parent"/>
+    <xacro:property name="${prop_prefix}_velocity_limit"
+                    value="${desc_cfg['velocity_limit']}"
+                    scope="parent"/>
     <xacro:property name="${prop_prefix}_velocity_limit_full_effort"
                     value="${desc_cfg['velocity_limit_full_effort']}"
@@ -76,10 +95,4 @@
                     value="${desc_cfg['clearance_under_fork']}"
                     scope="parent"/>
-    <xacro:property name="${prop_prefix}_color"
-                    value="${' '.join([str(desc_cfg['color']['r']),
-                                       str(desc_cfg['color']['g']),
-                                       str(desc_cfg['color']['b']),
-                                       str(desc_cfg['color']['a'])])}"
-                    scope="parent"/>
   </xacro:macro>
 </robot>

File: urdf/sensors/imus/generic_macros/set_imu_props_macro.xacro (robot description, xacro)
@@ -42,34 +42,37 @@
                                         str(desc_cfg['shape']['size']['z'])])}"
                     scope="parent"/>
-    <!--
-    The property 'mesh' is local to this macro, so no need to use scope="parent". This property is used to set
-    another property in the parent scope, which is '${prop_prefix}_mesh'.
-    -->
-    <xacro:property name="mesh_dir" value="$(find eut_robotics_description)/meshes"/>
-    <xacro:property name="${prop_prefix}_mesh_visual"
-                    value="${mesh_dir + '/' + desc_cfg['mesh_visual'] if desc_cfg['mesh_visual'] else ''}"
-                    scope="parent"/>
+    <xacro:property name="_imu_mesh_visual"    value="${desc_cfg.get('mesh_visual', '')}"/>
+    <xacro:property name="_imu_mesh_collision" value="${desc_cfg.get('mesh_collision', '')}"/>
+    <xacro:if value="${_imu_mesh_visual is not None and _imu_mesh_visual != ''}">
+      <xacro:property name="${prop_prefix}_mesh_visual"
+                      value="${_imu_mesh_visual}"
+                      scope="parent"/>
+    </xacro:if>
+    <xacro:if value="${_imu_mesh_visual is None or _imu_mesh_visual == ''}">
+      <xacro:property name="${prop_prefix}_mesh_visual"
+                      value=""
+                      scope="parent"/>
+    </xacro:if>
     <xacro:property name="${prop_prefix}_mesh_visual_has_color"
                     value="${desc_cfg['mesh_visual_has_color']}"
                     scope="parent"/>
-    <xacro:property name="${prop_prefix}_mesh_collision"
-                    value="${mesh_dir + '/' + desc_cfg['mesh_collision'] if desc_cfg['mesh_collision'] else ''}"
+    <xacro:property name="_imu_color"
+                    value="${desc_cfg.get('color', dict(r = 0, g = 0, b = 0, a = 1))}"/>
+    <xacro:property name="${prop_prefix}_color"
+                    value="${_imu_color['r']} ${_imu_color['g']} ${_imu_color['b']} ${_imu_color['a']}"
                     scope="parent"/>
-    <!--
-    To be able to do the comparion and the assignment of the resulting string in a single line, being the string
-    a concatenation of several values, you have to combine those values in a list, and then use 'join' to create the
-    string.
-    -->
+    <xacro:if value="${_imu_mesh_collision is not None and _imu_mesh_collision != ''}">
+      <xacro:property name="${prop_prefix}_mesh_collision"
+                      value="${_imu_mesh_collision}"
+                      scope="parent"/>
+    </xacro:if>
+    <xacro:unless value="${_imu_mesh_collision is None or _imu_mesh_collision == ''}">
+      <xacro:property name="${prop_prefix}_mesh_collision"
+                      value=""
+                      scope="parent"/>
+    </xacro:unless>
+    <xacro:property name="_imu_scale" value="${desc_cfg['scale']}"/>
     <xacro:property name="${prop_prefix}_scale"
-                    value="${' '.join([str(desc_cfg['scale']['x']),
-                                       str(desc_cfg['scale']['y']),
-                                       str(desc_cfg['scale']['z'])])
-                            if desc_cfg['scale'] else ''}"
-                    scope="parent"/>
-    <xacro:property name="${prop_prefix}_color"
-                    value="${' '.join([str(desc_cfg['color']['r']),
-                                       str(desc_cfg['color']['g']),
-                                       str(desc_cfg['color']['b']),
-                                       str(desc_cfg['color']['a'])])}"
+                    value="${_imu_scale['x']} ${_imu_scale['y']} ${_imu_scale['z']}"
                     scope="parent"/>
     <xacro:property name="${prop_prefix}_joint_root_fr_data_fr"

File: urdf/sensors/lidars/generic_macros/set_lidar_2d_props_macro.xacro (robot description, xacro)
@@ -42,34 +42,36 @@
                                         str(desc_cfg['shape']['size']['z'])])}"
                     scope="parent"/>
-    <!--
-    The property 'mesh' is local to this macro, so no need to use scope="parent". This property is used to set
-    another property in the parent scope, which is '${prop_prefix}_mesh'.
-    -->
-    <xacro:property name="mesh_dir" value="$(find eut_robotics_description)/meshes"/>
-    <xacro:property name="${prop_prefix}_mesh_visual"
-                    value="${mesh_dir + '/' + desc_cfg['mesh_visual'] if desc_cfg['mesh_visual'] else ''}"
-                    scope="parent"/>
+    <xacro:property name="_lidar_mesh_visual"    value="${desc_cfg.get('mesh_visual', '')}"/>
+    <xacro:property name="_lidar_mesh_collision" value="${desc_cfg.get('mesh_collision', '')}"/>
+    <xacro:if value="${_lidar_mesh_visual is not None and _lidar_mesh_visual != ''}">
+      <xacro:property name="${prop_prefix}_mesh_visual"
+                      value="${_lidar_mesh_visual}"
+                      scope="parent"/>
+    </xacro:if>
+    <xacro:if value="${_lidar_mesh_visual is None or _lidar_mesh_visual == ''}">
+      <xacro:property name="${prop_prefix}_mesh_visual"
+                      value=""
+                      scope="parent"/>
+    </xacro:if>
     <xacro:property name="${prop_prefix}_mesh_visual_has_color"
                     value="${desc_cfg['mesh_visual_has_color']}"
                     scope="parent"/>
-    <xacro:property name="${prop_prefix}_mesh_collision"
-                    value="${mesh_dir + '/' + desc_cfg['mesh_collision'] if desc_cfg['mesh_collision'] else ''}"
+    <xacro:property name="_lidar_color" value="${desc_cfg['color']}"/>
+    <xacro:property name="${prop_prefix}_color"
+                    value="${_lidar_color['r']} ${_lidar_color['g']} ${_lidar_color['b']} ${_lidar_color['a']}"
                     scope="parent"/>
-    <!--
-    To be able to do the comparion and the assignment of the resulting string in a single line, being the string
-    a concatenation of several values, you have to combine those values in a list, and then use 'join' to create the
-    string.
-    -->
+    <xacro:if value="${_lidar_mesh_collision is not None and _lidar_mesh_collision != ''}">
+      <xacro:property name="${prop_prefix}_mesh_collision"
+                      value="${_lidar_mesh_collision}"
+                      scope="parent"/>
+    </xacro:if>
+    <xacro:unless value="${_lidar_mesh_collision is None or _lidar_mesh_collision == ''}">
+      <xacro:property name="${prop_prefix}_mesh_collision"
+                      value=""
+                      scope="parent"/>
+    </xacro:unless>
+    <xacro:property name="_lidar_scale" value="${desc_cfg['scale']}"/>
     <xacro:property name="${prop_prefix}_scale"
-                    value="${' '.join([str(desc_cfg['scale']['x']),
-                                       str(desc_cfg['scale']['y']),
-                                       str(desc_cfg['scale']['z'])])
-                            if desc_cfg['scale'] else ''}"
-                    scope="parent"/>
-    <xacro:property name="${prop_prefix}_color"
-                    value="${' '.join([str(desc_cfg['color']['r']),
-                                       str(desc_cfg['color']['g']),
-                                       str(desc_cfg['color']['b']),
-                                       str(desc_cfg['color']['a'])])}"
+                    value="${_lidar_scale['x']} ${_lidar_scale['y']} ${_lidar_scale['z']}"
                     scope="parent"/>
     <xacro:property name="${prop_prefix}_joint_root_fr_data_fr"
