Commit message: Changed the way robot_prefix is created

File: urdf/robots/flart/description.xacro (robot description, xacro)
@@ -31,10 +31,9 @@
   <xacro:arg name="use_front_imu_sim"    default="True"/>
   <!-- args into properties for easy manipulation -->
-  <xacro:property name="robname"              value="$(arg robot_name)"/>
-  <xacro:property name="ns"                   value="$(arg namespace)"/>
+  <xacro:property name="robname" value="$(arg robot_name)"/>
+  <xacro:property name="ns"      value="$(arg namespace)"/>
   <xacro:property name="robot_namespace"
                   value="${(ns + robname) if ns in ('', '/') else (ns.rstrip('/') + '/' + robname)}"/>
-  <xacro:property name="robot_prefix"
-                  value="${(robname + '_') if ns in ('', '/') else (ns.strip('/').replace('/', '_') + '_' + robname + '_')}"/>
+  <xacro:property name="robot_prefix" value="${robname + '_'}"/>
   <xacro:property name="use_visual_meshes"    value="$(arg use_visual_meshes)"/>
   <xacro:property name="use_collision_meshes" value="$(arg use_collision_meshes)"/>

Commit message: Adequate description.xacro to the new macros for body and wheel

File: urdf/robots/flart/description.xacro (robot description, xacro)
@@ -10,6 +10,8 @@
   <!-- INCLUDES -->
   <xacro:include filename="${urdf_dir}/common/all_commons.xacro"/>
-  <xacro:include filename="${urdf_dir}/bases/mecanum_r_base_macro.xacro"/>
-  <xacro:include filename="${urdf_dir}/bases/set_mecanum_r_base_props_macro.xacro"/>
+  <xacro:include filename="${urdf_dir}/bases/rectangular_body_macro.xacro"/>
+  <xacro:include filename="${urdf_dir}/bases/set_rectangular_body_props_macro.xacro"/>
+  <xacro:include filename="${urdf_dir}/wheels/wheel_macro.xacro"/>
+  <xacro:include filename="${urdf_dir}/wheels/set_wheel_props_macro.xacro"/>
   <xacro:include filename="${urdf_dir}/extras/fork_macro.xacro"/>
   <xacro:include filename="${urdf_dir}/extras/set_fork_props_macro.xacro"/>
@@ -22,4 +24,5 @@
   <!-- ===================================================================== -->
   <!-- ARGS -->
+  <!-- ===================================================================== -->
   <xacro:arg name="robot_name"           default="${desc_cfg['name']}"/>
   <xacro:arg name="namespace"            default=""/>
@@ -71,35 +74,134 @@
   <!-- MECANUM RECTANGULAR BASE -->
   <!-- ===================================================================== -->
-  <xacro:set_mecanum_r_base_props desc_cfg="${desc_cfg['mecanum_rectangular_base']}" prop_prefix="base"/>
-  <xacro:mecanum_r_base
-    base_name="base"
-    front_left_wheel_name="front_left_wheel"
-    front_right_wheel_name="front_right_wheel"
-    rear_left_wheel_name="rear_left_wheel"
-    rear_right_wheel_name="rear_right_wheel"
-    prefix="${robot_prefix}"
-    body_mass="${base_body_mass}"
-    body_size="${base_body_size}"
-    body_wheelbase="${base_body_wheelbase}"
-    body_track_width="${base_body_track_width}"
-    body_ground_clearance="${base_body_ground_clearance}"
-    body_mesh_visual="${base_body_mesh_visual if use_visual_meshes else ''}"
-    body_mesh_visual_has_color="${base_body_mesh_visual_has_color}"
-    body_mesh_collision="${base_body_mesh_collision if use_collision_meshes else ''}"
-    body_scale="${base_body_scale}"
-    body_color="${base_body_color}"
-    mecanum_wheel_mass="${base_mecanum_wheel_mass}"
-    mecanum_wheel_size="${base_mecanum_wheel_size}"
-    mecanum_wheel_velocity_limit="${base_mecanum_wheel_velocity_limit}"
-    mecanum_wheel_effort_limit="${base_mecanum_wheel_effort_limit}"
-    mecanum_wheel_mu_forward="${base_mecanum_wheel_mu_forward}"
-    mecanum_wheel_mu_lateral="${base_mecanum_wheel_mu_lateral}"
-    mecanum_wheel_slip_forward="${base_mecanum_wheel_slip_forward}"
-    mecanum_wheel_slip_lateral="${base_mecanum_wheel_slip_lateral}"
-    mecanum_wheel_mesh_visual_left="${base_mecanum_wheel_mesh_visual_left if use_visual_meshes else ''}"
-    mecanum_wheel_mesh_visual_right="${base_mecanum_wheel_mesh_visual_right if use_visual_meshes else ''}"
-    mecanum_wheel_mesh_visual_has_color="${base_mecanum_wheel_mesh_visual_has_color}"
-    mecanum_wheel_scale="${base_mecanum_wheel_scale}"
-    mecanum_wheel_color="${base_mecanum_wheel_color}"/>
+  <!--
+  A base is composed of a body and wheels.
+  In this case, the base is rectangular with mecanum wheels.
+  The rectangular_body macro defines the following links and joints:
+  - Links:
+    * ${prefix}${name}_footprint_link = ${robot_prefix}${base_name}_footprint_link
+    * ${prefix}${name}_link = ${robot_prefix}${base_name}_link
+  - Joints:
+    * ${prefix}${name}_joint = ${robot_prefix}${base_name}_joint, joining the links
+      ${robot_prefix}${base_name}_footprint_link and ${robot_prefix}${base_name}_link.
+  THE LINK '${robot_prefix}${base_name}_link' IS LOCATED AT THE CENTER OF THE BOTTOM FACE OF THE BASE BODY.
+  THE LINK '${robot_prefix}${base_name}_footprint_link' IS LOCATED ON THE GROUND, JUST BELOW THE LINK
+  '${robot_prefix}${base_name}_link'.
+  ANOTHER WAY TO SEE IS, THE LINK '${robot_prefix}${base_name}_footprint_link' IS LOCATED ON THE GROUND, AND THE LINK
+  '${robot_prefix}${base_name}_link' IS JUST OVER IT, AT A HEIGHT OF 'GROUND_CLEARANCE' METERS.
+  -->
+  <xacro:property name="base_name"              value="base"/>
+  <xacro:property name="front_left_wheel_name"  value="front_left_wheel"/>  <!-- flw -->
+  <xacro:property name="front_right_wheel_name" value="front_right_wheel"/> <!-- frw -->
+  <xacro:property name="rear_left_wheel_name"   value="rear_left_wheel"/>   <!-- rlw -->
+  <xacro:property name="rear_right_wheel_name"  value="rear_right_wheel"/>  <!-- rrw -->
+  <xacro:set_rectangular_body_props desc_cfg="${desc_cfg['base']['body']}" prop_prefix="base_body"/>
+  <xacro:property name="base_body_half_wheelbase"   value="${0.5 * base_body_wheelbase}"/>
+  <xacro:property name="base_body_half_track_width" value="${0.5 * base_body_track_width}"/>
+  <xacro:rectangular_body
+    name="${base_name}"
+    prefix="${robot_prefix}"
+    mass="${base_body_mass}"
+    size="${base_body_size_x} ${base_body_size_y} ${base_body_size_z}"
+    ground_clearance="${base_body_ground_clearance}"
+    mesh_visual="${base_body_mesh_visual if use_visual_meshes else ''}"
+    mesh_visual_has_color="${base_body_mesh_visual_has_color}"
+    color="${base_body_color}"
+    mesh_collision="${base_body_mesh_collision if use_collision_meshes else ''}"
+    scale="${base_body_scale}"/>
+  <!--
+  Definition of the four mecanum wheels.
+  -->
+  <xacro:set_wheel_props desc_cfg="${desc_cfg['base']['wheel']}" prop_prefix="wheel"/>
+  <!--
+  The front left and the rear right mecanum wheels are of the same type, left type.
+  The front right and the rear left mecanum wheels are of the same type, right type.
+  The left and right meshes for the same mecanum wheel model are supposed to be called '<side>_xxx.stl'
+  where {{side}} is either 'left' or 'right', and 'xxx' is the rest of the file name.
+  Therefore, in the property '${prop_prefix}_mesh_visual', we could have and empty value (no mesh) or a value like
+  '/path/to/meshes/{{side}}_<whatever>'.ext'
+  Next, we get the left and right mesh names by replacing {{side}} with 'left' and 'right', respectively, if a non-empty
+  mesh name is provided. If no mesh name is provided, the left and right mesh names are also empty.
+  -->
+  <xacro:property name="wheel_mesh_visual_left"
+                  value="${wheel_mesh_visual.replace('[side]', 'left') if wheel_mesh_visual else ''}"/>
+  <xacro:property name="wheel_mesh_visual_right"
+                  value="${wheel_mesh_visual.replace('[side]', 'right') if wheel_mesh_visual else ''}"/>
+  <xacro:property name="z_wheel" value="${-base_body_ground_clearance + wheel_radius}"/>
+  <xacro:wheel
+    name="${front_left_wheel_name}"
+    prefix="${robot_prefix}"
+    parent_frame="${robot_prefix}${base_name}_link"
+    mass="${wheel_mass}"
+    shape="${wheel_shape}"
+    velocity_limit="${wheel_velocity_limit}"
+    effort_limit="${wheel_effort_limit}"
+    mu="${wheel_mu}"
+    mu2="${wheel_mu2}"
+    slip1="${wheel_slip1}"
+    slip2="${wheel_slip2}"
+    mesh_visual="${wheel_mesh_visual_left}"
+    mesh_visual_has_color="${wheel_mesh_visual_has_color}"
+    color="${wheel_color}"
+    scale="${wheel_scale}"
+    joint_parent_fr_wheel_fr="${base_body_half_wheelbase} ${base_body_half_track_width} ${z_wheel} 0 0 0"
+    base_root_fr="${robot_prefix}${base_name}_footprint_link"
+    fdir1_base_root_fr="${cos(radians(45))} ${sin(radians(45))} 0"/>
+  <xacro:wheel
+    name="${front_right_wheel_name}"
+    prefix="${robot_prefix}"
+    parent_frame="${robot_prefix}${base_name}_link"
+    mass="${wheel_mass}"
+    shape="${wheel_shape}"
+    velocity_limit="${wheel_velocity_limit}"
+    effort_limit="${wheel_effort_limit}"
+    mu="${wheel_mu}"
+    mu2="${wheel_mu2}"
+    slip1="${wheel_slip1}"
+    slip2="${wheel_slip2}"
+    mesh_visual="${wheel_mesh_visual_right}"
+    mesh_visual_has_color="${wheel_mesh_visual_has_color}"
+    color="${wheel_color}"
+    scale="${wheel_scale}"
+    joint_parent_fr_wheel_fr="${base_body_half_wheelbase} ${-base_body_half_track_width} ${z_wheel} 0 0 0"
+    base_root_fr="${robot_prefix}${base_name}_footprint_link"
+    fdir1_base_root_fr="${-cos(radians(45))} ${sin(radians(45))} 0"/>
+  <xacro:wheel
+    name="${rear_left_wheel_name}"
+    prefix="${robot_prefix}"
+    parent_frame="${robot_prefix}${base_name}_link"
+    mass="${wheel_mass}"
+    shape="${wheel_shape}"
+    velocity_limit="${wheel_velocity_limit}"
+    effort_limit="${wheel_effort_limit}"
+    mu="${wheel_mu}"
+    mu2="${wheel_mu2}"
+    slip1="${wheel_slip1}"
+    slip2="${wheel_slip2}"
+    mesh_visual="${wheel_mesh_visual_right}"
+    mesh_visual_has_color="${wheel_mesh_visual_has_color}"
+    color="${wheel_color}"
+    scale="${wheel_scale}"
+    joint_parent_fr_wheel_fr="${-base_body_half_wheelbase} ${base_body_half_track_width} ${z_wheel} 0 0 0"
+    base_root_fr="${robot_prefix}${base_name}_footprint_link"
+    fdir1_base_root_fr="${-cos(radians(45))} ${sin(radians(45))} 0"/>
+  <xacro:wheel
+    name="${rear_right_wheel_name}"
+    prefix="${robot_prefix}"
+    parent_frame="${robot_prefix}${base_name}_link"
+    mass="${wheel_mass}"
+    shape="${wheel_shape}"
+    velocity_limit="${wheel_velocity_limit}"
+    effort_limit="${wheel_effort_limit}"
+    mu="${wheel_mu}"
+    mu2="${wheel_mu2}"
+    slip1="${wheel_slip1}"
+    slip2="${wheel_slip2}"
+    mesh_visual="${wheel_mesh_visual_left}"
+    mesh_visual_has_color="${wheel_mesh_visual_has_color}"
+    color="${wheel_color}"
+    scale="${wheel_scale}"
+    joint_parent_fr_wheel_fr="${-base_body_half_wheelbase} ${-base_body_half_track_width} ${z_wheel} 0 0 0"
+    base_root_fr="${robot_prefix}${base_name}_footprint_link"
+    fdir1_base_root_fr="${cos(radians(45))} ${sin(radians(45))} 0"/>
   <!-- ===================================================================== -->
   <!-- FORK -->

Commit message: Added max_contacts field to the wheel.
With this new input field we can configure the max_contacts tag under the gazebo tag

File: urdf/robots/flart/description.xacro (robot description, xacro)
@@ -136,4 +136,5 @@
     velocity_limit="${wheel_velocity_limit}"
     effort_limit="${wheel_effort_limit}"
+    max_contacts="${wheel_max_contacts}"
     mu="${wheel_mu}"
     mu2="${wheel_mu2}"
@@ -155,4 +156,5 @@
     velocity_limit="${wheel_velocity_limit}"
     effort_limit="${wheel_effort_limit}"
+    max_contacts="${wheel_max_contacts}"
     mu="${wheel_mu}"
     mu2="${wheel_mu2}"
@@ -174,4 +176,5 @@
     velocity_limit="${wheel_velocity_limit}"
     effort_limit="${wheel_effort_limit}"
+    max_contacts="${wheel_max_contacts}"
     mu="${wheel_mu}"
     mu2="${wheel_mu2}"
@@ -193,4 +196,5 @@
     velocity_limit="${wheel_velocity_limit}"
     effort_limit="${wheel_effort_limit}"
+    max_contacts="${wheel_max_contacts}"
     mu="${wheel_mu}"
     mu2="${wheel_mu2}"

File: urdf/wheels/set_wheel_props_macro.xacro (robot description, xacro)
@@ -42,4 +42,5 @@
     <xacro:property name="${prop_prefix}_velocity_limit" value="${desc_cfg['velocity_limit']}" scope="parent"/>
     <xacro:property name="${prop_prefix}_effort_limit"   value="${desc_cfg['effort_limit']}"   scope="parent"/>
+    <xacro:property name="${prop_prefix}_max_contacts"   value="${desc_cfg.get('max_contacts', 10)}" scope="parent"/>
     <xacro:property name="${prop_prefix}_mu"             value="${desc_cfg['mu']}"             scope="parent"/>
     <xacro:property name="${prop_prefix}_mu2"            value="${desc_cfg['mu2']}"            scope="parent"/>

File: urdf/wheels/wheel_macro.xacro (robot description, xacro)
@@ -19,4 +19,5 @@
                        velocity_limit:=100
                        effort_limit:=100000
+                       max_contacts:=3
                        mu:=1.0
                        mu2:=0.05
@@ -114,5 +115,5 @@
     </joint>
     <gazebo reference="${prefix}${name}_link">
-      <max_contacts>2</max_contacts> <!-- Default is 10 -->
+      <max_contacts>${max_contacts}</max_contacts> <!-- Default is 10 -->
       <collision>
         <surface>

Commit message: Removed fields use_front_lidar and use_front_imu
Use field 'enabled' in the simulation configuration field for front_lidar and front_imu.

File: urdf/robots/flart/description.xacro (robot description, xacro)
@@ -31,6 +31,7 @@
   <xacro:arg name="use_sim_mode"         default="False"/>
   <xacro:arg name="sim_cfg_file"         default=""/>
-  <xacro:arg name="use_front_lidar_sim"  default="True"/>
-  <xacro:arg name="use_front_imu_sim"    default="True"/>
+  <!--
+  Create properties from args for easy manipulation.
+  -->
   <!-- args into properties for easy manipulation -->
   <xacro:property name="robname" value="$(arg robot_name)"/>
@@ -49,9 +50,11 @@
   -->
   <xacro:property name="sim_cfg_file" value="$(arg sim_cfg_file)"/>
-  <xacro:property name="sim_cfg"
-                  value="${xacro.load_yaml(sim_cfg_file)
-                           if use_sim_mode and sim_cfg_file else dict()}"/>
-  <xacro:property name="use_front_lidar_sim" value="$(arg use_front_lidar_sim)"/>
-  <xacro:property name="use_front_imu_sim"   value="$(arg use_front_imu_sim)"/>
+  <!--
+  If the 'use_sim_mode' argument is True, then the 'sim_cfg_file' argument is required (non-empty).
+  -->
+  <xacro:if value="${use_sim_mode and not sim_cfg_file}">
+    ${xacro.fatal("The argument 'sim_cfg_file' is empty while 'use_sim_mode' is set to True")}
+  </xacro:if>
+  <xacro:property name="sim_cfg" value="${xacro.load_yaml(sim_cfg_file) if use_sim_mode else dict()}"/>
   <!-- ===================================================================== -->
   <!-- ROBOT -->
@@ -285,4 +288,5 @@
   <xacro:property name="joint_base_fr_front_lidar_fr_x"
                   value="${(0.5 * base_body_size_x) + (0.5 * front_lidar_cfg['shape']['size']['x']) - 0.028}"/>
+  <xacro:property name="front_lidar_sim_cfg" value="${sim_cfg.get('front_lidar', dict()) if use_sim_mode else dict()}"/>
   <xacro:robosense_helios_16p
     name="front_lidar"
@@ -291,5 +295,5 @@
     parent_frame="${robot_prefix}base_link"
     joint_parent_fr_root_fr="${joint_base_fr_front_lidar_fr_x} 0 0.28 0 0 0"
-    sim_cfg="${sim_cfg.get('front_lidar') if use_sim_mode and sim_cfg and use_front_lidar_sim else None}"
+    sim_cfg="${front_lidar_sim_cfg if front_lidar_sim_cfg.get('enabled', False) else None}"
     use_mesh_visual="${use_visual_meshes}"
     use_mesh_collision="${use_collision_meshes}"/>
@@ -307,4 +311,5 @@
   <xacro:property name="joint_front_lidar_fr_front_imu_fr"
                   value="0 0 ${front_lidar_cfg['shape']['size']['z']} 0 0 0"/>
+  <xacro:property name="front_imu_sim_cfg" value="${sim_cfg.get('front_imu', dict()) if use_sim_mode else dict()}"/>
   <xacro:um7
     name="front_imu"
@@ -313,8 +318,9 @@
     parent_frame="${robot_prefix}front_lidar_root_link"
     joint_parent_fr_root_fr="${joint_front_lidar_fr_front_imu_fr}"
-    sim_cfg="${sim_cfg.get('front_imu') if use_sim_mode and sim_cfg and use_front_imu_sim else None}"
+    sim_cfg="${front_imu_sim_cfg if front_imu_sim_cfg.get('enabled', False) else None}"
     use_mesh_visual="${use_visual_meshes}"
     use_mesh_collision="${use_collision_meshes}"/>
   <xacro:if value="${use_sim_mode}">
+    <!--
     <xacro:include filename="${urdf_dir}/robots/flart/ros2_control_sim.xacro"/>
     <xacro:r2c namespace="${robot_namespace}"

Commit message: Include odom_frame field in the application

File: urdf/robots/flart/description.xacro (robot description, xacro)
@@ -27,4 +27,8 @@
   <xacro:arg name="robot_name"           default="${desc_cfg['name']}"/>
   <xacro:arg name="namespace"            default=""/>
+  <!--
+  Note that robot_prefix, defined below, will be appended to the odom_frame name.
+  -->
+  <xacro:arg name="odom_frame"           default="odom"/>
   <xacro:arg name="use_visual_meshes"    default="True"/>
   <xacro:arg name="use_collision_meshes" default="False"/>
@@ -40,4 +44,5 @@
                   value="${(ns + robname) if ns in ('', '/') else (ns.rstrip('/') + '/' + robname)}"/>
   <xacro:property name="robot_prefix" value="${robname + '_'}"/>
+  <xacro:property name="odom_frame"           value="$(arg odom_frame)"/>
   <xacro:property name="use_visual_meshes"    value="$(arg use_visual_meshes)"/>
   <xacro:property name="use_collision_meshes" value="$(arg use_collision_meshes)"/>
