Commit message: Added plugins gz::sim::systems::VelocityControl and gz::sim::systems::OdometryPublisher into the flart robot

File: urdf/robots/flart/description.xacro (robot description, xacro)
@@ -335,4 +335,104 @@
                rear_left_wheel_joint_name="${robot_prefix}rear_left_wheel_joint"
                rear_right_wheel_joint_name="${robot_prefix}rear_right_wheel_joint"/>
+  -->
+    <xacro:property name="velocity_control_sim_cfg"
+                    value="${sim_cfg.get('gz_sim_systems_VelocityControl', dict())}"/>
+    <xacro:property name="odometry_publisher_sim_cfg"
+                    value="${sim_cfg.get('gz_sim_systems_OdometryPublisher', dict())}"/>
+    <gazebo>
+      <!--
+      Reference for system plugins:
+      https://gazebosim.org/api/gazebo/6/namespaceignition_1_1gazebo_1_1systems.html
+      -->
+      <xacro:if value="${velocity_control_sim_cfg.get('enabled', False)}">
+        <xacro:property name="initial_linear"
+                        value="${velocity_control_sim_cfg.get('initial_linear', dict(x=0, y=0, z=0))}"/>
+        <xacro:property name="initial_angular"
+                        value="${velocity_control_sim_cfg.get('initial_angular', dict(x=0, y=0, z=0))}"/>
+        <!--
+        Reference: https://gazebosim.org/api/gazebo/6/classignition_1_1gazebo_1_1systems_1_1VelocityControl.html
+        Linear and angular velocity controller which is directly set on a model.
+        -->
+        <plugin filename="gz-sim-velocity-control-system" name="gz::sim::systems::VelocityControl">
+          <topic>${robot_namespace}/cmd_vel</topic>
+          <initial_linear>${initial_linear['x']} ${initial_linear['y']} ${initial_linear['z']}</initial_linear>
+          <initial_angular>${initial_angular['x']} ${initial_angular['y']} ${initial_angular['z']}</initial_angular>
+        </plugin>
+      </xacro:if>
+      <xacro:if value="${odometry_publisher_sim_cfg.get('enabled', False)}">
+        <!--
+        Reference: https://gazebosim.org/api/gazebo/6/classignition_1_1gazebo_1_1systems_1_1OdometryPublisher.html
+        This plugin publishes the absolute pose (position and orientation) and velocities of the robot with respect to
+        Gazebo's world frame.
+        Strictly speaking, odometry is the pose (and some might consider velocities as well) of the robot with respect
+        to its starting pose.
+        Global localization, on the other hand, is the pose (again, some might consider velocities as well) of the robot
+        with respect to a fixed global frame, considered the root frame for the application.
+        The root frame for the application is usually called 'map' or 'world', and the odometry frame is usually called
+        'odom'.
+        Each robot has its own odometry frame in an application, while there is usually a single global frame for the
+        application.
+        The whole point of the explanation above is to let the reader now that although the plugin is called
+        'OdometryPublisher', it is in fact a source of global localization for the robot, with respect to Gazebo's world
+        frame.
+        Therefore, the plugin 'OdometryPublisher' is providing the transformation 'T_world_fr_robot_root_fr', where
+        the term 'robot_root_fr' is the generic expression to describe the frame that acts as the root frame for the
+        robot, in this file, '${robot_prefix}base_footprint_link', but in other robots it could be
+        '${robot_prefix}base_link' or any other name.
+        Therefore, in the application where this xacro file is used, it is needed to compute the transformations
+        'T_odom_fr_robot_root_frame' and transformation 'T_world_fr_odom_fr'.
+        The transformation 'T_odom_fr_robot_root_fr' can be computed, for example, by integrating the velocities
+        of the robot in the odometry frame, or using an Extended Kalman Filter (EKF) or a similar method.
+        The relation between these three transformations is:
+        T_world_fr_robot_root_fr = T_world_fr_odom_fr * T_odom_fr_robot_root_fr
+              ^                       ^                          ^
+        provided by the plugin     derived                  this is computed
+        T_world_fr_odom_fr = T_world_fr_robot_root_fr * inv(T_odom_fr_robot_root_fr)
+        When in simulation, the transformation 'T_world_fr_odom_fr' can be computed by the node in the package
+        'eut_fake_localization', and the transformation 'T_odom_fr_robot_root_fr' can be computed by the
+        'eut_ground_vehicle_twist_odometry' node, for example.
+        -->
+        <xacro:property name="odom_publish_frequency"
+                        value="${odometry_publisher_sim_cfg.get('odom_publish_frequency', 50)}"/>
+        <xacro:property name="offset"
+                        value="${odometry_publisher_sim_cfg.get('offset', dict(x=0, y=0, z=0, R=0, P=0, Y=0))}"/>
+        <xacro:property name="gaussian_noise"
+                        value="${odometry_publisher_sim_cfg.get('gaussian_noise', 0)}"/>
+        <plugin filename="gz-sim-odometry-publisher-system" name="gz::sim::systems::OdometryPublisher">
+          <odom_frame>${robot_prefix}${odom_frame}</odom_frame>
+          <robot_base_frame>${robot_prefix}${base_name}_footprint_link</robot_base_frame>
+          <odom_publish_frequency>${odom_publish_frequency}</odom_publish_frequency>
+          <!--
+          Custom topic on which this system will publish odometry messages.
+          We use the odom_covariance_topic to publish the odometry with covariance messages.
+          <odom_topic>...</odom_topic>
+          -->
+          <!--
+          Custom topic on which this system will publish odometry with covariance messages.
+          -->
+          <odom_covariance_topic>${robot_namespace}/odom</odom_covariance_topic>
+          <!--
+          Custom topic on which this system will publish the transform from odom_frame to robot_base_frame.
+          -->
+          <tf_topic>/tf</tf_topic>
+          <dimensions>2</dimensions> <!-- 2D (x, y, yaw) -->
+          <!--
+          Position offset relative to the body fixed frame, the default value is 0 0 0.
+          This offset will be added to the odometry message.
+          -->
+          <xyz_offset>${offset['x']} ${offset['y']} ${offset['z']}</xyz_offset>
+          <!--
+          Rotation offset relative to the body fixed frame, the default value is 0 0 0.
+          This offset will be added to the odometry message.
+          -->
+          <rpy_offset>${offset['R']} ${offset['P']} ${offset['Y']}</rpy_offset>
+          <!--
+          Standard deviation of the Gaussian noise to be added to pose and twist messages.
+          This element is optional, and the default value is 0.
+          -->
+          <gaussian_noise>${gaussian_noise}</gaussian_noise>
+        </plugin>
+      </xacro:if>
+    </gazebo>
   </xacro:if>
 </robot>

Commit message: Substitute 4 mecanum wheels with 3 motowheels
One in the front, 2 at the back.
By now, they use fixed joints.

File: urdf/robots/flart/description.xacro (robot description, xacro)
@@ -65,15 +65,4 @@
   <!-- ROBOT -->
   <!-- ===================================================================== -->
-  <!--
-  Names used in this robot for devices/parts:
-  - base
-  - front_left_wheel
-  - front_right_wheel
-  - rear_left_wheel
-  - rear_right_wheel
-  - fork
-  - front_lidar
-  - front_imu
-  -->
   <xacro:property name="robot_size_x" value="${desc_cfg['size']['x']}"/>
   <xacro:property name="robot_size_y" value="${desc_cfg['size']['y']}"/>
@@ -102,6 +91,5 @@
   -->
   <xacro:property name="base_name"              value="base"/>
-  <xacro:property name="front_left_wheel_name"  value="front_left_wheel"/>  <!-- flw -->
-  <xacro:property name="front_right_wheel_name" value="front_right_wheel"/> <!-- frw -->
+  <xacro:property name="front_wheel_name"       value="front_wheel"/>       <!-- fw -->
   <xacro:property name="rear_left_wheel_name"   value="rear_left_wheel"/>   <!-- rlw -->
   <xacro:property name="rear_right_wheel_name"  value="rear_right_wheel"/>  <!-- rrw -->
@@ -123,28 +111,26 @@
     scale="${base_body_scale}"/>
   <!--
-  Definition of the four mecanum wheels.
-  -->
+  Definition of the wheel blocks:
+  wheel_block = rotation_gear + wheel
+  Front and rear wheels can rotate, so this way the omnidirectional motion is achieved.
+  -->
+  <link name="${robot_prefix}${front_wheel_name}_gear_link">
+    <xacro:null_inertia/>
+  </link>
+  <xacro:property name="z_wheel_gear" value="0.278"/>
+  <joint name="${robot_prefix}${front_wheel_name}_gear_joint" type="fixed">
+    <parent link="${robot_prefix}${base_name}_link"/>
+    <child link="${robot_prefix}${front_wheel_name}_gear_link"/>
+    <origin rpy="0 0 0" xyz="${base_body_half_wheelbase} 0 ${z_wheel_gear}"/>
+  </joint>
   <xacro:set_wheel_props desc_cfg="${desc_cfg['base']['wheel']}" prop_prefix="wheel"/>
-  <!--
-  The front left and the rear right mecanum wheels are of the same type, left type.
-  The front right and the rear left mecanum wheels are of the same type, right type.
-  The left and right meshes for the same mecanum wheel model are supposed to be called '<side>_xxx.stl'
-  where {{side}} is either 'left' or 'right', and 'xxx' is the rest of the file name.
-  Therefore, in the property '${prop_prefix}_mesh_visual', we could have and empty value (no mesh) or a value like
-  '/path/to/meshes/{{side}}_<whatever>'.ext'
-  Next, we get the left and right mesh names by replacing {{side}} with 'left' and 'right', respectively, if a non-empty
-  mesh name is provided. If no mesh name is provided, the left and right mesh names are also empty.
-  -->
-  <xacro:property name="wheel_mesh_visual_left"
-                  value="${wheel_mesh_visual.replace('[side]', 'left') if wheel_mesh_visual else ''}"/>
-  <xacro:property name="wheel_mesh_visual_right"
-                  value="${wheel_mesh_visual.replace('[side]', 'right') if wheel_mesh_visual else ''}"/>
-  <xacro:property name="z_wheel" value="${-base_body_ground_clearance + wheel_radius}"/>
+  <xacro:property name="z_wheel" value="${-z_wheel_gear - base_body_ground_clearance + wheel_radius}"/>
   <xacro:wheel
-    name="${front_left_wheel_name}"
-    prefix="${robot_prefix}"
-    parent_frame="${robot_prefix}${base_name}_link"
+    name="${front_wheel_name}"
+    prefix="${robot_prefix}"
+    parent_frame="${robot_prefix}${front_wheel_name}_gear_link"
     mass="${wheel_mass}"
     shape="${wheel_shape}"
+    joint_type="${wheel_joint_type}"
     velocity_limit="${wheel_velocity_limit}"
     effort_limit="${wheel_effort_limit}"
@@ -154,17 +140,26 @@
     slip1="${wheel_slip1}"
     slip2="${wheel_slip2}"
-    mesh_visual="${wheel_mesh_visual_left}"
+    mesh_visual="${wheel_mesh_visual}"
     mesh_visual_has_color="${wheel_mesh_visual_has_color}"
     color="${wheel_color}"
     scale="${wheel_scale}"
-    joint_parent_fr_wheel_fr="${base_body_half_wheelbase} ${base_body_half_track_width} ${z_wheel} 0 0 0"
-    base_root_fr="${robot_prefix}${base_name}_footprint_link"
-    fdir1_base_root_fr="${cos(radians(45))} ${sin(radians(45))} 0"/>
+    joint_parent_fr_wheel_fr="0 0 ${z_wheel} 0 0 0"
+    fdir1_fr="${robot_prefix}${front_wheel_name}_gear_link"
+    fdir1="1 0 0"/>
+  <link name="${robot_prefix}${rear_left_wheel_name}_gear_link">
+    <xacro:null_inertia/>
+  </link>
+  <joint name="${robot_prefix}${rear_left_wheel_name}_gear_joint" type="fixed">
+    <parent link="${robot_prefix}${base_name}_link"/>
+    <child link="${robot_prefix}${rear_left_wheel_name}_gear_link"/>
+    <origin rpy="0 0 0" xyz="${-base_body_half_wheelbase} ${base_body_half_track_width} ${z_wheel_gear}"/>
+  </joint>
   <xacro:wheel
-    name="${front_right_wheel_name}"
-    prefix="${robot_prefix}"
-    parent_frame="${robot_prefix}${base_name}_link"
+    name="${rear_left_wheel_name}"
+    prefix="${robot_prefix}"
+    parent_frame="${robot_prefix}${rear_left_wheel_name}_gear_link"
     mass="${wheel_mass}"
     shape="${wheel_shape}"
+    joint_type="${wheel_joint_type}"
     velocity_limit="${wheel_velocity_limit}"
     effort_limit="${wheel_effort_limit}"
@@ -174,17 +169,26 @@
     slip1="${wheel_slip1}"
     slip2="${wheel_slip2}"
-    mesh_visual="${wheel_mesh_visual_right}"
+    mesh_visual="${wheel_mesh_visual}"
     mesh_visual_has_color="${wheel_mesh_visual_has_color}"
     color="${wheel_color}"
     scale="${wheel_scale}"
-    joint_parent_fr_wheel_fr="${base_body_half_wheelbase} ${-base_body_half_track_width} ${z_wheel} 0 0 0"
-    base_root_fr="${robot_prefix}${base_name}_footprint_link"
-    fdir1_base_root_fr="${-cos(radians(45))} ${sin(radians(45))} 0"/>
+    joint_parent_fr_wheel_fr="0 0 ${z_wheel} 0 0 0"
+    fdir1_fr="${robot_prefix}${rear_left_wheel_name}_gear_link"
+    fdir1="1 0 0"/>
+  <link name="${robot_prefix}${rear_right_wheel_name}_gear_link">
+    <xacro:null_inertia/>
+  </link>
+  <joint name="${robot_prefix}${rear_right_wheel_name}_gear_joint" type="fixed">
+    <parent link="${robot_prefix}${base_name}_link"/>
+    <child link="${robot_prefix}${rear_right_wheel_name}_gear_link"/>
+    <origin rpy="0 0 0" xyz="${-base_body_half_wheelbase} ${-base_body_half_track_width} ${z_wheel_gear}"/>
+  </joint>
   <xacro:wheel
-    name="${rear_left_wheel_name}"
-    prefix="${robot_prefix}"
-    parent_frame="${robot_prefix}${base_name}_link"
+    name="${rear_right_wheel_name}"
+    prefix="${robot_prefix}"
+    parent_frame="${robot_prefix}${rear_right_wheel_name}_gear_link"
     mass="${wheel_mass}"
     shape="${wheel_shape}"
+    joint_type="${wheel_joint_type}"
     velocity_limit="${wheel_velocity_limit}"
     effort_limit="${wheel_effort_limit}"
@@ -194,31 +198,11 @@
     slip1="${wheel_slip1}"
     slip2="${wheel_slip2}"
-    mesh_visual="${wheel_mesh_visual_right}"
+    mesh_visual="${wheel_mesh_visual}"
     mesh_visual_has_color="${wheel_mesh_visual_has_color}"
     color="${wheel_color}"
     scale="${wheel_scale}"
-    joint_parent_fr_wheel_fr="${-base_body_half_wheelbase} ${base_body_half_track_width} ${z_wheel} 0 0 0"
-    base_root_fr="${robot_prefix}${base_name}_footprint_link"
-    fdir1_base_root_fr="${-cos(radians(45))} ${sin(radians(45))} 0"/>
-  <xacro:wheel
-    name="${rear_right_wheel_name}"
-    prefix="${robot_prefix}"
-    parent_frame="${robot_prefix}${base_name}_link"
-    mass="${wheel_mass}"
-    shape="${wheel_shape}"
-    velocity_limit="${wheel_velocity_limit}"
-    effort_limit="${wheel_effort_limit}"
-    max_contacts="${wheel_max_contacts}"
-    mu="${wheel_mu}"
-    mu2="${wheel_mu2}"
-    slip1="${wheel_slip1}"
-    slip2="${wheel_slip2}"
-    mesh_visual="${wheel_mesh_visual_left}"
-    mesh_visual_has_color="${wheel_mesh_visual_has_color}"
-    color="${wheel_color}"
-    scale="${wheel_scale}"
-    joint_parent_fr_wheel_fr="${-base_body_half_wheelbase} ${-base_body_half_track_width} ${z_wheel} 0 0 0"
-    base_root_fr="${robot_prefix}${base_name}_footprint_link"
-    fdir1_base_root_fr="${cos(radians(45))} ${sin(radians(45))} 0"/>
+    joint_parent_fr_wheel_fr="0 0 ${z_wheel} 0 0 0"
+    fdir1_fr="${robot_prefix}${rear_right_wheel_name}_gear_link"
+    fdir1="1 0 0"/>
   <!-- ===================================================================== -->
   <!-- FORK -->
@@ -420,5 +404,5 @@
           Custom topic on which this system will publish the transform from odom_frame to robot_base_frame.
           -->
-          <tf_topic>/tf</tf_topic>
+          <tf_topic>${robot_namespace}/tf_odom_fr_robot_root_fr</tf_topic>
           <dimensions>2</dimensions> <!-- 2D (x, y, yaw) -->
           <!--

Commit message: Added JointPositionController to the flart's description to control the fork

File: urdf/robots/flart/description.xacro (robot description, xacro)
@@ -113,5 +113,6 @@
   Definition of the wheel blocks:
   wheel_block = rotation_gear + wheel
-  Front and rear wheels can rotate, so this way the omnidirectional motion is achieved.
+  Front and rear wheels can rotate around an axis to get the proper orientation, so this way the omnidirectional motion
+  is achieved.
   -->
   <link name="${robot_prefix}${front_wheel_name}_gear_link">
@@ -315,4 +316,7 @@
     use_mesh_visual="${use_visual_meshes}"
     use_mesh_collision="${use_collision_meshes}"/>
+  <!--
+  The plugin 'gz_ros2_control' is not used.
+  -->
   <xacro:if value="${use_sim_mode}">
     <!--
@@ -324,9 +328,13 @@
                rear_left_wheel_joint_name="${robot_prefix}rear_left_wheel_joint"
                rear_right_wheel_joint_name="${robot_prefix}rear_right_wheel_joint"/>
-  -->
-    <xacro:property name="velocity_control_sim_cfg"
-                    value="${sim_cfg.get('gz_sim_systems_VelocityControl', dict())}"/>
-    <xacro:property name="odometry_publisher_sim_cfg"
-                    value="${sim_cfg.get('gz_sim_systems_OdometryPublisher', dict())}"/>
+    -->
+    <xacro:property name="base_vel_ctrl_sim_cfg"
+                    value="${sim_cfg.get('base_velocity_controller', dict())}"/>
+    <xacro:property name="base_odom_pub_sim_cfg"
+                    value="${sim_cfg.get('base_odometry_publisher', dict())}"/>
+    <xacro:property name="fork_pos_ctrl_sim_cfg"
+                    value="${sim_cfg.get('fork_position_controller', dict())}"/>
+    <xacro:property name="fork_pos_pub_sim_cfg"
+                    value="${sim_cfg.get('fork_position_publisher', dict())}"/>
     <gazebo>
       <!--
@@ -334,9 +342,13 @@
       https://gazebosim.org/api/gazebo/6/namespaceignition_1_1gazebo_1_1systems.html
       -->
-      <xacro:if value="${velocity_control_sim_cfg.get('enabled', False)}">
+      <!--
+      Plugin VelocityControl to control the robot's motion by publishing a twist message (command message) that
+      is subscribed by the plugin.
+      -->
+      <xacro:if value="${base_vel_ctrl_sim_cfg.get('enabled', False)}">
         <xacro:property name="initial_linear"
-                        value="${velocity_control_sim_cfg.get('initial_linear', dict(x=0, y=0, z=0))}"/>
+                        value="${base_vel_ctrl_sim_cfg.get('initial_linear', dict(x=0, y=0, z=0))}"/>
         <xacro:property name="initial_angular"
-                        value="${velocity_control_sim_cfg.get('initial_angular', dict(x=0, y=0, z=0))}"/>
+                        value="${base_vel_ctrl_sim_cfg.get('initial_angular', dict(x=0, y=0, z=0))}"/>
         <!--
         Reference: https://gazebosim.org/api/gazebo/6/classignition_1_1gazebo_1_1systems_1_1VelocityControl.html
@@ -349,5 +361,8 @@
         </plugin>
       </xacro:if>
-      <xacro:if value="${odometry_publisher_sim_cfg.get('enabled', False)}">
+      <!--
+      Plugin 'OdometryPublisher' to publish the robot's pose on the GZ's world frame.
+      -->
+      <xacro:if value="${base_odom_pub_sim_cfg.get('enabled', False)}">
         <!--
         Reference: https://gazebosim.org/api/gazebo/6/classignition_1_1gazebo_1_1systems_1_1OdometryPublisher.html
@@ -383,9 +398,9 @@
         -->
         <xacro:property name="odom_publish_frequency"
-                        value="${odometry_publisher_sim_cfg.get('odom_publish_frequency', 50)}"/>
+                        value="${base_odom_pub_sim_cfg.get('odom_publish_frequency', 50)}"/>
         <xacro:property name="offset"
-                        value="${odometry_publisher_sim_cfg.get('offset', dict(x=0, y=0, z=0, R=0, P=0, Y=0))}"/>
+                        value="${base_odom_pub_sim_cfg.get('offset', dict(x=0, y=0, z=0, R=0, P=0, Y=0))}"/>
         <xacro:property name="gaussian_noise"
-                        value="${odometry_publisher_sim_cfg.get('gaussian_noise', 0)}"/>
+                        value="${base_odom_pub_sim_cfg.get('gaussian_noise', 0)}"/>
         <plugin filename="gz-sim-odometry-publisher-system" name="gz::sim::systems::OdometryPublisher">
           <odom_frame>${robot_prefix}${odom_frame}</odom_frame>
@@ -421,4 +436,48 @@
           -->
           <gaussian_noise>${gaussian_noise}</gaussian_noise>
+        </plugin>
+      </xacro:if>
+      <xacro:if value="${fork_pos_ctrl_sim_cfg.get('enabled', False)}">
+        <!--
+        Reference: https://gazebosim.org/api/sim/8/classgz_1_1sim_1_1systems_1_1JointPositionController.html
+        -->
+        <plugin filename="gz-sim-joint-position-controller-system" name="gz::sim::systems::JointPositionController">
+          <joint_name>${robot_prefix}fork_root_joint</joint_name>
+          <joint_index>0</joint_index>
+          <!--
+          The following tags are NOT USED HERE, but are left commented for reference.
+          - <use_actuator_msg>: True to enable the use of actutor message for position command. Relies on
+          <actuator_number> for the index of the position actuator and defaults to topic "/actuators".
+          Used with <use_actuator_commands> to set the index of the position actuator.
+          - <actuator_number>
+          - <p_gain>: The proportional gain of the PID. Default value is 1.
+          - <i_gain>: The integral gain of the PID. Default value is 0.1.
+          - <d_gain>: The derivative gain of the PID. Default value is 0.001.
+          - <i_max>: The integral upper limit of the PID. Default value is 1.
+          - <i_min>: The integral lower limit of the PID. Default value is -1.
+          - <cmd_min>: The command minimum value of the PID. Default value is -1000.
+          - <cmd_offset>: Command offset (feed-forward) of the PID. Default value is 0.
+          -->
+          <!--
+          Bypasses the PID and creates a perfect position.
+          The maximum speed on the joint can be set using the <cmd_max> tag.
+          -->
+          <use_velocity_commands>true</use_velocity_commands>
+          <cmd_max>${fork_pos_ctrl_sim_cfg.get('v_max', 0.5)}</cmd_max>
+          <topic>${robot_namespace}/robot_description/fork_root_joint/cmd_pos</topic>
+          <!--
+          Initial position of a joint.
+          -->
+          <initial_position>0</initial_position>
+        </plugin>
+      </xacro:if>
+      <xacro:if value="${fork_pos_pub_sim_cfg.get('enabled', False)}">
+        <!--
+        Plugin 'JointStatePublisher' to publish the position of the fork joint.
+        Reference: https://gazebosim.org/api/sim/7/classgz_1_1sim_1_1systems_1_1JointStatePublisher.html#details
+        -->
+        <plugin filename="gz-sim-joint-state-publisher-system" name="gz::sim::systems::JointStatePublisher">
+          <topic>${robot_namespace}/robot_description/fork_root_joint/pos</topic>
+          <joint_name>flart1_fork_root_joint</joint_name>
         </plugin>
       </xacro:if>
