Commit message: Refactor lidar macros

File: urdf/sensors/lidars/all_lidars_macros.xacro (robot description, xacro)
@@ -1,4 +1,6 @@
 <?xml version="1.0"?>
 <robot name="all_lidars" xmlns:xacro="http://www.ros.org/wiki/xacro" xmlns:gz="http://gazebosim.org/schema">
+  <xacro:include filename="$(find eut_robotics_description)/urdf/sensors/lidars/generic_macros/set_props_plugin_lidar_2d_macro.xacro"/>
+  <xacro:include filename="$(find eut_robotics_description)/urdf/sensors/lidars/generic_macros/set_props_plugin_lidar_3d_ring_macro.xacro"/>
   <xacro:include filename="$(find eut_robotics_description)/urdf/sensors/lidars/robosense_airy_macro.xacro"/>
   <xacro:include filename="$(find eut_robotics_description)/urdf/sensors/lidars/robosense_helios_16p_macro.xacro"/>

File: urdf/sensors/lidars/generic_macros/plugin_lidar_2d_macro.xacro (robot description, xacro)
@@ -1,5 +1,5 @@
 <?xml version="1.0"?>
-<robot xmlns:xacro="http://ros.org/wiki/xacro" xmlns:gz="http://gazebosim.org/schema">
-  <xacro:macro name="lidar_2d_plugin"
+<robot name="plugin_lidar_2d" xmlns:xacro="http://www.ros.org/wiki/xacro" xmlns:gz="http://gazebosim.org/schema">
+  <xacro:macro name="plugin_lidar_2d"
                params="sensor_name
                        reference_link
@@ -14,7 +14,7 @@
     <!--
     According to the documentation at 'http://sdformat.org/spec?ver=1.7&elem=sensor#sensor_ray'
-    The 'ray' type is equivalent to 'lidar' type.
-    It is preferred to use 'lidar' since 'ray' will be deprecated at some point.
-    The 'ray' type is maintained for legacy support.
+    The 'gpu_ray' type is equivalent to the 'gpu_lidar' type.
+    It is preferred to use the 'gpu_lidar' type since 'gpu_ray' type will be deprecated at some point.
+    The 'gpu_ray' type is maintained for legacy support.
     -->
     <xacro:property name="hor_min_max_angles_deg" value="${hor_fov_deg.split()}"/>
@@ -37,5 +37,6 @@
         <topic>${topic}</topic>
         <!--
-        If the label <gz_frame_id> is not set, Gazebo will use as the 'frame_id' for the message the string '<model>::${parent_frame}::${laser_id}_link', which probably is not what you want.
+        If the label <gz_frame_id> is not set, Gazebo will use as the 'frame_id' for the message the string
+        '<model>::${parent_frame}::${laser_id}_link', which is probably what you do not want.
         -->
         <gz_frame_id>${reference_link}</gz_frame_id>

File: urdf/sensors/lidars/generic_macros/plugin_lidar_3d_ring_macro.xacro (robot description, xacro)
@@ -50,6 +50,6 @@
 - dist_span has 2 values between quotes in this order 'min_dist max_dist'
 -->
-<robot xmlns:xacro="http://ros.org/wiki/xacro" xmlns:gz="http://gazebosim.org/schema">
-  <xacro:macro name="lidar_3d_ring_plugin"
+<robot name="plugin_lidar_3d_ring" xmlns:xacro="http://www.ros.org/wiki/xacro" xmlns:gz="http://gazebosim.org/schema">
+  <xacro:macro name="plugin_lidar_3d_ring"
                params="sensor_name
                        reference_link
@@ -83,7 +83,7 @@
     <xacro:property name="min_dist"              value="${min_max_dists[0]}"/>
     <xacro:property name="max_dist"              value="${min_max_dists[1]}"/>
-    <xacro:property name="gaussian_noise_list"   value="${gaussian_noise.split()}"/>
-    <xacro:property name="gaussian_noise_mean"   value="${gaussian_noise_list[0]}"/>
-    <xacro:property name="gaussian_noise_stddev" value="${gaussian_noise_list[1]}"/>
+    <xacro:property name="gaussian_noise_seq"    value="${gaussian_noise.split()}"/>
+    <xacro:property name="gaussian_noise_mean"   value="${gaussian_noise_seq[0]}"/>
+    <xacro:property name="gaussian_noise_stddev" value="${gaussian_noise_seq[1]}"/>
     <gazebo reference="${reference_link}">
       <gravity>True</gravity>
