Commit message: Update realsense_d435.xacro

File: urdf/sensors/cameras/realsense_d435.xacro (robot description, xacro)
@@ -335,5 +335,5 @@
       <!-- camera color joints and links -->
       <link name="${prefix}${name}_color_frame"/>
-      <joint name="${name}_color_joint" type="fixed">
+      <joint name="${prefix}${name}_color_joint" type="fixed">
         <parent link="${prefix}${name}_link" />
         <child link="${prefix}${name}_color_frame" />
