Commit message: feat(sensors): [2105-14] Add gazebo visual materials
Add Gazebo material blocks for sensor and camera visuals when visual geometry is enabled, a color is configured, and the corresponding simulation plugin is active. This keeps RViz visual generation separate from Gazebo material coloring while avoiding material blocks for non-rendered links.

File: urdf/sensors/cameras/orbbec_gemini335le_rgbd_macro.xacro (robot description, xacro)
@@ -114,4 +114,12 @@
                                            c_mesh_use_low_res="${c_mesh_use_low_res}"
                                            joint_parent_fr_root_fr="${joint_parent_fr_root_fr}"/>
+    <xacro:if value="${use_visual and color != '' and (sim_rgbd_enabled or sim_left_ir_enabled or sim_right_ir_enabled or sim_imu_enabled)}">
+      <gazebo reference="${prefix}${name}_bottom_screw_frame">
+        <material>
+          <ambient>${color}</ambient>
+          <diffuse>${color}</diffuse>
+        </material>
+      </gazebo>
+    </xacro:if>
     <xacro:if value="${sim_rgbd_enabled}">
       <xacro:plugin_camera_rgbd name="${prefix}${name}_rgbd"

File: urdf/sensors/cameras/orbbec_gemini335le_split_macro.xacro (robot description, xacro)
@@ -137,4 +137,12 @@
                                            c_mesh_use_low_res="${c_mesh_use_low_res}"
                                            joint_parent_fr_root_fr="${joint_parent_fr_root_fr}"/>
+    <xacro:if value="${use_visual and color != '' and (sim_depth_enabled or sim_color_enabled or sim_left_ir_enabled or sim_right_ir_enabled or sim_imu_enabled)}">
+      <gazebo reference="${prefix}${name}_bottom_screw_frame">
+        <material>
+          <ambient>${color}</ambient>
+          <diffuse>${color}</diffuse>
+        </material>
+      </gazebo>
+    </xacro:if>
     <xacro:if value="${sim_depth_enabled}">
       <xacro:plugin_camera_depth name="${prefix}${name}_depth"

File: urdf/sensors/cameras/realsense_d435_rgbd_macro.xacro (robot description, xacro)
@@ -209,4 +209,12 @@
                                        use_sensor_frames_and_joints="${use_sensor_frames_and_joints}"
                                        joint_parent_fr_root_fr="${joint_parent_fr_root_fr}"/>
+    <xacro:if value="${use_visual and color != '' and (sim_rgbd_enabled or sim_infra1_enabled or sim_infra2_enabled)}">
+      <gazebo reference="${prefix}${name}_bottom_screw_frame">
+        <material>
+          <ambient>${color}</ambient>
+          <diffuse>${color}</diffuse>
+        </material>
+      </gazebo>
+    </xacro:if>
     <xacro:if value="${sim_rgbd_enabled and sim_rgbd_base_topic != ''}">
       <xacro:include filename="$(find robotics_description)/urdf/sensors/cameras/generic_macros/plugin_camera_rgbd_macro.xacro"/>

File: urdf/sensors/cameras/realsense_d435_split_macro.xacro (robot description, xacro)
@@ -240,4 +240,12 @@
                                        use_sensor_frames_and_joints="${use_sensor_frames_and_joints}"
                                        joint_parent_fr_root_fr="${joint_parent_fr_root_fr}"/>
+    <xacro:if value="${use_visual and color != '' and (sim_color_enabled or sim_depth_enabled or sim_infra1_enabled or sim_infra2_enabled)}">
+      <gazebo reference="${prefix}${name}_bottom_screw_frame">
+        <material>
+          <ambient>${color}</ambient>
+          <diffuse>${color}</diffuse>
+        </material>
+      </gazebo>
+    </xacro:if>
     <xacro:if value="${sim_depth_enabled}">
       <xacro:include filename="$(find robotics_description)/urdf/sensors/cameras/generic_macros/plugin_camera_depth_macro.xacro"/>

File: urdf/sensors/imus/box_imu_macro.xacro (robot description, xacro)
@@ -105,4 +105,12 @@
     </joint>
     <xacro:if value="${sim_enabled and sim_topic != ''}">
+      <xacro:if value="${use_visual and color != ''}">
+        <gazebo reference="${prefix}${name}_root_link">
+          <material>
+            <ambient>${color}</ambient>
+            <diffuse>${color}</diffuse>
+          </material>
+        </gazebo>
+      </xacro:if>
       <xacro:include filename="$(find robotics_description)/urdf/sensors/imus/generic_macros/plugin_imu_macro.xacro"/>
       <xacro:plugin_imu

File: urdf/sensors/lidars/hokuyo_utm30lx_macro.xacro (robot description, xacro)
@@ -177,4 +177,12 @@
     -->
     <xacro:if value="${sim_enabled and sim_topic != ''}">
+      <xacro:if value="${use_visual and color != ''}">
+        <gazebo reference="${prefix}${name}_root_link">
+          <material>
+            <ambient>${color}</ambient>
+            <diffuse>${color}</diffuse>
+          </material>
+        </gazebo>
+      </xacro:if>
       <xacro:include filename="$(find robotics_description)/urdf/sensors/lidars/generic_macros/plugin_lidar_2d_macro.xacro"/>
       <xacro:plugin_lidar_2d

File: urdf/sensors/lidars/leuze_rsl400_macro.xacro (robot description, xacro)
@@ -116,4 +116,12 @@
     -->
     <xacro:if value="${sim_enabled and sim_topic != ''}">
+      <xacro:if value="${use_visual and color != ''}">
+        <gazebo reference="${prefix}${name}_root_link">
+          <material>
+            <ambient>${color}</ambient>
+            <diffuse>${color}</diffuse>
+          </material>
+        </gazebo>
+      </xacro:if>
       <xacro:include filename="$(find robotics_description)/urdf/sensors/lidars/generic_macros/plugin_lidar_2d_macro.xacro"/>
       <xacro:plugin_lidar_2d

File: urdf/sensors/lidars/robosense_airy_macro.xacro (robot description, xacro)
@@ -254,4 +254,12 @@
     -->
     <xacro:if value="${sim_lidar_enabled and sim_lidar_base_topic != ''}">
+      <xacro:if value="${use_visual and color != ''}">
+        <gazebo reference="${prefix}${name}_root_link">
+          <material>
+            <ambient>${color}</ambient>
+            <diffuse>${color}</diffuse>
+          </material>
+        </gazebo>
+      </xacro:if>
       <xacro:include filename="$(find robotics_description)/urdf/sensors/lidars/generic_macros/plugin_lidar_3d_ring_macro.xacro"/>
       <xacro:plugin_lidar_3d_ring

File: urdf/sensors/lidars/robosense_helios_16_macro.xacro (robot description, xacro)
@@ -183,4 +183,12 @@
     -->
     <xacro:if value="${sim_enabled and sim_base_topic != ''}">
+      <xacro:if value="${use_visual and color != ''}">
+        <gazebo reference="${prefix}${name}_root_link">
+          <material>
+            <ambient>${color}</ambient>
+            <diffuse>${color}</diffuse>
+          </material>
+        </gazebo>
+      </xacro:if>
       <xacro:include filename="$(find robotics_description)/urdf/sensors/lidars/generic_macros/plugin_lidar_3d_ring_macro.xacro"/>
       <xacro:plugin_lidar_3d_ring

File: urdf/sensors/lidars/robosense_m1_plus_macro.xacro (robot description, xacro)
@@ -134,4 +134,12 @@
     </joint>
     <xacro:if value="${sim_enabled and sim_base_topic != ''}">
+      <xacro:if value="${use_visual and color != ''}">
+        <gazebo reference="${prefix}${name}_root_link">
+          <material>
+            <ambient>${color}</ambient>
+            <diffuse>${color}</diffuse>
+          </material>
+        </gazebo>
+      </xacro:if>
       <xacro:include filename="$(find robotics_description)/urdf/sensors/lidars/generic_macros/plugin_lidar_3d_ring_macro.xacro"/>
       <xacro:plugin_lidar_3d_ring

File: urdf/sensors/lidars/sick_s300_macro.xacro (robot description, xacro)
@@ -171,4 +171,12 @@
     -->
     <xacro:if value="${sim_enabled and sim_topic != ''}">
+      <xacro:if value="${use_visual and color != ''}">
+        <gazebo reference="${prefix}${name}_root_link">
+          <material>
+            <ambient>${color}</ambient>
+            <diffuse>${color}</diffuse>
+          </material>
+        </gazebo>
+      </xacro:if>
       <xacro:include filename="$(find robotics_description)/urdf/sensors/lidars/generic_macros/plugin_lidar_2d_macro.xacro"/>
       <xacro:plugin_lidar_2d
