Commit message: Renamed set_shaped_link_macro to link_w_shape_macro
New name is clearer in intentions.

File: urdf/common/all_commons.xacro (robot description, xacro)
@@ -5,4 +5,4 @@
   <xacro:include filename="$(find eut_robotics_description)/urdf/common/link_r_macro.xacro"/>
   <xacro:include filename="$(find eut_robotics_description)/urdf/common/link_s_macro.xacro"/>
-  <xacro:include filename="$(find eut_robotics_description)/urdf/common/set_shaped_link_macro.xacro"/>
+  <xacro:include filename="$(find eut_robotics_description)/urdf/common/link_w_shape_macro.xacro"/>
 </robot>

File: urdf/common/link_w_shape_macro.xacro (robot description, xacro)
@@ -9,6 +9,6 @@
 shape='s  2*radius  2*radius  2*radius'  -> sphere
 -->
-<robot name="set_shaped_link" xmlns:xacro="http://ros.org/wiki/xacro" xmlns:gz="http://gazebosim.org/schema">
-  <xacro:macro name="set_shaped_link"
+<robot name="link_w_shape" xmlns:xacro="http://ros.org/wiki/xacro" xmlns:gz="http://gazebosim.org/schema">
+  <xacro:macro name="link_w_shape"
                params="name
                        prefix

File: urdf/sensors/imus/generic_macros/imu_macro.xacro (robot description, xacro)
@@ -79,5 +79,5 @@
     <xacro:property name="shape_lst"  value="${shape.split()}"/>
     <xacro:property name="vci_pose_z" value="${0.5 * float(shape_lst[3])}"/>
-    <xacro:set_shaped_link
+    <xacro:link_w_shape
       name="${name}_root"
       prefix="${prefix}"

File: urdf/sensors/lidars/generic_macros/lidar_body_macro.xacro (robot description, xacro)
@@ -59,5 +59,5 @@
                        joint_root_fr_data_fr
                        joint_parent_fr_root_fr">
-    <xacro:include filename="$(find eut_robotics_description)/urdf/common/set_shaped_link_macro.xacro"/>
+    <xacro:include filename="$(find eut_robotics_description)/urdf/common/all_commons.xacro"/>
     <!--
     Convention:
@@ -66,5 +66,5 @@
     <xacro:property name="shape_lst"  value="${shape.split()}"/>
     <xacro:property name="vci_pose_z" value="${0.5 * float(shape_lst[3])}"/>
-    <xacro:set_shaped_link
+    <xacro:link_w_shape
       name="${name}_root"
       prefix="${prefix}"

File: urdf/wheels/wheel_macro.xacro (robot description, xacro)
@@ -92,5 +92,5 @@
     </xacro:unless>
     <!-- No mesh collision for the wheel, just a primitive cylinder along the y-axis or a sphere -->
-    <xacro:set_shaped_link
+    <xacro:link_w_shape
       name="${name}"
       prefix="${prefix}"

Commit message: Rename package to robotics_description and neutralize docs wording

File: urdf/common/all_commons.xacro (robot description, xacro)
@@ -2,10 +2,10 @@
 <robot name="all_commons" xmlns:xacro="http://www.ros.org/wiki/xacro" xmlns:gz="http://gazebosim.org/schema">
   <!--
-  <xacro:include filename="$(find eut_robotics_description)/urdf/common/inertia_macros.xacro"/>
+  <xacro:include filename="$(find robotics_description)/urdf/common/inertia_macros.xacro"/>
   -->
-  <xacro:include filename="$(find eut_robotics_description)/urdf/common/generic_link_macro.xacro"/>
-  <xacro:include filename="$(find eut_robotics_description)/urdf/common/inertial_macros.xacro"/>
-  <xacro:include filename="$(find eut_robotics_description)/urdf/common/make_namespace_macro.xacro"/>
-  <xacro:include filename="$(find eut_robotics_description)/urdf/common/make_prefix_macro.xacro"/>
-  <xacro:include filename="$(find eut_robotics_description)/urdf/common/visual_collision_macros.xacro"/>
+  <xacro:include filename="$(find robotics_description)/urdf/common/generic_link_macro.xacro"/>
+  <xacro:include filename="$(find robotics_description)/urdf/common/inertial_macros.xacro"/>
+  <xacro:include filename="$(find robotics_description)/urdf/common/make_namespace_macro.xacro"/>
+  <xacro:include filename="$(find robotics_description)/urdf/common/make_prefix_macro.xacro"/>
+  <xacro:include filename="$(find robotics_description)/urdf/common/visual_collision_macros.xacro"/>
 </robot>

File: urdf/common/visual_collision_macros.xacro (robot description, xacro)
@@ -6,10 +6,10 @@
 S means string
 B means boolean
-Note: In some expressions used in <xacro:if> tags you will observer the symgol '&lt;' instead of '<'.
+Note: In some expressions used in <xacro:if> tags, the symbol '&lt;' appears instead of '<'.
       This is because the character '<' is reserved in XML files. Therefore, to use it inside an attribute value, it
       must be escaped as '&lt;'.
 -->
 <robot name="visual_collision" xmlns:xacro="http://www.ros.org/wiki/xacro" xmlns:gz="http://gazebosim.org/schema">
-  <xacro:include filename="$(find eut_robotics_description)/urdf/common/set_basic_geometry_macro.xacro"/>
+  <xacro:include filename="$(find robotics_description)/urdf/common/set_basic_geometry_macro.xacro"/>
   <!--
   Macro for visual element with box shape.

File: urdf/extras/fork_macro.xacro (robot description, xacro)
@@ -82,6 +82,6 @@
                        limits:='0.0 0.0 0.0 0.0'
                        joint_parent_fr_root_fr">
-    <xacro:include filename="$(find eut_robotics_description)/urdf/common/all_commons.xacro"/>
-    <xacro:include filename="$(find eut_robotics_description)/urdf/extras/fork_tine_macro.xacro"/>
+    <xacro:include filename="$(find robotics_description)/urdf/common/all_commons.xacro"/>
+    <xacro:include filename="$(find robotics_description)/urdf/extras/fork_tine_macro.xacro"/>
     <xacro:property name="tine_size_seq" value="${tine_size.split()}"/>
     <xacro:if value="${len(tine_size_seq) != 3}">

File: urdf/extras/fork_tine_macro.xacro (robot description, xacro)
@@ -69,5 +69,5 @@
                        tine_mass:=0.1
                        joint_parent_fr_tine_fr:='0.0 0.0 0.0 0.0 0.0 0.0'">
-    <xacro:include filename="$(find eut_robotics_description)/urdf/common/all_commons.xacro"/>
+    <xacro:include filename="$(find robotics_description)/urdf/common/all_commons.xacro"/>
     <link name="${prefix}${name}_link">
       <xacro:if value="${use_visual}">

File: urdf/sensors/all_sensors_macro.xacro (robot description, xacro)
@@ -1,6 +1,6 @@
 <?xml version="1.0"?>
 <robot name="all_sensors" xmlns:xacro="http://www.ros.org/wiki/xacro" xmlns:gz="http://gazebosim.org/schema">
-  <xacro:include filename="$(find eut_robotics_description)/urdf/sensors/cameras/all_cameras_macros.xacro"/>
-  <xacro:include filename="$(find eut_robotics_description)/urdf/sensors/imus/all_imus_macros.xacro"/>
-  <xacro:include filename="$(find eut_robotics_description)/urdf/sensors/lidars/all_lidars_macros.xacro"/>
+  <xacro:include filename="$(find robotics_description)/urdf/sensors/cameras/all_cameras_macros.xacro"/>
+  <xacro:include filename="$(find robotics_description)/urdf/sensors/imus/all_imus_macros.xacro"/>
+  <xacro:include filename="$(find robotics_description)/urdf/sensors/lidars/all_lidars_macros.xacro"/>
 </robot>

File: urdf/sensors/cameras/all_cameras_macros.xacro (robot description, xacro)
@@ -1,5 +1,5 @@
 <?xml version="1.0"?>
 <robot name="all_cameras" xmlns:xacro="http://www.ros.org/wiki/xacro" xmlns:gz="http://gazebosim.org/schema">
-    <xacro:include filename="$(find eut_robotics_description)/urdf/sensors/cameras/generic_macros/set_props_plugin_camera_all_macro.xacro"/>
-    <xacro:include filename="$(find eut_robotics_description)/urdf/sensors/cameras/realsense_d435.xacro"/>
+    <xacro:include filename="$(find robotics_description)/urdf/sensors/cameras/generic_macros/set_props_plugin_camera_all_macro.xacro"/>
+    <xacro:include filename="$(find robotics_description)/urdf/sensors/cameras/realsense_d435.xacro"/>
 </robot>

File: urdf/sensors/cameras/generic_macros/plugin_camera_bounding_box_macro.xacro (robot description, xacro)
@@ -171,5 +171,5 @@
                        info_topic
                        trigger_topic:=''" >
-    <xacro:include filename="$(find eut_robotics_description)/urdf/sensors/cameras/generic_macros/plugin_camera_common_macro.xacro"/>
+    <xacro:include filename="$(find robotics_description)/urdf/sensors/cameras/generic_macros/plugin_camera_common_macro.xacro"/>
     <xacro:if value="${box_type != '2d' and box_type != 'visible_2d' and box_type != 'visible_box_2d' and box_type != 'full_2d' and box_type != 'full_box_2d' and box_type != '3d'}">
       ${xacro.fatal('Invalid box_type. Valid: 2d | visible_2d | visible_box_2d | full_2d | full_box_2d | 3d')}

File: urdf/sensors/cameras/generic_macros/plugin_camera_common_macro.xacro (robot description, xacro)
@@ -112,5 +112,5 @@
       center_y_norm = (cy + 0.5) / image_height_in_pixels
       Why +0.5 in the formulas?
-      We normalize distortion center in edge coordinates where the left border is 0 and right border is W, hence the
+      Distortion center is normalized in edge coordinates where the left border is 0 and right border is W, hence the
       +0.5 shift from pixel-center coordinates.
   - Pass center_x_norm and center_y_norm in the distortion.center_x and distortion.center_y parameters.
@@ -345,5 +345,5 @@
       According to the sdformat documentation, if lens_projection is defined, it overrides the intrinsics parameters
       fx, fy, cx, cy.
-      Therefore, if lens_projection is defined, we use it.
+      Therefore, if lens_projection is defined, it is used.
       -->
       <xacro:if value="${lens_projection != ''}">
@@ -369,9 +369,9 @@
         When 'lens_projection' is used, still set the 'lens_xy_skew' in the intrinsics element since there is no other
         way to set it.
-        Since the rest of the element in intrinsics are required (see sdformat documentation), we must set them,
-        otherwise sdf parser will raise an error. However, in practical terms, no matter the values we give to fx, fy,
-        cx, cy here, they will be overridden by the values in projection (p_fx, p_fy, p_cx, p_cy), as we can read in the
+        Since the rest of the element in intrinsics are required (see sdformat documentation), they must be set,
+        otherwise sdf parser will raise an error. However, in practical terms, no matter the values assigned to fx, fy,
+        cx, cy here, they will be overridden by the values in projection (p_fx, p_fy, p_cx, p_cy), as described in the
         sdformat documentation.
-        Therefore, we set the parameters fx, fy, cx, cy to p_fx, p_fy, p_cx, p_cy respectively, just to avoid errors
+        Therefore, the parameters fx, fy, cx, cy are set to p_fx, p_fy, p_cx, p_cy respectively, just to avoid errors
         in sdf parsing, knowing that these values will be overridden later by the projection values.
         -->

File: urdf/sensors/cameras/generic_macros/plugin_camera_depth_macro.xacro (robot description, xacro)
@@ -115,5 +115,5 @@
       center_y_norm = (cy + 0.5) / image_height_in_pixels
       Why +0.5 in the formulas?
-      We normalize distortion center in edge coordinates where the left border is 0 and right border is W, hence the
+      Distortion center is normalized in edge coordinates where the left border is 0 and right border is W, hence the
       +0.5 shift from pixel-center coordinates.
   - Pass center_x_norm and center_y_norm in the distortion.center_x and distortion.center_y parameters.
@@ -248,5 +248,5 @@
                        distortion_center:='0.5 0.5'
                        gaussian_noise:='0.0 0.0'">
-    <xacro:include filename="$(find eut_robotics_description)/urdf/sensors/cameras/generic_macros/plugin_camera_common_macro.xacro"/>
+    <xacro:include filename="$(find robotics_description)/urdf/sensors/cameras/generic_macros/plugin_camera_common_macro.xacro"/>
     <xacro:if value="${type != 'depth_camera' and type != 'depth' and type != 'rgbd_camera' and type != 'rgbd'}">
       ${xacro.fatal("Invalid depth camera type")}

File: urdf/sensors/cameras/generic_macros/plugin_camera_macro.xacro (robot description, xacro)
@@ -94,5 +94,5 @@
   center_y_norm = (cy + 0.5) / image_height_in_pixels
   Why +0.5 in the formulas?
-  We normalize distortion center in edge coordinates where the left border is 0 and right border is W, hence the
+  Distortion center is normalized in edge coordinates where the left border is 0 and right border is W, hence the
   +0.5 shift from pixel-center coordinates.
 - Pass center_x_norm and center_y_norm in the distortion.center_x and distortion.center_y parameters.
@@ -226,5 +226,5 @@
                        distortion_center:='0.5 0.5'
                        gaussian_noise:='0.0 0.0'">
-    <xacro:include filename="$(find eut_robotics_description)/urdf/sensors/cameras/generic_macros/plugin_camera_common_macro.xacro"/>
+    <xacro:include filename="$(find robotics_description)/urdf/sensors/cameras/generic_macros/plugin_camera_common_macro.xacro"/>
     <gazebo reference="${reference_frame}">
       <gravity>${use_gravity}</gravity>

File: urdf/sensors/cameras/generic_macros/plugin_camera_segmentation_macro.xacro (robot description, xacro)
@@ -177,5 +177,5 @@
                        info_topic
                        trigger_topic:=''" >
-    <xacro:include filename="$(find eut_robotics_description)/urdf/sensors/cameras/generic_macros/plugin_camera_common_macro.xacro"/>
+    <xacro:include filename="$(find robotics_description)/urdf/sensors/cameras/generic_macros/plugin_camera_common_macro.xacro"/>
     <xacro:if value="${segmentation_type != 'semantic' and segmentation_type != 'panoptic' and segmentation_type != 'instance'}">
       ${xacro.fatal("Invalid segmentation_type. Valid: semantic | panoptic | instance")}

File: urdf/sensors/cameras/generic_macros/plugin_camera_thermal_macro.xacro (robot description, xacro)
@@ -165,5 +165,5 @@
                        info_topic
                        trigger_topic:=''" >
-    <xacro:include filename="$(find eut_robotics_description)/urdf/sensors/cameras/generic_macros/plugin_camera_common_macro.xacro"/>
+    <xacro:include filename="$(find robotics_description)/urdf/sensors/cameras/generic_macros/plugin_camera_common_macro.xacro"/>
     <xacro:property name='thermal_sequence' value='${thermal_data.split()}'/>
     <xacro:if value='${len(thermal_sequence) != 3}'>

File: urdf/sensors/cameras/realsense_d435.xacro (robot description, xacro)
@@ -205,5 +205,5 @@
                        depth_cam_sim_distortion_center:='0.5 0.5'
                        depth_cam_sim_gaussian_noise:='0.0 0.0'">
-    <xacro:include filename="$(find eut_robotics_description)/urdf/common/all_commons.xacro"/>
+    <xacro:include filename="$(find robotics_description)/urdf/common/all_commons.xacro"/>
     <!--
     The following values are approximate, and the camera node publishing TF values with actual calibrated camera
@@ -242,5 +242,5 @@
     -->
     <xacro:property name="mesh"
-                    value="eut_robotics_description/meshes/sensors/cameras/realsense_d435/mesh.stl"/>
+                    value="robotics_description/meshes/sensors/cameras/realsense_d435/mesh.stl"/>
     <xacro:property name="mesh_scale" value="1.0 1.0 1.0"/>
     <xacro:property name="origin"
@@ -348,6 +348,6 @@
     </xacro:if>
     <xacro:if value="${use_sim}">
-      <xacro:include filename="$(find eut_robotics_description)/urdf/sensors/cameras/generic_macros/plugin_camera_macro.xacro"/>
-      <xacro:include filename="$(find eut_robotics_description)/urdf/sensors/cameras/generic_macros/plugin_camera_depth_macro.xacro"/>
+      <xacro:include filename="$(find robotics_description)/urdf/sensors/cameras/generic_macros/plugin_camera_macro.xacro"/>
+      <xacro:include filename="$(find robotics_description)/urdf/sensors/cameras/generic_macros/plugin_camera_depth_macro.xacro"/>
       <xacro:make_namespace prop_id="camera_namespace" namespace="${namespace}" name="${name}"/>
       <xacro:if value="${color_cam_sim_enabled}">

File: urdf/sensors/imus/all_imus_macros.xacro (robot description, xacro)
@@ -1,5 +1,5 @@
 <?xml version="1.0"?>
 <robot name="all_imus" xmlns:xacro="http://www.ros.org/wiki/xacro" xmlns:gz="http://gazebosim.org/schema">
-  <xacro:include filename="$(find eut_robotics_description)/urdf/sensors/imus/generic_macros/set_props_plugin_imu_macro.xacro"/>
-  <xacro:include filename="$(find eut_robotics_description)/urdf/sensors/imus/um7_macro.xacro"/>
+  <xacro:include filename="$(find robotics_description)/urdf/sensors/imus/generic_macros/set_props_plugin_imu_macro.xacro"/>
+  <xacro:include filename="$(find robotics_description)/urdf/sensors/imus/um7_macro.xacro"/>
 </robot>

File: urdf/sensors/imus/um7_macro.xacro (robot description, xacro)
@@ -65,5 +65,5 @@
                        sim_lin_acc_gaussian_noise_dynamic_bias:='0 0 0 0 0 0'
                        sim_use_orientation:=True">
-    <xacro:include filename="$(find eut_robotics_description)/urdf/common/all_commons.xacro"/>
+    <xacro:include filename="$(find robotics_description)/urdf/common/all_commons.xacro"/>
     <xacro:property name="mass"   value="0.0110"/>
     <!--
@@ -85,5 +85,5 @@
     To access the mesh just use <package>/<path_to_mesh_within_package>.
     -->
-    <xacro:property name="mesh"       value="eut_robotics_description/meshes/sensors/imus/um7/mesh.dae"/>
+    <xacro:property name="mesh"       value="robotics_description/meshes/sensors/imus/um7/mesh.dae"/>
     <xacro:property name="mesh_scale" value="1.0 1.0 1.0"/>
     <!--
@@ -135,5 +135,5 @@
     </joint>
     <xacro:if value="${use_sim}">
-      <xacro:include filename="$(find eut_robotics_description)/urdf/sensors/imus/generic_macros/plugin_imu_macro.xacro"/>
+      <xacro:include filename="$(find robotics_description)/urdf/sensors/imus/generic_macros/plugin_imu_macro.xacro"/>
       <xacro:make_namespace prop_id="imu_namespace" namespace="${namespace}" name="${name}"/>
       <xacro:plugin_imu

File: urdf/sensors/lidars/all_lidars_macros.xacro (robot description, xacro)
@@ -1,7 +1,7 @@
 <?xml version="1.0"?>
 <robot name="all_lidars" xmlns:xacro="http://www.ros.org/wiki/xacro" xmlns:gz="http://gazebosim.org/schema">
-  <xacro:include filename="$(find eut_robotics_description)/urdf/sensors/lidars/generic_macros/set_props_plugin_lidar_2d_macro.xacro"/>
-  <xacro:include filename="$(find eut_robotics_description)/urdf/sensors/lidars/generic_macros/set_props_plugin_lidar_3d_ring_macro.xacro"/>
-  <xacro:include filename="$(find eut_robotics_description)/urdf/sensors/lidars/robosense_airy_macro.xacro"/>
-  <xacro:include filename="$(find eut_robotics_description)/urdf/sensors/lidars/robosense_helios_16p_macro.xacro"/>
+  <xacro:include filename="$(find robotics_description)/urdf/sensors/lidars/generic_macros/set_props_plugin_lidar_2d_macro.xacro"/>
+  <xacro:include filename="$(find robotics_description)/urdf/sensors/lidars/generic_macros/set_props_plugin_lidar_3d_ring_macro.xacro"/>
+  <xacro:include filename="$(find robotics_description)/urdf/sensors/lidars/robosense_airy_macro.xacro"/>
+  <xacro:include filename="$(find robotics_description)/urdf/sensors/lidars/robosense_helios_16p_macro.xacro"/>
 </robot>

File: urdf/sensors/lidars/robosense_airy_macro.xacro (robot description, xacro)
@@ -25,5 +25,5 @@
                        sim_dist_span
                        sim_gaussian_noise:='0 0'">
-    <xacro:include filename="$(find eut_robotics_description)/urdf/common/all_commons.xacro"/>
+    <xacro:include filename="$(find robotics_description)/urdf/common/all_commons.xacro"/>
     <xacro:property name="mass"   value="0.25"/>
     <!--
@@ -42,5 +42,5 @@
     -->
     <xacro:property name="mesh"
-                    value="eut_robotics_description/meshes/sensors/lidars/robosense_airy/mesh.stl"/>
+                    value="robotics_description/meshes/sensors/lidars/robosense_airy/mesh.stl"/>
     <!--
     The mesh represents a cylinder with its symmetry axis along the z-axis.
@@ -51,5 +51,5 @@
     -->
     <xacro:property name="low_res_mesh"
-                    value="eut_robotics_description/meshes/sensors/lidars/robosense_airy/mesh_low_res.dae"/>
+                    value="robotics_description/meshes/sensors/lidars/robosense_airy/mesh_low_res.dae"/>
     <!-- Scale for both meshes, standard mesh and low resolition mesh -->
     <xacro:property name="mesh_scale" value="1.0 1.0 1.0"/>
@@ -116,5 +116,5 @@
     Therefore, the driver is making a transformation of the data to provide each point of the point cloud, referred to
     the center of the base of the sensor.
-    Therefore, for practical purposes, we can assume the data frame is located at the center of the base of the sensor,
+    Therefore, for practical purposes, it can be assumed that the data frame is located at the center of the base of the sensor,
     coinciding with the root frame of the sensor.
     -->
@@ -125,5 +125,5 @@
     </joint>
     <xacro:if value="${use_sim}">
-      <xacro:include filename="$(find eut_robotics_description)/urdf/sensors/lidars/generic_macros/plugin_lidar_3d_ring_macro.xacro"/>
+      <xacro:include filename="$(find robotics_description)/urdf/sensors/lidars/generic_macros/plugin_lidar_3d_ring_macro.xacro"/>
       <!--
       The behaviour of the Gazebo Sim plugin for a 3D ring LiDAR is to publish two topics:

File: urdf/sensors/lidars/robosense_helios_16p_macro.xacro (robot description, xacro)
@@ -25,5 +25,5 @@
                        sim_dist_span
                        sim_gaussian_noise:='0 0'">
-    <xacro:include filename="$(find eut_robotics_description)/urdf/common/all_commons.xacro"/>
+    <xacro:include filename="$(find robotics_description)/urdf/common/all_commons.xacro"/>
     <xacro:property name="mass"   value="0.99"/>
     <!--
@@ -42,5 +42,5 @@
     -->
     <xacro:property name="mesh"
-                    value="eut_robotics_description/meshes/sensors/lidars/robosense_helios_16p/mesh.stl"/>
+                    value="robotics_description/meshes/sensors/lidars/robosense_helios_16p/mesh.stl"/>
     <!--
     The mesh represents a cylinder with its symmetry axis along the z-axis.
@@ -51,5 +51,5 @@
     -->
     <xacro:property name="low_res_mesh"
-                    value="eut_robotics_description/meshes/sensors/lidars/robosense_helios_16p/mesh_low_res.dae"/>
+                    value="robotics_description/meshes/sensors/lidars/robosense_helios_16p/mesh_low_res.dae"/>
     <!-- Scale for both meshes, standard mesh and low resolition mesh -->
     <xacro:property name="mesh_scale" value="1.0 1.0 1.0"/>
@@ -112,5 +112,5 @@
     </joint>
     <xacro:if value="${use_sim}">
-      <xacro:include filename="$(find eut_robotics_description)/urdf/sensors/lidars/generic_macros/plugin_lidar_3d_ring_macro.xacro"/>
+      <xacro:include filename="$(find robotics_description)/urdf/sensors/lidars/generic_macros/plugin_lidar_3d_ring_macro.xacro"/>
       <!--
       The behaviour of the Gazebo Sim plugin for a 3D ring LiDAR is to publish two topics:
