Commit message: refactor(robotics_description): align wheel and airy geometry conventions

File: urdf/common/visual_collision_macros.xacro (robot description, xacro)
@@ -212,11 +212,11 @@
       raised.
       -->
-      <xacro:if value="${len(c) == 5}">
+      <xacro:if value="${color != ''}">
+        <xacro:if value="${len(c) != 5}">
+          ${xacro.fatal("v_element: color must be 'color_name r g b a'")}
+        </xacro:if>
         <material name="${c[0]}">
           <color rgba="${c[1]} ${c[2]} ${c[3]} ${c[4]}"/>
         </material>
-      </xacro:if>
-      <xacro:if value="${color != '' and len(c) != 5}">
-        ${xacro.fatal("v_element: color must be 'color_name r g b a'")}
       </xacro:if>
     </visual>
@@ -250,4 +250,7 @@
     </collision>
   </xacro:macro>
+  <!-- ===================================================================== -->
+  <!-- MACROS BELOW ARE FOR INNER USE ONLY -->
+  <!-- ===================================================================== -->
   <!--
   Macro for internal use to set the common elements of the visual and collision tags.
@@ -271,10 +274,10 @@
                       shape_origin:='0.0 0.0 0.0 0.0 0.0 0.0'">
     <xacro:if value="${mesh != ''}">
-      <xacro:property name="sc_seq" value="${scale.split()}"/>
-      <xacro:property name="mo_seq" value="${mesh_origin.split()}"/>
-      <xacro:if value="${len(sc_seq) != 3}">
+      <xacro:property name="scale_items" value="${scale.split()}"/>
+      <xacro:if value="${len(scale_items) != 3}">
         ${xacro.fatal("vc_common: scale must be 'scale_x scale_y scale_z'")}
       </xacro:if>
-      <xacro:if value="${len(mo_seq) != 6}">
+      <xacro:property name="mo_items" value="${mesh_origin.split()}"/>
+      <xacro:if value="${len(mo_items) != 6}">
         ${xacro.fatal("vc_common: mesh origin must be 'x y z roll pitch yaw'")}
       </xacro:if>
@@ -282,5 +285,6 @@
         <mesh filename="package://${mesh}" scale="${scale}"/>
       </geometry>
-      <origin rpy="${mo_seq[3]} ${mo_seq[4]} ${mo_seq[5]}" xyz="${mo_seq[0]} ${mo_seq[1]} ${mo_seq[2]}"/>
+      <origin rpy="${mo_items[3]} ${mo_items[4]} ${mo_items[5]}"
+              xyz="${mo_items[0]} ${mo_items[1]} ${mo_items[2]}"/>
     </xacro:if>
     <xacro:if value="${mesh == ''}">
@@ -300,31 +304,31 @@
   -->
   <xacro:macro name="set_basic_geometry" params="shape:='b 0.0 0.0 0.0'">
-    <xacro:property name="sh_seq"  value="${shape.split()}"/>
-    <xacro:if value="${len(sh_seq) &lt; 2}">
+    <xacro:property name="shape_items"  value="${shape.split()}"/>
+    <xacro:if value="${len(shape_items) &lt; 2}">
       ${xacro.fatal("set_basic_geometry: shape parameter is too short")}
     </xacro:if>
-    <xacro:property name="shape_type" value="${sh_seq[0]}"/>
+    <xacro:property name="shape_type" value="${shape_items[0]}"/>
     <xacro:if value="${shape_type not in ('b', 'c', 's')}">
       ${xacro.fatal("The field 'shape' must be one of: 'b' (box), 'c' (cylinder), 's' (sphere)")}
     </xacro:if>
     <xacro:if value="${shape_type == 'b'}">
-      <xacro:if value="${len(sh_seq) &lt; 4}">
+      <xacro:if value="${len(shape_items) &lt; 4}">
         ${xacro.fatal("set_basic_geometry: invalid box shape. Expected: 'b sx sy sz'")}
       </xacro:if>
       <geometry>
-        <box size="${sh_seq[1]} ${sh_seq[2]} ${sh_seq[3]}"/>
+        <box size="${shape_items[1]} ${shape_items[2]} ${shape_items[3]}"/>
       </geometry>
     </xacro:if>
     <xacro:if value="${shape_type == 'c'}">
-      <xacro:if value="${len(sh_seq) &lt; 3}">
+      <xacro:if value="${len(shape_items) &lt; 3}">
         ${xacro.fatal("set_basic_geometry: invalid cylinder shape. Expected: 'c radius length'")}
       </xacro:if>
       <geometry>
-        <cylinder radius="${sh_seq[1]}" length="${sh_seq[2]}"/>
+        <cylinder radius="${shape_items[1]}" length="${shape_items[2]}"/>
       </geometry>
     </xacro:if>
     <xacro:if value="${shape_type == 's'}">
       <geometry>
-        <sphere radius="${sh_seq[1]}"/>
+        <sphere radius="${shape_items[1]}"/>
       </geometry>
     </xacro:if>

File: urdf/sensors/lidars/robosense_airy_macro.xacro (robot description, xacro)
@@ -163,8 +163,9 @@
     <xacro:property name="mesh_scale" value="1.0 1.0 1.0"/>
     <!--
-    Since, both, meshes, the standard and the low resolution, are cylinders with their symmetry axis along the z-axis,
-    and the frame of both meshes is located at their geometric center (see MeshLab), their frames coincide with the
-    frame of a cylinder shape, with its symmetry axis along the z-axis, so just one origin is needed no matter if
-    use_<v|c>_mesh is true or false.
+    Since, both, meshes, the standard and the low resolution, are cylinders with their symmetry
+    axis along the z-axis, and the frame of both meshes is located at their geometric center
+    (see MeshLab), their frames coincide with the frame of a cylinder shape, with its symmetry axis
+    along the z-axis, so just one origin is needed no matter whether use_<v|c>_mesh is true or
+    false.
     The body frame is located at the center of the bottom face of the cylinder.
     -->
@@ -214,16 +215,18 @@
     </link>
     <!--
-    Definition of the joint '${prefix}${name}_joint', that joins the lidar data link to its root link.
-    This pose sets the position and orientation of the sensor frame with respect the root frame, located at the center
-    of the bottom face of the cylinder.
-    The Airy sensor is 'ackwardly' designed IMHO (jfrascon), as the light source is not located at the center of the
-    dome, at some height, it is located deviated from the center of the dome, and at some height.
+    Definition of the joint '${prefix}${name}_joint', that joins the lidar data link to its root
+    link.
+    This pose sets the position and orientation of the sensor frame with respect the root frame,
+    located at the center of the bottom face of the cylinder.
+    The Airy sensor is 'ackwardly' designed IMHO (jfrascon), as the light source is not located at
+    the center of the dome, at some height, it is located deviated from the center of the dome, and
+    at some height.
     The location of the optical center is shown in page 63 of the Airy user manual.
     However, on page 27 it is stated that:
     "The origin of the coordinates for the LiDAR is defined at the center of the LiDAR base."
-    Therefore, the driver is making a transformation of the data to provide each point of the point cloud, referred to
-    the center of the base of the sensor.
-    Therefore, for practical purposes, it can be assumed that the data frame is located at the center of the base of the sensor,
-    coinciding with the root frame of the sensor.
+    Therefore, the driver is making a transformation of the data to provide each point of the point
+    cloud, referred to the center of the base of the sensor.
+    Therefore, for practical purposes, it can be assumed that the data frame is located at the
+    center of the base of the sensor, coinciding with the root frame of the sensor.
     -->
     <joint name="${prefix}${name}_joint" type="fixed">

File: urdf/wheels/steerable_wheel_macro.xacro (robot description, xacro)
@@ -18,11 +18,4 @@
 v_mesh_scale (S): Scale of the visual mesh, if use_visual is true and v_mesh is provided.
     v_mesh_scale (S) = 'sx (R) sy (R) sz (R)'.
-v_mesh_origin (S): String of the form 'x (R) y (R) z (R) roll (R) pitch (R) yaw (R)' used to place the visual mesh
-                   w.r.t the frame '${prefix}${name}_rotation_link'. Used only if use_visual is true and v_mesh is provided.
-                   IMPORTANT: The wheel frame convention is fixed:
-                     - +Y is the wheel spin axis.
-                     - +X is the rolling direction.
-                     - +Z points upward.
-                   v_mesh_origin must align the mesh to that convention.
 color (S): String of the form 'r (R) g (R) b (R) a (R)'. Used only if use_visual is true.
            If color is not empty, the provided color is applied to the object used in the visual element, either
@@ -118,5 +111,4 @@
                        v_mesh:=''
                        v_mesh_scale:='1.0 1.0 1.0'
-                       v_mesh_origin:='0.0 0.0 0.0 0.0 0.0 0.0'
                        color:=''
                        radius
@@ -136,17 +128,21 @@
     <xacro:include filename="$(find robotics_description)/urdf/common/all_commons.xacro"/>
     <!--
-    Frame convention for '${prefix}${name}_rotation_link':
+    If a wheel mesh is provided through `v_mesh`, that mesh must be modeled with the wheel "lying on
+    the ground". In that initial orientation, the wheel symmetry axis must be +Z.
+    This requirement is used so that meshes follow the same initial convention as the primitive
+    cylinder used when `v_mesh` is empty. A URDF cylinder is Z-axis aligned by default.
+    This macro uses the following wheel frame convention:
       - +Y is wheel spin axis.
       - +X is rolling direction.
       - +Z points upward.
-    If v_mesh is provided, v_mesh_origin must align the mesh to that convention.
-    If v_mesh is empty, a primitive cylinder is used for visual.
-    Collision is always enabled and always represented as a primitive cylinder (no collision mesh), to keep contacts
-    stable and fast.
-    Primitive cylinders are Z-axis aligned by default in URDF, so they are rotated by +pi/2 around X using:
-      shape_origin = "0.0 0.0 0.0 0.5*pi 0.0 0.0"
-    The same shape_origin is used by visual primitives and collision primitives.
+    For that reason, both the visual geometry and the collision geometry are rotated by +pi/2 around X
+    before they are attached to '${prefix}${name}_rotation_link'.
+    If `v_mesh` is empty, that +pi/2 rotation is applied to the primitive cylinder.
+    If `v_mesh` is provided, the same +pi/2 rotation is applied to the visual mesh.
+    Collision is always enabled and always represented as a primitive cylinder.
+    The same +pi/2 rotation is also applied to that collision geometry, so visual and collision use
+    the same wheel orientation.
     -->
-    <xacro:property name="shape_origin" value="0.0 0.0 0.0 ${0.5 * pi} 0.0 0.0"/>
+    <xacro:property name="wheel_origin" value="0.0 0.0 0.0 ${0.5 * pi} 0.0 0.0"/>
     <link name="${prefix}${name}_steerable_link">
       <!--
@@ -161,4 +157,10 @@
     <!-- Parsed as [x, y, z, roll, pitch, yaw]. -->
     <xacro:property name="j" value="${joint_parent_fr_wheel_fr.split()}"/>
+    <xacro:if value="${len(j) != 6}">
+      ${xacro.fatal(
+        "steerable_wheel: joint_parent_fr_wheel_fr must have 6 elements: "
+        "'x y z roll pitch yaw'"
+      )}
+    </xacro:if>
     <joint name="${prefix}${name}_steering_joint" type="${steering_joint_type}">
       <parent link="${parent_frame}"/>
@@ -183,8 +185,8 @@
         <xacro:visual_cylinder mesh="${v_mesh}"
                                scale="${v_mesh_scale}"
-                               mesh_origin="${v_mesh_origin}"
+                               mesh_origin="${wheel_origin}"
                                radius="${radius}"
                                length="${length}"
-                               shape_origin="${shape_origin}"
+                               shape_origin="${wheel_origin}"
                                color="${v_color}"/>
       </xacro:if>
@@ -195,11 +197,11 @@
       <xacro:collision_cylinder radius="${radius}"
                                 length="${length}"
-                                shape_origin="${shape_origin}"/>
+                                shape_origin="${wheel_origin}"/>
       <xacro:if value="${use_inertial}">
       <!--
       The inertia of a solid cylinder with uniform mass distribution, radius and length is used, with symmetry axis
       is the y-axis and center of mass is at the origin of the wheel's frame.
-      For that reason, the origin used is "0 0 0 0 0 0", unlinke the shape_origin used for visual and collision
-      elements.
+      For that reason, the origin used is "0 0 0 0 0 0", unlike the rotated geometry origin used for
+      visual and collision elements.
       In other words, solid_cylinder_inertia_y computes the same inertia as if solid_cylinder_inertia_z were used
       (assuming the cylinder's symmetry axis is along the z-axis, which is the default for a cylinder shape) but using

File: urdf/wheels/wheel_macro.xacro (robot description, xacro)
@@ -18,11 +18,4 @@
 v_mesh_scale (S): Scale of the visual mesh, if use_visual is true and v_mesh is provided.
     v_mesh_scale (S) = 'sx (R) sy (R) sz (R)'.
-v_mesh_origin (S): String of the form 'x (R) y (R) z (R) roll (R) pitch (R) yaw (R)' used to place the visual mesh
-                   w.r.t the frame '${prefix}${name}_rotation_link'. Used only if use_visual is true and v_mesh is provided.
-                   IMPORTANT: The wheel frame convention is fixed:
-                     - +Y is the wheel spin axis.
-                     - +X is the rolling direction.
-                     - +Z points upward.
-                   v_mesh_origin must align the mesh to that convention.
 color (S): String of the form 'r (R) g (R) b (R) a (R)'. Used only if use_visual is true.
            If color is not empty, the provided color is applied to the object used in the visual element, either
@@ -95,5 +88,4 @@
                        v_mesh:=''
                        v_mesh_scale:='1.0 1.0 1.0'
-                       v_mesh_origin:='0.0 0.0 0.0 0.0 0.0 0.0'
                        color:=''
                        radius
@@ -116,13 +108,21 @@
       - +X is rolling direction.
       - +Z points upward.
-    If v_mesh is provided, v_mesh_origin must align the mesh to that convention.
-    If v_mesh is empty, a primitive cylinder is used for visual.
-    Collision is always enabled and always represented as a primitive cylinder (no collision mesh), to keep contacts
-    stable and fast.
-    Primitive cylinders are Z-axis aligned by default in URDF, so they are rotated by +pi/2 around X using:
-      shape_origin = "0.0 0.0 0.0 0.5*pi 0.0 0.0"
-    The same shape_origin is used by visual primitives and collision primitives.
+    If a wheel mesh is provided through `v_mesh`, that mesh must be modeled with the wheel "lying on
+    the ground". In that initial orientation, the wheel symmetry axis must be +Z.
+    This requirement is used so that meshes follow the same initial convention as the primitive
+    cylinder used when `v_mesh` is empty. A URDF cylinder is Z-axis aligned by default.
+    This macro uses the following wheel frame convention:
+      - +Y is wheel spin axis.
+      - +X is rolling direction.
+      - +Z points upward.
+    For that reason, both the visual geometry and the collision geometry are rotated by +pi/2 around X
+    before they are attached to '${prefix}${name}_rotation_link'.
+    If `v_mesh` is empty, that +pi/2 rotation is applied to the primitive cylinder.
+    If `v_mesh` is provided, the same +pi/2 rotation is applied to the visual mesh.
+    Collision is always enabled and always represented as a primitive cylinder.
+    The same +pi/2 rotation is also applied to that collision geometry, so visual and collision use
+    the same wheel orientation.
     -->
-    <xacro:property name="shape_origin" value="0.0 0.0 0.0 ${0.5 * pi} 0.0 0.0"/>
+    <xacro:property name="wheel_origin" value="0.0 0.0 0.0 ${0.5 * pi} 0.0 0.0"/>
     <link name="${prefix}${name}_rotation_link">
       <xacro:if value="${use_visual}">
@@ -131,8 +131,8 @@
         <xacro:visual_cylinder mesh="${v_mesh}"
                                scale="${v_mesh_scale}"
-                               mesh_origin="${v_mesh_origin}"
+                               mesh_origin="${wheel_origin}"
                                radius="${radius}"
                                length="${length}"
-                               shape_origin="${shape_origin}"
+                               shape_origin="${wheel_origin}"
                                color="${v_color}"/>
       </xacro:if>
@@ -143,11 +143,11 @@
       <xacro:collision_cylinder radius="${radius}"
                                 length="${length}"
-                                shape_origin="${shape_origin}"/>
+                                shape_origin="${wheel_origin}"/>
       <xacro:if value="${use_inertial}">
       <!--
       The inertia of a solid cylinder with uniform mass distribution, radius and length is used, with symmetry axis
       is the y-axis and center of mass is at the origin of the wheel's frame.
-      For that reason, the origin used is "0 0 0 0 0 0", unlinke the shape_origin used for visual and collision
-      elements.
+      For that reason, the origin used is "0 0 0 0 0 0", unlike the rotated geometry origin used for
+      visual and collision elements.
       In other words, solid_cylinder_inertia_y computes the same inertia as if solid_cylinder_inertia_z were used
       (assuming the cylinder's symmetry axis is along the z-axis, which is the default for a cylinder shape) but using
@@ -168,4 +168,7 @@
     <!-- Parsed as [x, y, z, roll, pitch, yaw]. -->
     <xacro:property name="j" value="${joint_parent_fr_wheel_fr.split()}"/>
+    <xacro:if value="${len(j) != 6}">
+      ${xacro.fatal("wheel: joint_parent_fr_wheel_fr must have 6 elements: 'x y z roll pitch yaw'")}
+    </xacro:if>
     <joint name="${prefix}${name}_rotation_joint" type="${rotation_joint_type}">
       <parent link="${parent_frame}"/>
