Commit message: refactor(fork-simple): modernize the reference fork model
Rework the reference fork_simple assets and macros so they use the
current mesh layout and a clearer links-and-joints helper split.

This renames the shipped mesh artifacts, replaces the old _0 macro,
and updates the focused xacro test to exercise the new fork_simple
entry point.

File: urdf/extras/fork_simple/fork_simple_macro.xacro (robot description, xacro)
@@ -1,189 +1,158 @@
+<?xml version="1.0"?>
 <!--
-This macro provides a generic, simplified forklift-fork model.
-It is designed to work with a `fork_simple` mesh generated by
-`meshes/extras/fork_simple/fork_simple_stl_generator.py`
-Design choice:
-- A mesh is required (no primitive-box fallback). Building an equivalent fork from basic Xacro/URDF primitives
-  requires combining multiple shapes and offsets, which adds unnecessary complexity even for a simple model.
-  The generated mesh keeps the geometry representative while remaining lightweight for visual and collision use
-  in simulation.
-Intended usage:
-- This macro is a reusable base macro.
-- A model-specific macro (for a concrete fork model) should call it and pass the final parameter values.
-Convention for parameter types:
-R means real number (with decimal point)
-I means integer (without decimal point)
-S means string (any sequence of characters)
-B means boolean (true or false)
-name (S): base name for links and joints created by the macro.
-prefix (S): optional prefix prepended to all generated link/joint names.
-parent_frame (S): parent link/frame name for `${prefix}${name}_root_joint`.
-mesh (S): mesh filename resolved as package URI (for example
-    'robotics_description/meshes/extras/fork_simple/fork_simple_20260219.stl'),
-    used for both visual and collision (required).
-color (S): RGBA string for the visual material.
-  color (S) = 'r (R) g (R) b (R) a (R)'.
-mass (R): total mass of the fork body. Required only when `inertial_elements` is provided.
-tine_size (S): tine bounding-box size used for tine offset calculations:
-    tine_size (S) = 'sx (R) sy (R) sz (R)'.
-tine_separation (R): distance between inner faces of left/right tines.
-tine_union_size_x (R): X offset from `${prefix}${name}_root_link` to `${prefix}${name}_link`.
-inertial_elements (S): inertia tensor of the fork mesh, associated to `${prefix}${name}_root_link`
-    and expressed in that same link frame. Values must correspond to the real body mass
-    (i.e., already scaled to the real mass), not raw values computed with rho=1
-    (rho is material density in kg/m^3).
-    inertial_elements (S) = 'ixx (R) ixy (R) ixz (R) iyy (R) iyz (R) izz (R)'.
-    If empty, `<xacro:null_inertia/>` is used.
-center_of_mass (S): center of mass position for the inertial origin.
-    center_of_mass (S) = 'x (R) y (R) z (R)'.
-    Must be provided if `inertial_elements` is provided.
-limits (S): prismatic joint limits for `${prefix}${name}_root_joint`.
-    limits (S) = 'lower (R) upper (R) effort (R) velocity (R)'.
-joint_parent_fr_root_fr (S): pose of root frame with respect to `parent_frame`.
-    joint_parent_fr_root_fr (S) = 'x (R) y (R) z (R) roll (R) pitch (R) yaw (R)'.
+This file defines the public `fork_simple` model macro.
+It reuses the generic `fork_simple_links_joints` macro and provides the reference geometry, reference inertial data,
+and scaling rules needed to describe a concrete `fork_simple` instance.
+Reference mesh path:
+robotics_description/meshes/extras/fork_simple/fork_simple.stl
+Companion MeshLab report for that reference mesh:
+robotics_description/meshes/extras/fork_simple/fork_simple_meshlab_geometric_measures.txt
+Inertia-scaling procedure:
+robotics_description/doc/how_to_compute_inertia_w_meshlab.md
+MeshLab works with rho=1 (it does not model a specific material here), so the reference volume and the reference
+inertia tensor stored below correspond to the reference mesh with unit density.
+This macro interprets `scale='sx sy sz'` as a geometric scaling of that reference mesh and of the fork geometry
+derived from it.
+- The mesh sent to visual and collision is scaled through `mesh_scale`.
+- Geometric values such as tine sizes and tine separation are recomputed from the same `sx sy sz`.
+- The center of mass is scaled component-wise from the reference center of mass.
+- The mass scales with volume, which means constant density is assumed across scaled variants.
+- The inertia tensor is recomputed for anisotropic scaling (`sx`, `sy`, `sz` can differ), instead of applying a
+  single scalar factor to the reference tensor.
+The scale `'1.0 1.0 1.0'` reproduces the reference `fork_simple` model.
 -->
-<robot xmlns:xacro="http://www.ros.org/wiki/xacro" xmlns:gz="http://gazebosim.org/schema">
+<robot name="fork_simple" xmlns:xacro="http://www.ros.org/wiki/xacro" xmlns:gz="http://gazebosim.org/schema">
+  <!-- Import the generic links-and-joints implementation used by the concrete fork model wrapper below. -->
+  <xacro:include filename="$(find robotics_description)/urdf/extras/fork_simple/generic_macros/fork_simple_links_joints_macro.xacro"/>
   <xacro:macro name="fork_simple"
-               params="name
+               params="name:='fork_simple'
                        prefix:=''
                        parent_frame
-                       mesh
+                       scale:='1.0 1.0 1.0'
+                       use_inertial:=True
                        color:='0.0 0.0 0.0 1.0'
-                       mass:=''
-                       tine_size:='0.0 0.0 0.0'
-                       tine_separation:='0.0'
-                       tine_union_size_x:=0.0
-                       inertial_elements:=''
-                       center_of_mass:=''
-                       limits:='0.0 0.0 0.0 0.0'
+                       limits:='0.0 0.0 1000.0 1000.0'
                        joint_parent_fr_root_fr">
-    <xacro:include filename="$(find robotics_description)/urdf/common/all_commons.xacro"/>
-    <xacro:if value="${mesh == ''}">
-      ${xacro.fatal("fork_simple macro: mesh must not be empty")}
+    <xacro:property name="scale_seq" value="${scale.split()}"/>
+    <xacro:if value="${len(scale_seq) != 3}">
+      ${xacro.fatal("fork_simple macro: invalid scale. Expected: 'sx sy sz'")}
     </xacro:if>
-    <xacro:property name="tine_size_seq" value="${tine_size.split()}"/>
-    <xacro:if value="${len(tine_size_seq) != 3}">
-      ${xacro.fatal("fork_simple macro: invalid tine_size. Expected: 'sx sy sz'")}
-    </xacro:if>
-    <!-- Convert them from str into float, in case any value intervenes in calculations later on. -->
-    <xacro:property name="tine_size_x"           value="${float(tine_size_seq[0])}"/>
-    <xacro:property name="tine_size_y"           value="${float(tine_size_seq[1])}"/>
-    <xacro:property name="tine_size_z"           value="${float(tine_size_seq[2])}"/>
-    <xacro:property name="tine_separation_val"   value="${float(tine_separation)}"/>
-    <xacro:property name="tine_union_size_x_val" value="${float(tine_union_size_x)}"/>
-    <xacro:if value="${tine_size_x &lt;= 0.0 or tine_size_y &lt;= 0.0 or tine_size_z &lt;= 0.0}">
-      ${xacro.fatal("fork_simple macro: tine_size values must be > 0")}
-    </xacro:if>
-    <xacro:if value="${tine_separation_val &lt; 0.0}">
-      ${xacro.fatal("fork_simple macro: tine_separation must be >= 0")}
-    </xacro:if>
-    <xacro:if value="${tine_union_size_x_val &lt; 0.0}">
-      ${xacro.fatal("fork_simple macro: tine_union_size_x must be >= 0")}
+    <!-- Convert the three scale components to floats so geometry, mass, and inertia can be recomputed from them. -->
+    <xacro:property name="sx" value="${float(scale_seq[0])}"/>
+    <xacro:property name="sy" value="${float(scale_seq[1])}"/>
+    <xacro:property name="sz" value="${float(scale_seq[2])}"/>
+    <xacro:if value="${sx &lt;= 0.0 or sy &lt;= 0.0 or sz &lt;= 0.0}">
+      ${xacro.fatal("fork_simple macro: scale values must be > 0")}
     </xacro:if>
     <!--
-    Expected mesh frame convention (for STL generated by `fork_simple_stl_generator.py`):
+    Model-specific mesh path (package-relative, without package:// prefix).
+    The reference mesh frame is expected to follow the generator convention:
     - Origin: rear face of the tine union, centered in Y, on the bottom plane.
     - +X: from the rear union plate toward the tine tips.
     - +Y: side where the left tine is built (right tine is mirrored to -Y).
     - +Z: upward.
-    This frame placement is appropriate for robot integration with parent-frame offsets (typically defined in
-    model-specific wrappers through `joint_parent_fr_root_fr`), so visual and collision mesh origins are kept as
-    identity transforms: xyz="0 0 0", rpy="0 0 0".
+    Therefore, when integrating this fork model on a robot, `joint_parent_fr_root_fr` must be chosen
+    consistently with that frame convention.
     -->
-    <link name="${prefix}${name}_root_link">
-      <visual>
-        <geometry>
-          <mesh filename="package://${mesh}" scale="1.0 1.0 1.0"/>
-        </geometry>
-        <origin rpy="0 0 0" xyz="0 0 0"/>
-        <material name="${prefix}${name}_color">
-          <color rgba="${color}"/>
-        </material>
-      </visual>
-      <collision>
-        <geometry>
-          <mesh filename="package://${mesh}" scale="1.0 1.0 1.0"/>
-        </geometry>
-        <origin rpy="0 0 0" xyz="0 0 0"/>
-      </collision>
-      <xacro:if value="${inertial_elements != ''}">
-        <xacro:property name="inertia_seq" value="${inertial_elements.split()}"/>
-        <xacro:property name="com_seq" value="${center_of_mass.split()}"/>
-        <xacro:if value="${len(inertia_seq) != 6}">
-          ${xacro.fatal("fork_simple macro: invalid inertial_elements. Expected: 'ixx ixy ixz iyy iyz izz'")}
-        </xacro:if>
-        <xacro:if value="${len(com_seq) != 3}">
-          ${xacro.fatal("fork_simple macro: invalid center_of_mass. Expected: 'x y z'")}
-        </xacro:if>
-        <xacro:if value="${mass == ''}">
-          ${xacro.fatal("fork_simple macro: mass must be provided when inertial_elements are provided")}
-        </xacro:if>
-        <xacro:if value="${float(mass) &lt;= 0.0}">
-          ${xacro.fatal("fork_simple macro: mass must be > 0 when inertial_elements are provided")}
-        </xacro:if>
-        <inertial>
-          <mass value="${mass}"/>
-          <inertia ixx="${inertia_seq[0]}" ixy="${inertia_seq[1]}" ixz="${inertia_seq[2]}"
-                   iyy="${inertia_seq[3]}" iyz="${inertia_seq[4]}"
-                   izz="${inertia_seq[5]}"/>
-          <origin rpy="0 0 0" xyz="${com_seq[0]} ${com_seq[1]} ${com_seq[2]}"/>
-        </inertial>
-      </xacro:if>
-      <xacro:if value="${inertial_elements == ''}">
-        <xacro:null_inertia/>
-      </xacro:if>
-    </link>
-    <xacro:property name="limits_seq" value="${limits.split()}"/>
-    <xacro:if value="${len(limits_seq) != 4}">
-      ${xacro.fatal("fork_simple macro: invalid limits. Expected: 'lower upper effort velocity'")}
+    <xacro:property name="mesh" value="robotics_description/meshes/extras/fork_simple/fork_simple.stl"/>
+    <xacro:property name="mesh_scale" value="${sx} ${sy} ${sz}"/>
+    <!--
+    Reference geometry constants (meters), matching the reference mesh generator inputs.
+    These values are scaled below with `sx`, `sy`, and `sz` before they are passed to the generic links-and-joints
+    macro.
+    -->
+    <xacro:property name="tine_size_x_ref"       value="1.20"/>
+    <xacro:property name="tine_size_y_ref"       value="0.12"/>
+    <xacro:property name="tine_size_z_ref"       value="0.06"/>
+    <xacro:property name="tine_separation_ref"   value="0.25"/>
+    <xacro:property name="tine_union_size_x_ref" value="0.03"/>
+    <xacro:property name="tine_size_x"       value="${sx * tine_size_x_ref}"/>
+    <xacro:property name="tine_size_y"       value="${sy * tine_size_y_ref}"/>
+    <xacro:property name="tine_size_z"       value="${sz * tine_size_z_ref}"/>
+    <xacro:property name="tine_size"         value="${tine_size_x} ${tine_size_y} ${tine_size_z}"/>
+    <xacro:property name="tine_separation"   value="${sy * tine_separation_ref}"/>
+    <xacro:property name="tine_union_size_x" value="${sx * tine_union_size_x_ref}"/>
+    <!-- Path for simulation setups where inertial data is intentionally disabled. -->
+    <xacro:unless value="${use_inertial}">
+      <xacro:fork_simple_links_joints name="${name}"
+                                      prefix="${prefix}"
+                                      parent_frame="${parent_frame}"
+                                      mesh="${mesh}"
+                                      mesh_scale="${mesh_scale}"
+                                      color="${color}"
+                                      tine_size="${tine_size}"
+                                      tine_separation="${tine_separation}"
+                                      tine_union_size_x="${tine_union_size_x}"
+                                      limits="${limits}"
+                                      joint_parent_fr_root_fr="${joint_parent_fr_root_fr}"/>
+    </xacro:unless>
+    <!-- Inertial path: scale the reference fork geometry, mass, center of mass, and inertia tensor consistently. -->
+    <xacro:if value="${use_inertial}">
+      <!--
+      The reference mesh was measured in MeshLab with rho=1, so the stored volume and inertia tensor below are
+      unit-density reference values. The physical reference model used in this macro has a real mass of 100 kg at
+      scale 1.0. Therefore, the real material density used for all scaled variants is:
+        density = mass_ref_real / mesh_volume_ref
+      Once `sx`, `sy`, and `sz` are known:
+      - volume scales as `sx * sy * sz`
+      - center of mass scales component-wise
+      - second moments and products of inertia are recomputed with the anisotropic-scaling factors
+      - the resulting rho=1 inertia tensor is multiplied by `density` to obtain the real inertia tensor
+      -->
+      <xacro:property name="mass_ref_real"        value="100.0"/>
+      <xacro:property name="center_of_mass_ref_x" value="0.571591"/>
+      <xacro:property name="center_of_mass_ref_y" value="0.000000"/>
+      <xacro:property name="center_of_mass_ref_z" value="0.031427"/>
+      <xacro:property name="mesh_volume_ref"      value="0.018162"/>
+      <xacro:property name="density_scale"        value="${mass_ref_real / mesh_volume_ref}"/>
+      <xacro:property name="mesh_volume"          value="${mesh_volume_ref * sx * sy * sz}"/>
+      <xacro:property name="mass"                 value="${mass_ref_real * sx * sy * sz}"/>
+      <xacro:property name="center_of_mass_x"     value="${sx * center_of_mass_ref_x}"/>
+      <xacro:property name="center_of_mass_y"     value="${sy * center_of_mass_ref_y}"/>
+      <xacro:property name="center_of_mass_z"     value="${sz * center_of_mass_ref_z}"/>
+      <xacro:property name="center_of_mass"       value="${center_of_mass_x} ${center_of_mass_y} ${center_of_mass_z}"/>
+      <xacro:property name="ixx_ref" value="0.000637"/>
+      <xacro:property name="ixy_ref" value="0.000000"/>
+      <xacro:property name="ixz_ref" value="0.000014"/>
+      <xacro:property name="iyy_ref" value="0.002368"/>
+      <xacro:property name="iyz_ref" value="0.000000"/>
+      <xacro:property name="izz_ref" value="0.002991"/>
+      <!-- Recover the reference second moments from the reference inertia tensor. -->
+      <xacro:property name="jx_ref" value="${0.5 * (iyy_ref + izz_ref - ixx_ref)}"/>
+      <xacro:property name="jy_ref" value="${0.5 * (ixx_ref + izz_ref - iyy_ref)}"/>
+      <xacro:property name="jz_ref" value="${0.5 * (ixx_ref + iyy_ref - izz_ref)}"/>
+      <!-- Scale the rho=1 second moments and products of inertia for the anisotropic scaling `sx sy sz`. -->
+      <xacro:property name="jx_scaled_ref"  value="${(sx ** 3) * sy * sz * jx_ref}"/>
+      <xacro:property name="jy_scaled_ref"  value="${sx * (sy ** 3) * sz * jy_ref}"/>
+      <xacro:property name="jz_scaled_ref"  value="${sx * sy * (sz ** 3) * jz_ref}"/>
+      <xacro:property name="ixy_scaled_ref" value="${(sx ** 2) * (sy ** 2) * sz * ixy_ref}"/>
+      <xacro:property name="ixz_scaled_ref" value="${(sx ** 2) * sy * (sz ** 2) * ixz_ref}"/>
+      <xacro:property name="iyz_scaled_ref" value="${sx * (sy ** 2) * (sz ** 2) * iyz_ref}"/>
+      <!-- Rebuild the scaled rho=1 inertia tensor and then convert it to the real fork mass using `density_scale`. -->
+      <xacro:property name="ixx_scaled_ref" value="${jy_scaled_ref + jz_scaled_ref}"/>
+      <xacro:property name="iyy_scaled_ref" value="${jx_scaled_ref + jz_scaled_ref}"/>
+      <xacro:property name="izz_scaled_ref" value="${jx_scaled_ref + jy_scaled_ref}"/>
+      <xacro:property name="ixx" value="${density_scale * ixx_scaled_ref}"/>
+      <xacro:property name="ixy" value="${density_scale * ixy_scaled_ref}"/>
+      <xacro:property name="ixz" value="${density_scale * ixz_scaled_ref}"/>
+      <xacro:property name="iyy" value="${density_scale * iyy_scaled_ref}"/>
+      <xacro:property name="iyz" value="${density_scale * iyz_scaled_ref}"/>
+      <xacro:property name="izz" value="${density_scale * izz_scaled_ref}"/>
+      <xacro:property name="inertial_elements" value="${ixx} ${ixy} ${ixz} ${iyy} ${iyz} ${izz}"/>
+      <xacro:fork_simple_links_joints name="${name}"
+                                      prefix="${prefix}"
+                                      parent_frame="${parent_frame}"
+                                      mesh="${mesh}"
+                                      mesh_scale="${mesh_scale}"
+                                      color="${color}"
+                                      mass="${mass}"
+                                      tine_size="${tine_size}"
+                                      tine_separation="${tine_separation}"
+                                      tine_union_size_x="${tine_union_size_x}"
+                                      inertial_elements="${inertial_elements}"
+                                      center_of_mass="${center_of_mass}"
+                                      limits="${limits}"
+                                      joint_parent_fr_root_fr="${joint_parent_fr_root_fr}"/>
     </xacro:if>
-    <xacro:property name="lower_limit"    value="${float(limits_seq[0])}"/>
-    <xacro:property name="upper_limit"    value="${float(limits_seq[1])}"/>
-    <xacro:property name="effort_limit"   value="${float(limits_seq[2])}"/>
-    <xacro:property name="velocity_limit" value="${float(limits_seq[3])}"/>
-    <xacro:if value="${lower_limit > upper_limit}">
-      ${xacro.fatal("fork_simple macro: lower_limit must be &lt;= upper_limit")}
-    </xacro:if>
-    <xacro:if value="${effort_limit &lt;= 0.0 or velocity_limit &lt;= 0.0}">
-      ${xacro.fatal("fork_simple macro: effort_limit and velocity_limit must be > 0")}
-    </xacro:if>
-    <xacro:property name="j" value="${joint_parent_fr_root_fr.split()}"/>
-    <xacro:if value="${len(j) != 6}">
-      ${xacro.fatal("fork_simple macro: invalid joint_parent_fr_root_fr. Expected: 'x y z roll pitch yaw'")}
-    </xacro:if>
-    <joint name="${prefix}${name}_root_joint" type="prismatic">
-      <parent link="${parent_frame}"/>
-      <child link="${prefix}${name}_root_link"/>
-      <origin rpy="${j[3]} ${j[4]} ${j[5]}" xyz="${j[0]} ${j[1]} ${j[2]}"/>
-      <axis xyz="0 0 1"/>
-      <limit lower="${lower_limit}"
-             upper="${upper_limit}"
-             effort="${effort_limit}"
-             velocity="${velocity_limit}"/>
-    </joint>
-    <link name="${prefix}${name}_link">
-        <xacro:null_inertia/>
-    </link>
-    <joint name="${prefix}${name}_joint" type="fixed">
-      <parent link="${prefix}${name}_root_link"/>
-      <child link="${prefix}${name}_link"/>
-      <origin rpy="0 0 0" xyz="${tine_union_size_x_val} 0 ${tine_size_z}"/>
-    </joint>
-    <link name="${prefix}${name}_left_tine_link">
-        <xacro:null_inertia/>
-    </link>
-    <joint name="${prefix}${name}_left_tine_joint" type="fixed">
-      <parent link="${prefix}${name}_link"/>
-      <child link="${prefix}${name}_left_tine_link"/>
-      <origin rpy="0 0 0" xyz="${tine_size_x/2} ${tine_separation_val/2 + tine_size_y/2} 0"/>
-    </joint>
-    <link name="${prefix}${name}_right_tine_link">
-        <xacro:null_inertia/>
-    </link>
-    <joint name="${prefix}${name}_right_tine_joint" type="fixed">
-      <parent link="${prefix}${name}_link"/>
-      <child link="${prefix}${name}_right_tine_link"/>
-      <origin rpy="0 0 0" xyz="${tine_size_x/2} ${-tine_separation_val/2 - tine_size_y/2} 0"/>
-    </joint>
   </xacro:macro>
 </robot>
