Commit message: feat(robotics_description): update fork and lidar descriptions
Replace the old scaled fork_simple description with the current fixed-dimension fork model and add the associated tine meshes.

Refresh the Robosense Airy and RealSense helper macros, rename the Hokuyo xacro entrypoint, and add the Sick S300 description assets and example configuration files needed by the updated robot packages.

File: urdf/sensors/cameras/realsense_d435_links_joints_macro.xacro (robot description, xacro)
@@ -49,5 +49,5 @@
                        use_inertial:=True
                        use_v_mesh:=True
-                       color:='0.5 0.5 0.5 1.0'
+                       color:=''
                        use_c_mesh:=False
                        use_sensor_frames_and_joints

File: urdf/sensors/cameras/realsense_d435_rgbd_macro.xacro (robot description, xacro)
@@ -125,5 +125,5 @@
                        use_inertial:=True
                        use_v_mesh:=True
-                       color:='0.5 0.5 0.5 1.0'
+                       color:=''
                        use_c_mesh:=False
                        use_sensor_frames_and_joints

File: urdf/sensors/lidars/robosense_airy_macro.xacro (robot description, xacro)
@@ -159,5 +159,5 @@
     -->
     <xacro:property name="low_res_mesh"
-                    value="robotics_description/meshes/sensors/lidars/robosense_airy/mesh_low_res.dae"/>
+                    value="robotics_description/meshes/sensors/lidars/robosense_airy/mesh_low_res.stl"/>
     <!-- Scale for both meshes, standard mesh and low resolition mesh -->
     <xacro:property name="mesh_scale" value="1.0 1.0 1.0"/>

Commit message: refactor(robotics_description): update fork_simple carriage geometry
Rename the carriage length argument to carriage_size_x and express the\ncarriage and mast geometry from the new carriage frame.\n\nKeep the macro behavior aligned with the fork modules that mount sensors\nrelative to the carriage link.

File: urdf/extras/fork_simple/fork_simple_macro.xacro (robot description, xacro)
@@ -43,35 +43,76 @@
                        color:=''
                        use_c_mesh:=False
-                       carriage_len_x:='0.03'
-                       carriage_len_y
+                       carriage_size_x:='0.03'
                        limits:='0.0 0.0 1000.0 1000.0'
                        joint_parent_fr_root_fr">
     <xacro:property name="tine_mesh"
                     value="robotics_description/meshes/extras/fork_tine/basic_open_tine_120.stl"/>
-    <xacro:property name="tine_size_x"     value="1.20"/>
-    <xacro:property name="tine_size_y"     value="0.12"/>
-    <xacro:property name="tine_size_z"     value="0.06"/>
-    <xacro:property name="tine_separation" value="0.25"/>
-    <xacro:property name="tine_mass"       value="20.0"/>
-    <xacro:property name="min_carriage_len_y"
-                    value="${tine_separation + (2 * tine_size_y)}"/>
+    <xacro:property name="tine_size_x"        value="1.20"/>
+    <xacro:property name="tine_size_y"        value="0.12"/>
+    <xacro:property name="tine_size_z"        value="0.06"/>
+    <xacro:property name="tine_separation"    value="0.25"/>
+    <xacro:property name="tine_mass"          value="20.0"/>
+    <!--
+    The carriage is the part that joints the tines.
+    Carriage and tines move vertically together along the left and righ mast.
+    -->
+    <xacro:property name="carriage_size_y" value="${tine_separation}"/>
+    <xacro:property name="carriage_size_z" value="${tine_size_z}"/>
     <xacro:property name="v_color" value="${(prefix + name + '_color ' + color) if color != '' else ''}"/>
-    <xacro:if value="${float(carriage_len_x) &lt;= 0.0}">
-      ${xacro.fatal("fork_simple macro: carriage_len_x must be > 0")}
-    </xacro:if>
-    <xacro:if value="${float(carriage_len_y) &lt; min_carriage_len_y}">
-      ${xacro.fatal("fork_simple macro: carriage_len_y must be at least tine_separation + 2*tine_size_y")}
-    </xacro:if>
-    <!--
-    Use 20 kg when `carriage_len_y == min_carriage_len_y`.
-    For larger carriage widths, scale the carriage mass linearly with `carriage_len_y`.
-    -->
-    <xacro:property name="carriage_mass" value="${20.0 * (float(carriage_len_y) / min_carriage_len_y)}"/>
-    <!--
-    Use 10 kg when `carriage_len_x == 0.06`.
-    For larger or smaller carriage lengths, scale the tine-stop mass linearly with
-    `carriage_len_x`.
-    -->
-    <xacro:property name="tine_stop_mass" value="${10.0 * (float(carriage_len_x) / 0.06)}"/>
+    <xacro:if value="${float(carriage_size_x) &lt;= 0.0}">
+      ${xacro.fatal("fork_simple macro: carriage_size_x must be > 0")}
+    </xacro:if>
+    <!--
+    Compute the carriage's mass in a simple way, just proportional to its len_x, so that a 0.03 m
+    long carriage has a mass of 20 kg, which is reasonable for a steel box of that size.
+    -->
+    <xacro:property name="carriage_mass" value="${20.0 * (float(carriage_size_x) / 0.03)}"/>
+    <!--
+    Check limits for the prismatic joint.
+    -->
+    <xacro:property name="limits_seq" value="${limits.split()}"/>
+    <xacro:if value="${len(limits_seq) != 4}">
+      ${xacro.fatal("fork_simple macro: invalid limits. Expected: 'lower upper velocity effort'")}
+    </xacro:if>
+    <xacro:property name="lower_limit"    value="${limits_seq[0]}"/>
+    <xacro:property name="upper_limit"    value="${limits_seq[1]}"/>
+    <xacro:property name="velocity_limit" value="${limits_seq[2]}"/>
+    <xacro:property name="effort_limit"   value="${limits_seq[3]}"/>
+    <!--
+    Lower limit for the fork joint must be less than or equal to upper limit.
+    Limits must satisfy lower <= 0 <= upper so that the joint can be initialized at its rest
+    position (q=0) without violating the range motion.
+    If lower > 0, then q=0 is outside the motion limits and the fork will be initialized in an
+    invalid configuration.
+    If upper < 0, then q=0 is outside the motion limits and the fork will be initialized in an
+    invalid configuration too.
+    -->
+    <xacro:if value="${lower_limit > upper_limit}">
+      ${xacro.fatal("fork_simple macro: lower_limit must be &lt;= upper_limit")}
+    </xacro:if>
+    <xacro:if value="${lower_limit > 0.0 or upper_limit &lt; 0.0}">
+      ${xacro.fatal("xacro arg fork_limits must satisfy lower &lt;= 0 &lt;= upper, so q=0 is valid")}
+    </xacro:if>
+    <xacro:if value="${effort_limit &lt;= 0.0 or velocity_limit &lt;= 0.0}">
+      ${xacro.fatal("fork_simple macro: effort_limit and velocity_limit must be > 0")}
+    </xacro:if>
+    <!--
+    A mast is the vertical row along with the carriage moves.
+    There are two mast, left and right.
+    -->
+    <xacro:property name="mast_size_x" value="${carriage_size_x}"/>
+    <xacro:property name="mast_size_y" value="${tine_size_y}"/>
+    <!--
+    After the checks on the limits above, we know that `upper_limit - lower_limit` is positive and
+    represents the total vertical travel of the fork, so we can use it as the mast's size in z to
+    cover the whole vertical travel of the fork.
+    -->
+    <xacro:property name="mast_size_z" value="${upper_limit - lower_limit}"/>
+    <!--
+    Compute the mass of each mast in a simple way, just proportional to its size in z, so that a 1 m
+    long mast has a mass of 10 kg.
+    mass = 10 kg * (size_z / 1 m) = 10 kg * size_z
+    -->
+    <xacro:property name="mast_mass" value="${10.0 * mast_size_z}"/>
     <link name="${prefix}${name}_root_link">
       <xacro:null_inertia/>
@@ -86,18 +127,12 @@
       <origin rpy="${j[3]} ${j[4]} ${j[5]}" xyz="${j[0]} ${j[1]} ${j[2]}"/>
     </joint>
-    <!--
-    The carriage is the part moved by the prismatic joint.
-    Both tine links and both tine-stop links are attached to the carriage with fixed
-    joints, so they move together with the carriage.
-    -->
-    <xacro:property name="carriage_len_z" value="${tine_size_z}"/>
-    <xacro:property name="carriage_origin_x" value="${0.5 * carriage_len_x}"/>
+    <xacro:property name="carriage_origin_x" value="${-0.5 * float(carriage_size_x)}"/>
     <xacro:property name="carriage_origin_y" value="0"/>
-    <xacro:property name="carriage_origin_z" value="${0.5 * tine_size_z}"/>
+    <xacro:property name="carriage_origin_z" value="${-0.5 * carriage_size_z}"/>
     <link name="${prefix}${name}_carriage_link">
       <xacro:if value="${use_visual}">
         <visual>
           <geometry>
-            <box size="${carriage_len_x} ${carriage_len_y} ${carriage_len_z}"/>
+            <box size="${carriage_size_x} ${carriage_size_y} ${carriage_size_z}"/>
           </geometry>
           <origin rpy="0 0 0" xyz="${carriage_origin_x} ${carriage_origin_y} ${carriage_origin_z}"/>
@@ -112,5 +147,5 @@
         <collision>
           <geometry>
-            <box size="${carriage_len_x} ${carriage_len_y} ${carriage_len_z}"/>
+            <box size="${carriage_size_x} ${carriage_size_y} ${carriage_size_z}"/>
           </geometry>
           <origin rpy="0 0 0" xyz="${carriage_origin_x} ${carriage_origin_y} ${carriage_origin_z}"/>
@@ -118,6 +153,6 @@
       </xacro:if>
       <xacro:if value="${use_inertial}">
-        <xacro:solid_box_inertial mass="${carriage_mass}"
-                                  size="${carriage_len_x} ${carriage_len_y} ${carriage_len_z}"
+        <xacro:solid_box_inertia mass="${carriage_mass}"
+                                  size="${carriage_size_x} ${carriage_size_y} ${carriage_size_z}"
                                   origin="${carriage_origin_x} ${carriage_origin_y} ${carriage_origin_z} 0 0 0"/>
       </xacro:if>
@@ -126,22 +161,11 @@
       </xacro:unless>
     </link>
-    <xacro:property name="limits_seq" value="${limits.split()}"/>
-    <xacro:if value="${len(limits_seq) != 4}">
-      ${xacro.fatal("fork_simple macro: invalid limits. Expected: 'lower upper velocity effort'")}
-    </xacro:if>
-    <xacro:property name="lower_limit"    value="${float(limits_seq[0])}"/>
-    <xacro:property name="upper_limit"    value="${float(limits_seq[1])}"/>
-    <xacro:property name="velocity_limit" value="${float(limits_seq[2])}"/>
-    <xacro:property name="effort_limit"   value="${float(limits_seq[3])}"/>
-    <xacro:if value="${lower_limit > upper_limit}">
-      ${xacro.fatal("fork_simple macro: lower_limit must be &lt;= upper_limit")}
-    </xacro:if>
-    <xacro:if value="${effort_limit &lt;= 0.0 or velocity_limit &lt;= 0.0}">
-      ${xacro.fatal("fork_simple macro: effort_limit and velocity_limit must be > 0")}
-    </xacro:if>
+    <xacro:property name="carriage_mount_x" value="${carriage_size_x}"/>
+    <xacro:property name="carriage_mount_y" value="0"/>
+    <xacro:property name="carriage_mount_z" value="${carriage_size_z}"/>
     <joint name="${prefix}${name}_carriage_joint" type="prismatic">
       <parent link="${prefix}${name}_root_link"/>
       <child link="${prefix}${name}_carriage_link"/>
-      <origin rpy="0 0 0" xyz="0 0 0"/>
+      <origin rpy="0 0 0" xyz="${carriage_mount_x} ${carriage_mount_y} ${carriage_mount_z}"/>
       <axis xyz="0 0 1"/>
       <limit lower="${lower_limit}"
@@ -150,18 +174,11 @@
              velocity="${velocity_limit}"/>
     </joint>
-    <!-- Left tine-stop link. This is the rear stop box for the left tine. -->
-    <xacro:property name="tine_stop_len_x" value="${carriage_len_x}"/>
-    <xacro:property name="tine_stop_len_y" value="${tine_size_y}"/>
-    <xacro:property name="tine_stop_len_z" value="${2 * tine_size_z}"/>
-    <xacro:property name="tine_stop_origin_x" value="${-0.5 * tine_stop_len_x}"/>
-    <xacro:property name="tine_stop_origin_y" value="0"/>
-    <xacro:property name="tine_stop_origin_z" value="0"/>
-    <link name="${prefix}${name}_left_tine_stop_link">
+    <link name="${prefix}${name}_left_mast_link">
       <xacro:if value="${use_visual}">
         <visual>
           <geometry>
-            <box size="${tine_stop_len_x} ${tine_stop_len_y} ${tine_stop_len_z}"/>
-          </geometry>
-          <origin rpy="0 0 0" xyz="${tine_stop_origin_x} ${tine_stop_origin_y} ${tine_stop_origin_z}"/>
+            <box size="${mast_size_x} ${mast_size_y} ${mast_size_z}"/>
+          </geometry>
+          <origin rpy="0 0 0" xyz="0 0 0"/>
           <xacro:if value="${color != ''}">
             <material name="${prefix}${name}_color">
@@ -174,25 +191,28 @@
         <collision>
           <geometry>
-            <box size="${tine_stop_len_x} ${tine_stop_len_y} ${tine_stop_len_z}"/>
-          </geometry>
-          <origin rpy="0 0 0" xyz="${tine_stop_origin_x} ${tine_stop_origin_y} ${tine_stop_origin_z}"/>
+            <box size="${mast_size_x} ${mast_size_y} ${mast_size_z}"/>
+          </geometry>
+          <origin rpy="0 0 0" xyz="0 0 0"/>
         </collision>
       </xacro:if>
       <xacro:if value="${use_inertial}">
-        <xacro:solid_box_inertial mass="${tine_stop_mass}"
-                                  size="${tine_stop_len_x} ${tine_stop_len_y} ${tine_stop_len_z}"
-                                  origin="${tine_stop_origin_x} ${tine_stop_origin_y} ${tine_stop_origin_z} 0 0 0"/>
-      </xacro:if>
-      <xacro:unless value="${use_inertial}">
-        <xacro:null_inertia/>
-      </xacro:unless>
-    </link>
-    <xacro:property name="tine_stop_mount_x" value="${carriage_len_x}"/>
-    <xacro:property name="tine_stop_mount_y" value="${0.5*(tine_separation + tine_size_y)}"/>
-    <xacro:property name="tine_stop_mount_z" value="${2*tine_size_z}"/>
-    <joint name="${prefix}${name}_left_tine_stop_joint" type="fixed">
-      <parent link="${prefix}${name}_carriage_link"/>
-      <child link="${prefix}${name}_left_tine_stop_link"/>
-      <origin rpy="0 0 0" xyz="${tine_stop_mount_x} ${tine_stop_mount_y} ${tine_stop_mount_z}"/>
+        <xacro:solid_box_inertia mass="${mast_mass}"
+                                  size="${mast_size_x} ${mast_size_y} ${mast_size_z}"
+                                  origin="0 0 0 0 0 0"/>
+      </xacro:if>
+      <xacro:unless value="${use_inertial}">
+        <xacro:null_inertia/>
+      </xacro:unless>
+    </link>
+    <xacro:property name="left_mast_mount_x" value="${0.5 * mast_size_x}"/>
+    <xacro:property name="left_mast_mount_y" value="${0.5*(tine_separation + tine_size_y)}"/>
+    <!--
+    Remember after the checks on the limits above, we know lower_limit <= 0 <= upper_limit.
+    -->
+    <xacro:property name="left_mast_mount_z" value="${lower_limit + (0.5 * mast_size_z)}"/>
+    <joint name="${prefix}${name}_left_mast_joint" type="fixed">
+      <parent link="${prefix}${name}_root_link"/>
+      <child link="${prefix}${name}_left_mast_link"/>
+      <origin rpy="0 0 0" xyz="${left_mast_mount_x} ${left_mast_mount_y} ${left_mast_mount_z}"/>
     </joint>
     <!-- Left tine link. This is the main load-bearing tine geometry. -->
@@ -217,5 +237,5 @@
       </xacro:if>
       <xacro:if value="${use_inertial}">
-        <xacro:solid_box_inertial mass="${tine_mass}"
+        <xacro:solid_box_inertia mass="${tine_mass}"
                                   size="${tine_size_x} ${tine_size_y} ${tine_size_z}"
                                   origin="${tine_origin_x} ${tine_origin_y} ${tine_origin_z} 0 0 0"/>
@@ -225,20 +245,19 @@
       </xacro:unless>
     </link>
-    <xacro:property name="tine_mount_x" value="${tine_stop_mount_x + (0.5 * tine_size_x)}"/>
-    <xacro:property name="tine_mount_y" value="${tine_stop_mount_y}"/>
-    <xacro:property name="tine_mount_z" value="${tine_size_z}"/>
+    <xacro:property name="left_tine_mount_x" value="${0.5 * tine_size_x}"/>
+    <xacro:property name="left_tine_mount_y" value="${left_mast_mount_y}"/>
+    <xacro:property name="left_tine_mount_z" value="0"/>
     <joint name="${prefix}${name}_left_tine_joint" type="fixed">
       <parent link="${prefix}${name}_carriage_link"/>
       <child link="${prefix}${name}_left_tine_link"/>
-      <origin rpy="0 0 0" xyz="${tine_mount_x} ${tine_mount_y} ${tine_mount_z}"/>
-    </joint>
-    <!-- Right tine-stop link. This is the rear stop box for the right tine. -->
-    <link name="${prefix}${name}_right_tine_stop_link">
+      <origin rpy="0 0 0" xyz="${left_tine_mount_x} ${left_tine_mount_y} ${left_tine_mount_z}"/>
+    </joint>
+    <link name="${prefix}${name}_right_mast_link">
       <xacro:if value="${use_visual}">
         <visual>
           <geometry>
-            <box size="${tine_stop_len_x} ${tine_stop_len_y} ${tine_stop_len_z}"/>
-          </geometry>
-          <origin rpy="0 0 0" xyz="${tine_stop_origin_x} ${tine_stop_origin_y} ${tine_stop_origin_z}"/>
+            <box size="${mast_size_x} ${mast_size_y} ${mast_size_z}"/>
+          </geometry>
+          <origin rpy="0 0 0" xyz="0 0 0"/>
           <xacro:if value="${color != ''}">
             <material name="${prefix}${name}_color">
@@ -251,22 +270,25 @@
         <collision>
           <geometry>
-            <box size="${tine_stop_len_x} ${tine_stop_len_y} ${tine_stop_len_z}"/>
-          </geometry>
-          <origin rpy="0 0 0" xyz="${tine_stop_origin_x} ${tine_stop_origin_y} ${tine_stop_origin_z}"/>
+            <box size="${mast_size_x} ${mast_size_y} ${mast_size_z}"/>
+          </geometry>
+          <origin rpy="0 0 0" xyz="0 0 0"/>
         </collision>
       </xacro:if>
       <xacro:if value="${use_inertial}">
-        <xacro:solid_box_inertial mass="${tine_stop_mass}"
-                                  size="${tine_stop_len_x} ${tine_stop_len_y} ${tine_stop_len_z}"
-                                  origin="${tine_stop_origin_x} ${tine_stop_origin_y} ${tine_stop_origin_z} 0 0 0"/>
-      </xacro:if>
-      <xacro:unless value="${use_inertial}">
-        <xacro:null_inertia/>
-      </xacro:unless>
-    </link>
-    <joint name="${prefix}${name}_right_tine_stop_joint" type="fixed">
-      <parent link="${prefix}${name}_carriage_link"/>
-      <child link="${prefix}${name}_right_tine_stop_link"/>
-      <origin rpy="0 0 0" xyz="${tine_stop_mount_x} ${-tine_stop_mount_y} ${tine_stop_mount_z}"/>
+        <xacro:solid_box_inertia mass="${mast_mass}"
+                                  size="${mast_size_x} ${mast_size_y} ${mast_size_z}"
+                                  origin="0 0 0 0 0 0"/>
+      </xacro:if>
+      <xacro:unless value="${use_inertial}">
+        <xacro:null_inertia/>
+      </xacro:unless>
+    </link>
+    <xacro:property name="right_mast_mount_x" value="${left_mast_mount_x}"/>
+    <xacro:property name="right_mast_mount_y" value="${-left_mast_mount_y}"/>
+    <xacro:property name="right_mast_mount_z" value="${left_mast_mount_z}"/>
+    <joint name="${prefix}${name}_right_mast_joint" type="fixed">
+      <parent link="${prefix}${name}_root_link"/>
+      <child link="${prefix}${name}_right_mast_link"/>
+      <origin rpy="0 0 0" xyz="${right_mast_mount_x} ${right_mast_mount_y} ${right_mast_mount_z}"/>
     </joint>
     <!-- Right tine link. This is the main load-bearing tine geometry. -->
@@ -288,5 +310,5 @@
       </xacro:if>
       <xacro:if value="${use_inertial}">
-        <xacro:solid_box_inertial mass="${tine_mass}"
+        <xacro:solid_box_inertia mass="${tine_mass}"
                                   size="${tine_size_x} ${tine_size_y} ${tine_size_z}"
                                   origin="${tine_origin_x} ${tine_origin_y} ${tine_origin_z} 0 0 0"/>
@@ -296,8 +318,11 @@
       </xacro:unless>
     </link>
+    <xacro:property name="right_tine_mount_x" value="${left_tine_mount_x}"/>
+    <xacro:property name="right_tine_mount_y" value="${-left_tine_mount_y}"/>
+    <xacro:property name="right_tine_mount_z" value="${left_tine_mount_z}"/>
     <joint name="${prefix}${name}_right_tine_joint" type="fixed">
       <parent link="${prefix}${name}_carriage_link"/>
       <child link="${prefix}${name}_right_tine_link"/>
-      <origin rpy="0 0 0" xyz="${tine_mount_x} ${-tine_mount_y} ${tine_mount_z}"/>
+      <origin rpy="0 0 0" xyz="${right_tine_mount_x} ${right_tine_mount_y} ${right_tine_mount_z}"/>
     </joint>
   </xacro:macro>
