Commit message: refactor(fork): [0410-02] update simple fork geometry
Add thin bottom plate links to the left and right tines so the fork geometry explicitly represents the lower tine plates.

Change the prismatic joint limit validation to require q = 0 to be at least 5 mm away from both limits. This keeps the spawned joint inside the valid range and preserves a minimum total travel of 1 cm.

File: urdf/extras/fork_simple/fork_simple_macro.xacro (robot description, xacro)
@@ -49,9 +49,10 @@
     <xacro:property name="tine_mesh"
                     value="robotics_description/meshes/extras/fork_tine/basic_open_tine_120.stl"/>
-    <xacro:property name="tine_size_x"        value="1.20"/>
-    <xacro:property name="tine_size_y"        value="0.12"/>
-    <xacro:property name="tine_size_z"        value="0.06"/>
-    <xacro:property name="tine_separation"    value="0.25"/>
-    <xacro:property name="tine_mass"          value="20.0"/>
+    <xacro:property name="tine_size_x"         value="1.20"/>
+    <xacro:property name="tine_size_y"         value="0.12"/>
+    <xacro:property name="tine_size_z"         value="0.06"/>
+    <xacro:property name="tine_separation"     value="0.25"/>
+    <xacro:property name="tine_mass"           value="20.0"/>
+    <xacro:property name="tine_wall_thickness" value="0.001"/>
     <!--
     Check limits for the prismatic joint.
@@ -66,17 +67,14 @@
     <xacro:property name="effort_limit"   value="${limits_seq[3]}"/>
     <!--
-    Lower limit for the fork joint must be less than or equal to upper limit.
-    Limits must satisfy lower <= 0 <= upper so that the joint can be initialized at its rest
-    position (q=0) without violating the range motion.
-    If lower > 0, then q=0 is outside the motion limits and the fork will be initialized in an
-    invalid configuration.
-    If upper < 0, then q=0 is outside the motion limits and the fork will be initialized in an
-    invalid configuration too.
-    -->
-    <xacro:if value="${lower_limit > upper_limit}">
-      ${xacro.fatal("fork_simple macro: lower_limit must be &lt;= upper_limit")}
-    </xacro:if>
-    <xacro:if value="${lower_limit > 0.0 or upper_limit &lt; 0.0}">
-      ${xacro.fatal("xacro arg fork_limits must satisfy lower &lt;= 0 &lt;= upper, so q=0 is valid")}
+    The robot is spawned with this prismatic joint at q = 0. The lower limit must be at least
+    0.005 m below q = 0 and the upper limit must be at least 0.005 m above q = 0.
+    This keeps the spawned joint 5 mm away from each limit and gives the joint at least 1 cm
+    of total motion.
+    -->
+    <xacro:if value="${float(lower_limit) > -0.005}">
+      ${xacro.fatal("fork_simple macro: lower_limit must be &lt;= -0.005 m")}
+    </xacro:if>
+    <xacro:if value="${float(upper_limit) &lt; 0.005}">
+      ${xacro.fatal("fork_simple macro: upper_limit must be >= 0.005 m")}
     </xacro:if>
     <xacro:if value="${effort_limit &lt;= 0.0 or velocity_limit &lt;= 0.0}">
@@ -116,5 +114,5 @@
     -->
     <xacro:property name="carriage_mass"
-                    value="${20.0 * (carriage_size_x * carriage_size_z) / (tine_size_z * tine_size_z))}"/>
+                    value="${20.0 * (carriage_size_x * carriage_size_z) / (tine_size_z * tine_size_z)}"/>
     <!-- At minimum mast_size_x is 0.005 m -->
     <xacro:property name="mast_size_x" value="${carriage_size_x - tine_shank_size_x}"/>
@@ -225,4 +223,48 @@
       <origin rpy="0 0 0" xyz="${left_tine_mount_x} ${left_tine_mount_y} ${left_tine_mount_z}"/>
     </joint>
+    <!-- Bottom plate link for the left tine -->
+    <!--
+    The link is located in the middle of the bottom face of the plate.
+    -->
+    <xacro:property name="tine_bottom_plate_origin_z" value="${0.5 * tine_wall_thickness}"/>
+    <link name="${prefix}${name}_left_tine_bottom_plate_link">
+      <xacro:if value="${use_visual}">
+        <visual>
+          <geometry>
+            <box size="${tine_size_x} ${tine_size_y} ${tine_wall_thickness}"/>
+          </geometry>
+          <origin rpy="0 0 0" xyz="0 0 ${tine_bottom_plate_origin_z}"/>
+          <xacro:if value="${color != ''}">
+            <material name="${prefix}${name}_color">
+              <color rgba="${color}"/>
+            </material>
+          </xacro:if>
+        </visual>
+      </xacro:if>
+      <xacro:if value="${use_collision}">
+        <collision>
+          <geometry>
+            <box size="${tine_size_x} ${tine_size_y} ${tine_wall_thickness}"/>
+          </geometry>
+          <origin rpy="0 0 0" xyz="0 0 ${tine_bottom_plate_origin_z}"/>
+        </collision>
+      </xacro:if>
+      <xacro:if value="${use_inertial}">
+        <xacro:solid_box_inertia mass="${mast_mass}"
+                                  size="${tine_size_x} ${tine_size_y} ${tine_wall_thickness}"
+                                  origin="0 0 ${tine_bottom_plate_origin_z} 0 0 0"/>
+      </xacro:if>
+      <xacro:unless value="${use_inertial}">
+        <xacro:null_inertia/>
+      </xacro:unless>
+    </link>
+    <xacro:property name="left_tine_bottom_plate_mount_x" value="${mast_size_x + (0.5 * tine_size_x)}"/>
+    <xacro:property name="left_tine_bottom_plate_mount_y" value="${0.5*(tine_separation + tine_size_y)}"/>
+    <xacro:property name="left_tine_bottom_plate_mount_z" value="0"/>
+    <joint name="${prefix}${name}_left_tine_bottom_plate_joint" type="fixed">
+      <parent link="${prefix}${name}_root_link"/>
+      <child link="${prefix}${name}_left_tine_bottom_plate_link"/>
+      <origin rpy="0 0 0" xyz="${left_tine_bottom_plate_mount_x} ${left_tine_bottom_plate_mount_y} ${left_tine_bottom_plate_mount_z}"/>
+    </joint>
     <!-- Left tine-shank -->
     <link name="${prefix}${name}_left_tine_shank_link">
@@ -302,7 +344,4 @@
     <xacro:property name="left_mast_mount_x" value="${0.5 * mast_size_x}"/>
     <xacro:property name="left_mast_mount_y" value="${0.5*(tine_separation + mast_size_y)}"/>
-    <!--
-    Remember after the checks on the limits above, we know lower_limit <= 0 <= upper_limit.
-    -->
     <xacro:property name="left_mast_mount_z" value="${lower_limit + (0.5 * mast_size_z)}"/>
     <joint name="${prefix}${name}_left_mast_joint" type="fixed">
@@ -311,5 +350,4 @@
       <origin rpy="0 0 0" xyz="${left_mast_mount_x} ${left_mast_mount_y} ${left_mast_mount_z}"/>
     </joint>
-   -------------------------
     <!-- Right tine link -->
     <xacro:property name="tine_origin_x" value="0"/>
@@ -349,4 +387,48 @@
       <origin rpy="0 0 0" xyz="${right_tine_mount_x} ${right_tine_mount_y} ${right_tine_mount_z}"/>
     </joint>
+    <!-- Bottom plate link for the right tine -->
+    <!--
+    The link is located in the middle of the bottom face of the plate.
+    -->
+    <xacro:property name="tine_bottom_plate_origin_z" value="${0.5 * tine_wall_thickness}"/>
+    <link name="${prefix}${name}_right_tine_bottom_plate_link">
+      <xacro:if value="${use_visual}">
+        <visual>
+          <geometry>
+            <box size="${tine_size_x} ${tine_size_y} ${tine_wall_thickness}"/>
+          </geometry>
+          <origin rpy="0 0 0" xyz="0 0 ${tine_bottom_plate_origin_z}"/>
+          <xacro:if value="${color != ''}">
+            <material name="${prefix}${name}_color">
+              <color rgba="${color}"/>
+            </material>
+          </xacro:if>
+        </visual>
+      </xacro:if>
+      <xacro:if value="${use_collision}">
+        <collision>
+          <geometry>
+            <box size="${tine_size_x} ${tine_size_y} ${tine_wall_thickness}"/>
+          </geometry>
+          <origin rpy="0 0 0" xyz="0 0 ${tine_bottom_plate_origin_z}"/>
+        </collision>
+      </xacro:if>
+      <xacro:if value="${use_inertial}">
+        <xacro:solid_box_inertia mass="${mast_mass}"
+                                  size="${tine_size_x} ${tine_size_y} ${tine_wall_thickness}"
+                                  origin="0 0 ${tine_bottom_plate_origin_z} 0 0 0"/>
+      </xacro:if>
+      <xacro:unless value="${use_inertial}">
+        <xacro:null_inertia/>
+      </xacro:unless>
+    </link>
+    <xacro:property name="right_tine_bottom_plate_mount_x" value="${left_tine_bottom_plate_mount_x}"/>
+    <xacro:property name="right_tine_bottom_plate_mount_y" value="${-left_tine_bottom_plate_mount_y}"/>
+    <xacro:property name="right_tine_bottom_plate_mount_z" value="${left_tine_bottom_plate_mount_z}"/>
+    <joint name="${prefix}${name}_right_tine_bottom_plate_joint" type="fixed">
+      <parent link="${prefix}${name}_root_link"/>
+      <child link="${prefix}${name}_right_tine_bottom_plate_link"/>
+      <origin rpy="0 0 0" xyz="${right_tine_bottom_plate_mount_x} ${right_tine_bottom_plate_mount_y} ${right_tine_bottom_plate_mount_z}"/>
+    </joint>
     <!-- Right tine-shank -->
     <link name="${prefix}${name}_right_tine_shank_link">

Commit message: feat(fork_simple): [0417-01] add optional front closing plates for fork tines
Add configurable front plates to close the U-shaped openings of fork tines.

Changes:
- Add 'tine_open' parameter to fork_simple macro (default: False)
- When tine_open=False, create front closing plates for both tines
- Front plates: 1mm thick, positioned at tine front opening center
- Plate dimensions: tine_size - 2mm (1mm margin per side)
- Plates attached to left_tine_link and right_tine_link respectively
- Bottom plates remain anchored to root_link (don't move with carriage)

The front plates close the open mesh geometry (U-shaped cross-section)
when tines need to be sealed. Set tine_open=True to leave tines open.

File: urdf/extras/fork_simple/fork_simple_macro.xacro (robot description, xacro)
@@ -43,4 +43,5 @@
                        color:=''
                        use_c_mesh:=False
+                       tine_open:=False
                        carriage_size_x:=0.06
                        carriage_size_z:=0.06
@@ -267,4 +268,50 @@
       <origin rpy="0 0 0" xyz="${left_tine_bottom_plate_mount_x} ${left_tine_bottom_plate_mount_y} ${left_tine_bottom_plate_mount_z}"/>
     </joint>
+    <!-- Front plate link for the left tine (when closed) -->
+    <xacro:unless value="${tine_open}">
+      <xacro:property name="front_tine_plate_size_x" value="${tine_wall_thickness}"/>
+      <xacro:property name="front_tine_plate_size_y" value="${tine_size_y - 2*tine_wall_thickness}"/>
+      <xacro:property name="front_tine_plate_size_z" value="${tine_size_z - 2*tine_wall_thickness}"/>
+      <xacro:property name="front_tine_plate_origin_x" value="${-0.5 * front_tine_plate_size_x}"/>
+      <link name="${prefix}${name}_left_tine_front_plate_link">
+        <xacro:if value="${use_visual}">
+          <visual>
+            <geometry>
+              <box size="${front_tine_plate_size_x} ${front_tine_plate_size_y} ${front_tine_plate_size_z}"/>
+            </geometry>
+            <origin rpy="0 0 0" xyz="${front_tine_plate_origin_x} 0 0"/>
+            <xacro:if value="${color != ''}">
+              <material name="${prefix}${name}_color">
+                <color rgba="${color}"/>
+              </material>
+            </xacro:if>
+          </visual>
+        </xacro:if>
+        <xacro:if value="${use_collision}">
+          <collision>
+            <geometry>
+              <box size="${front_tine_plate_size_x} ${front_tine_plate_size_y} ${front_tine_plate_size_z}"/>
+            </geometry>
+            <origin rpy="0 0 0" xyz="${front_tine_plate_origin_x} 0 0"/>
+          </collision>
+        </xacro:if>
+        <xacro:if value="${use_inertial}">
+          <xacro:solid_box_inertia mass="0.1"
+                                    size="${front_tine_plate_size_x} ${front_tine_plate_size_y} ${front_tine_plate_size_z}"
+                                    origin="${front_tine_plate_origin_x} 0 0 0 0 0"/>
+        </xacro:if>
+        <xacro:unless value="${use_inertial}">
+          <xacro:null_inertia/>
+        </xacro:unless>
+      </link>
+      <xacro:property name="left_tine_front_plate_mount_x" value="${0.5 * tine_size_x}"/>
+      <xacro:property name="left_tine_front_plate_mount_y" value="0"/>
+      <xacro:property name="left_tine_front_plate_mount_z" value="${-0.5 * tine_size_z}"/>
+      <joint name="${prefix}${name}_left_tine_front_plate_joint" type="fixed">
+        <parent link="${prefix}${name}_left_tine_link"/>
+        <child link="${prefix}${name}_left_tine_front_plate_link"/>
+        <origin rpy="0 0 0" xyz="${left_tine_front_plate_mount_x} ${left_tine_front_plate_mount_y} ${left_tine_front_plate_mount_z}"/>
+      </joint>
+    </xacro:unless>
     <!-- Left tine-shank -->
     <link name="${prefix}${name}_left_tine_shank_link">
@@ -431,4 +478,46 @@
       <origin rpy="0 0 0" xyz="${right_tine_bottom_plate_mount_x} ${right_tine_bottom_plate_mount_y} ${right_tine_bottom_plate_mount_z}"/>
     </joint>
+    <!-- Front plate link for the right tine (when closed) -->
+    <xacro:unless value="${tine_open}">
+      <link name="${prefix}${name}_right_tine_front_plate_link">
+        <xacro:if value="${use_visual}">
+          <visual>
+            <geometry>
+              <box size="${front_tine_plate_size_x} ${front_tine_plate_size_y} ${front_tine_plate_size_z}"/>
+            </geometry>
+            <origin rpy="0 0 0" xyz="${front_tine_plate_origin_x} 0 0"/>
+            <xacro:if value="${color != ''}">
+              <material name="${prefix}${name}_color">
+                <color rgba="${color}"/>
+              </material>
+            </xacro:if>
+          </visual>
+        </xacro:if>
+        <xacro:if value="${use_collision}">
+          <collision>
+            <geometry>
+              <box size="${front_tine_plate_size_x} ${front_tine_plate_size_y} ${front_tine_plate_size_z}"/>
+            </geometry>
+            <origin rpy="0 0 0" xyz="${front_tine_plate_origin_x} 0 0"/>
+          </collision>
+        </xacro:if>
+        <xacro:if value="${use_inertial}">
+          <xacro:solid_box_inertia mass="0.1"
+                                    size="${front_tine_plate_size_x} ${front_tine_plate_size_y} ${front_tine_plate_size_z}"
+                                    origin="${front_tine_plate_origin_x} 0 0 0 0 0"/>
+        </xacro:if>
+        <xacro:unless value="${use_inertial}">
+          <xacro:null_inertia/>
+        </xacro:unless>
+      </link>
+      <xacro:property name="right_tine_front_plate_mount_x" value="${left_tine_front_plate_mount_x}"/>
+      <xacro:property name="right_tine_front_plate_mount_y" value="0"/>
+      <xacro:property name="right_tine_front_plate_mount_z" value="${left_tine_front_plate_mount_z}"/>
+      <joint name="${prefix}${name}_right_tine_front_plate_joint" type="fixed">
+        <parent link="${prefix}${name}_right_tine_link"/>
+        <child link="${prefix}${name}_right_tine_front_plate_link"/>
+        <origin rpy="0 0 0" xyz="${right_tine_front_plate_mount_x} ${right_tine_front_plate_mount_y} ${right_tine_front_plate_mount_z}"/>
+      </joint>
+    </xacro:unless>
     <!-- Right tine-shank -->
     <link name="${prefix}${name}_right_tine_shank_link">
