Commit message: feat(sensors): add bridge examples for lidar and imu
Rename the lidar and IMU example simulation files to the new example_<sensor>_simulation.yaml convention and add matching bridge channel examples.

Also align the lidar and IMU set_props helpers with the bridge-driven topic forwarding pattern used by the current robot integrations.

File: urdf/sensors/imus/generic_macros/set_props_plugin_imu_macro.xacro (robot description, xacro)
@@ -3,5 +3,6 @@
   <xacro:macro name="set_props_plugin_imu"
                params="prop_prefix
-                       imu_sim_cfg:=dict()">
+                       imu_sim_cfg:=dict()
+                       imu_bridge_channel_cfg:=dict()">
     <!--
     If imu_sim_cfg does not have the field 'enabled' or if it is set to False, then set all the simulation
@@ -41,4 +42,7 @@
       <xacro:property name="${prop_prefix}_sim_use_orientation"
                       value="False"
+                      scope="parent"/>
+      <xacro:property name="${prop_prefix}_sim_topic"
+                      value=""
                       scope="parent"/>
     </xacro:unless>
@@ -123,4 +127,7 @@
                       value="${imu_sim_cfg['use_orientation']}"
                       scope="parent"/>
+      <xacro:property name="${prop_prefix}_sim_topic"
+                      value="${imu_bridge_channel_cfg.get('gz_topic_name', '')}"
+                      scope="parent"/>
     </xacro:if>
   </xacro:macro>

File: urdf/sensors/lidars/generic_macros/set_props_plugin_lidar_2d_macro.xacro (robot description, xacro)
@@ -4,4 +4,5 @@
                params="prop_prefix
                        lidar_2d_sim_cfg:=dict()
+                       lidar_2d_bridge_channel_cfg:=dict()
                        default_sim_always_on:=True
                        default_sim_visualize:=False
@@ -13,8 +14,8 @@
   <!--
   If lidar_2d_sim_cfg does not have the field 'enabled' or if it is set to False, then set all the simulation
-  properties to disable the simulation of the 3D lidar ring.
+  properties to disable the simulation of the 2D lidar.
   -->
   <xacro:unless value="${lidar_2d_sim_cfg.get('enabled', False)}">
-    <xacro:property name="${prop_prefix}_use_sim"            value="False"                      scope="parent"/>
+    <xacro:property name="${prop_prefix}_sim_enabled"        value="False"                      scope="parent"/>
     <xacro:property name="${prop_prefix}_sim_always_on"      value="False"                      scope="parent"/>
     <xacro:property name="${prop_prefix}_sim_visualize"      value="False"                      scope="parent"/>
@@ -24,4 +25,5 @@
     <xacro:property name="${prop_prefix}_sim_dist_span"      value="dict(min=0, max=0)"         scope="parent"/>
     <xacro:property name="${prop_prefix}_sim_gaussian_noise" value="dict(mean=0.0, stddev=0.0)" scope="parent"/>
+    <xacro:property name="${prop_prefix}_sim_topic"          value=""                           scope="parent"/>
   </xacro:unless>
   <!--
@@ -30,5 +32,5 @@
   -->
   <xacro:if value="${lidar_2d_sim_cfg.get('enabled', False)}">
-    <xacro:property name="${prop_prefix}_use_sim"
+    <xacro:property name="${prop_prefix}_sim_enabled"
                     value="True"
                     scope="parent"/>
@@ -54,4 +56,7 @@
                     value="${lidar_2d_sim_cfg.get('gaussian_noise', default_sim_gaussian_noise)}"
                     scope="parent"/>
+    <xacro:property name="${prop_prefix}_sim_topic"
+                    value="${lidar_2d_bridge_channel_cfg.get('gz_topic_name', '')}"
+                    scope="parent"/>
     </xacro:if>
   </xacro:macro>

File: urdf/sensors/lidars/generic_macros/set_props_plugin_lidar_3d_ring_macro.xacro (robot description, xacro)
@@ -3,5 +3,6 @@
   <xacro:macro name="set_props_plugin_lidar_3d_ring"
                params="prop_prefix
-                       lidar_3d_sim_cfg:=dict()">
+                       lidar_3d_sim_cfg:=dict()
+                       lidar_3d_bridge_channel_cfg:=dict()">
     <!--
     If lidar_3d_sim_cfg does not have the field 'enabled' or if it is set to False, then set all the simulation
@@ -19,4 +20,5 @@
       <xacro:property name="${prop_prefix}_sim_dist_span"      value="0 0"   scope="parent"/>
       <xacro:property name="${prop_prefix}_sim_gaussian_noise" value="0 0"   scope="parent"/>
+      <xacro:property name="${prop_prefix}_sim_topic"          value=""      scope="parent"/>
     </xacro:unless>
     <!--
@@ -63,4 +65,7 @@
                       value="${sim_gaussian_noise['mean']} ${sim_gaussian_noise['stddev']}"
                       scope="parent"/>
+      <xacro:property name="${prop_prefix}_sim_topic"
+                      value="${lidar_3d_bridge_channel_cfg.get('gz_topic_name', '')}"
+                      scope="parent"/>
     </xacro:if>
   </xacro:macro>
