Commit message: refactor(helios): rename the Robosense Helios 16 assets and examples
Rename the Robosense Helios 16 mesh directory, macro references, and
focused xacro test so the visible name consistently uses
`robosense_helios_16`.

Also refresh the package README and test README to document the current
naming and the recommended simulation configuration workflow.

File: test/test_xacros/test_robosense_helios_16.xacro (robot description, xacro)
@@ -1,4 +1,4 @@
 <?xml version="1.0"?>
-<robot name="test_robosense_helios_16p" xmlns:xacro="http://www.ros.org/wiki/xacro">
+<robot name="test_robosense_helios_16" xmlns:xacro="http://www.ros.org/wiki/xacro">
   <xacro:include filename="$(find robotics_description)/urdf/common/all_commons.xacro"/>
   <xacro:include filename="$(find robotics_description)/urdf/sensors/lidars/robosense_helios_16_macro.xacro"/>
@@ -9,5 +9,5 @@
                                         sim_cfg="${sim_cfg}"/>
   <link name="base_link"/>
-  <xacro:robosense_helios_16p name="lidar3d"
+  <xacro:robosense_helios_16 name="lidar3d"
                               parent_frame="base_link"
                               joint_parent_fr_root_fr="0 0 0 0 0 0"

File: urdf/sensors/lidars/robosense_helios_16_macro.xacro (robot description, xacro)
@@ -65,6 +65,6 @@
 namespace.
 -->
-<robot name="robosense_helios_16p" xmlns:xacro="http://www.ros.org/wiki/xacro" xmlns:gz="http://gazebosim.org/schema">
-  <xacro:macro name="robosense_helios_16p"
+<robot name="robosense_helios_16" xmlns:xacro="http://www.ros.org/wiki/xacro" xmlns:gz="http://gazebosim.org/schema">
+  <xacro:macro name="robosense_helios_16"
                params="name
                        prefix:=''
@@ -108,5 +108,5 @@
     -->
     <xacro:property name="mesh"
-                    value="robotics_description/meshes/sensors/lidars/robosense_helios_16p/mesh.stl"/>
+                    value="robotics_description/meshes/sensors/lidars/robosense_helios_16/mesh.stl"/>
     <!--
     The mesh represents a cylinder with its symmetry axis along the z-axis.
@@ -117,5 +117,5 @@
     -->
     <xacro:property name="low_res_mesh"
-                    value="robotics_description/meshes/sensors/lidars/robosense_helios_16p/mesh_low_res.dae"/>
+                    value="robotics_description/meshes/sensors/lidars/robosense_helios_16/mesh_low_res.dae"/>
     <!-- Scale for both meshes, standard mesh and low resolition mesh -->
     <xacro:property name="mesh_scale" value="1.0 1.0 1.0"/>
