Commit message: refactor(gz): [0207-02] rename pose reference macro
Rename the Gazebo OdometryPublisher wrapper macro to plugin_pose_in_reference_frame_publisher so the name describes that the published pose is expressed in a reference frame.

Update the macro file, documentation, aggregate include, and xacro test to use the new public macro name.

File: test/test_xacros/test_gz_system_plugins.xacro (robot description, xacro)
@@ -15,5 +15,5 @@
       initial_linear="0 0 0"
       initial_angular="0 0 0"/>
-    <xacro:plugin_referenced_frame_pose_publisher
+    <xacro:plugin_pose_in_reference_frame_publisher
       reference_frame="map"
       published_robot_frame="base_link"

File: urdf/gz_system_plugins/all_gz_system_plugins.xacro (robot description, xacro)
@@ -13,5 +13,5 @@
   <xacro:include filename="$(find robotics_description)/urdf/gz_system_plugins/plugin_joint_state_publisher_macro.xacro"/>
   <xacro:include filename="$(find robotics_description)/urdf/gz_system_plugins/plugin_linear_battery_macro.xacro"/>
-  <xacro:include filename="$(find robotics_description)/urdf/gz_system_plugins/plugin_referenced_frame_pose_publisher_macro.xacro"/>
+  <xacro:include filename="$(find robotics_description)/urdf/gz_system_plugins/plugin_pose_in_reference_frame_publisher_macro.xacro"/>
   <xacro:include filename="$(find robotics_description)/urdf/gz_system_plugins/plugin_velocity_control_macro.xacro"/>
 </robot>

File: urdf/gz_system_plugins/plugin_pose_in_reference_frame_publisher_macro.xacro (robot description, xacro)
@@ -1,6 +1,6 @@
 <?xml version="1.0"?>
 <!--
-This file defines the macro `plugin_referenced_frame_pose_publisher`.
-The `plugin_referenced_frame_pose_publisher` macro emits the XML for one Gazebo Sim plugin of type
+This file defines the macro `plugin_pose_in_reference_frame_publisher`.
+The `plugin_pose_in_reference_frame_publisher` macro emits the XML for one Gazebo Sim plugin of type
 `gz::sim::systems::OdometryPublisher` attached to a robot model.
 The Gazebo plugin publishes one message of type `gz::msgs::Odometry`, one message of type
@@ -114,7 +114,7 @@
 https://gazebosim.org/api/sim/8/classgz_1_1sim_1_1systems_1_1OdometryPublisher.html
 -->
-<robot name="plugin_referenced_frame_pose_publisher_macro" xmlns:xacro="http://www.ros.org/wiki/xacro"
+<robot name="plugin_pose_in_reference_frame_publisher_macro" xmlns:xacro="http://www.ros.org/wiki/xacro"
        xmlns:gz="http://gazebosim.org/schema">
-  <xacro:macro name="plugin_referenced_frame_pose_publisher"
+  <xacro:macro name="plugin_pose_in_reference_frame_publisher"
                params="reference_frame
                        published_robot_frame
@@ -130,5 +130,5 @@
                        gaussian_noise:=0">
     <xacro:if value="${dimensions not in (2, 3)}">
-      ${xacro.fatal("plugin_referenced_frame_pose_publisher: dimensions must be 2 or 3")}
+      ${xacro.fatal("plugin_pose_in_reference_frame_publisher: dimensions must be 2 or 3")}
     </xacro:if>
     <plugin filename="gz-sim-odometry-publisher-system" name="gz::sim::systems::OdometryPublisher">

Commit message: refactor(gz): [0507-01] rename pose publisher macro
Rename the pose publisher macro and documentation to plugin_pose_publisher_in_reference_frame so the public name reads with pose_publisher as the core concept. Update the aggregate plugin include, README link, and xacro test usage to match the new macro name.

File: test/test_xacros/test_gz_system_plugins.xacro (robot description, xacro)
@@ -15,5 +15,5 @@
       initial_linear="0 0 0"
       initial_angular="0 0 0"/>
-    <xacro:plugin_pose_in_reference_frame_publisher
+    <xacro:plugin_pose_publisher_in_reference_frame
       reference_frame="map"
       robot_frame="base_link"

File: urdf/gz_system_plugins/all_gz_system_plugins.xacro (robot description, xacro)
@@ -13,5 +13,5 @@
   <xacro:include filename="$(find robotics_description)/urdf/gz_system_plugins/plugin_joint_state_publisher_macro.xacro"/>
   <xacro:include filename="$(find robotics_description)/urdf/gz_system_plugins/plugin_linear_battery_macro.xacro"/>
-  <xacro:include filename="$(find robotics_description)/urdf/gz_system_plugins/plugin_pose_in_reference_frame_publisher_macro.xacro"/>
+  <xacro:include filename="$(find robotics_description)/urdf/gz_system_plugins/plugin_pose_publisher_in_reference_frame_macro.xacro"/>
   <xacro:include filename="$(find robotics_description)/urdf/gz_system_plugins/plugin_velocity_control_macro.xacro"/>
 </robot>

File: urdf/gz_system_plugins/plugin_pose_publisher_in_reference_frame_macro.xacro (robot description, xacro)
@@ -1,6 +1,6 @@
 <?xml version="1.0"?>
 <!--
-This file defines the macro `plugin_pose_in_reference_frame_publisher`.
-The `plugin_pose_in_reference_frame_publisher` macro emits the XML for one Gazebo Sim plugin of type
+This file defines the macro `plugin_pose_publisher_in_reference_frame`.
+The `plugin_pose_publisher_in_reference_frame` macro emits the XML for one Gazebo Sim plugin of type
 `gz::sim::systems::OdometryPublisher` attached to a robot model.
 The Gazebo plugin publishes one message of type `gz::msgs::Odometry`, one message of type
@@ -113,7 +113,7 @@
 https://gazebosim.org/api/sim/8/classgz_1_1sim_1_1systems_1_1OdometryPublisher.html
 -->
-<robot name="plugin_pose_in_reference_frame_publisher_macro" xmlns:xacro="http://www.ros.org/wiki/xacro"
+<robot name="plugin_pose_publisher_in_reference_frame_macro" xmlns:xacro="http://www.ros.org/wiki/xacro"
        xmlns:gz="http://gazebosim.org/schema">
-  <xacro:macro name="plugin_pose_in_reference_frame_publisher"
+  <xacro:macro name="plugin_pose_publisher_in_reference_frame"
                params="reference_frame
                        robot_frame
@@ -129,5 +129,5 @@
                        gaussian_noise:=0">
     <xacro:if value="${dimensions not in (2, 3)}">
-      ${xacro.fatal("plugin_pose_in_reference_frame_publisher: dimensions must be 2 or 3")}
+      ${xacro.fatal("plugin_pose_publisher_in_reference_frame: dimensions must be 2 or 3")}
     </xacro:if>
     <plugin filename="gz-sim-odometry-publisher-system" name="gz::sim::systems::OdometryPublisher">
