Commit message: feat(lidars): [2105-01] Add configurable range resolution
Add a dist_res parameter to the generic lidar plugin macros and propagate it through the 2D and 3D lidar set_props and concrete lidar wrappers. This keeps the default range resolution at 0.0 for existing models while allowing simulation YAML files to opt into a linear range resolution.

File: urdf/sensors/lidars/generic_macros/plugin_lidar_2d_macro.xacro (robot description, xacro)
@@ -18,4 +18,5 @@
                        hor_res_deg
                        dist_span
+                       dist_res:=0.0
                        gaussian_noise:='0 0'
                        namespace:=''
@@ -32,4 +33,5 @@
                                 ver_res_deg="1.0"
                                 dist_span="${dist_span}"
+                                dist_res="${dist_res}"
                                 gaussian_noise="${gaussian_noise}"
                                 namespace="${namespace}"

File: urdf/sensors/lidars/generic_macros/plugin_lidar_3d_ring_macro.xacro (robot description, xacro)
@@ -46,4 +46,5 @@
 - ver_res_deg has 1 value.
 - dist_span has 2 values between quotes in this order 'min_dist max_dist'
+- dist_res has 1 value, in meters.
 -->
 <robot name="plugin_lidar_3d_ring" xmlns:xacro="http://www.ros.org/wiki/xacro" xmlns:gz="http://gazebosim.org/schema">
@@ -59,4 +60,5 @@
                        ver_res_deg
                        dist_span
+                       dist_res:=0.0
                        gaussian_noise:='0 0'
                        namespace:=''
@@ -136,6 +138,5 @@
             <min>${min_dist}</min>
             <max>${max_dist}</max>
-            <!-- DO NOT TOUCH, LEAVE IT TO 0.0 -->
-            <resolution>0.0</resolution>
+            <resolution>${dist_res}</resolution>
           </range>
           <noise>

File: urdf/sensors/lidars/generic_macros/set_props_plugin_lidar_2d_macro.xacro (robot description, xacro)
@@ -19,4 +19,5 @@
       <xacro:property name="${prop_prefix}_hor_res_deg"    value="0"     scope="parent"/>
       <xacro:property name="${prop_prefix}_dist_span"      value="0 0"   scope="parent"/>
+      <xacro:property name="${prop_prefix}_dist_res"       value="0.0"   scope="parent"/>
       <xacro:property name="${prop_prefix}_gaussian_noise" value="0 0"   scope="parent"/>
       <xacro:property name="${prop_prefix}_topic"          value=""      scope="parent"/>
@@ -53,4 +54,7 @@
                       value="${sim_dist_span['min_dist']} ${sim_dist_span['max_dist']}"
                       scope="parent"/>
+      <xacro:property name="${prop_prefix}_dist_res"
+                      value="${sim_cfg.get('dist_res', 0.0)}"
+                      scope="parent"/>
       <xacro:property name="sim_gaussian_noise"
                       value="${sim_cfg['gaussian_noise']}"/>

File: urdf/sensors/lidars/generic_macros/set_props_plugin_lidar_3d_ring_macro.xacro (robot description, xacro)
@@ -21,4 +21,5 @@
       <xacro:property name="${prop_prefix}_ver_res_deg"    value="0"     scope="parent"/>
       <xacro:property name="${prop_prefix}_dist_span"      value="0 0"   scope="parent"/>
+      <xacro:property name="${prop_prefix}_dist_res"       value="0.0"   scope="parent"/>
       <xacro:property name="${prop_prefix}_gaussian_noise" value="0 0"   scope="parent"/>
       <xacro:property name="${prop_prefix}_base_topic"     value=""      scope="parent"/>
@@ -63,4 +64,7 @@
                       value="${sim_dist_span['min_dist']} ${sim_dist_span['max_dist']}"
                       scope="parent"/>
+      <xacro:property name="${prop_prefix}_dist_res"
+                      value="${sim_cfg.get('dist_res', 0.0)}"
+                      scope="parent"/>
       <xacro:property name="sim_gaussian_noise"
                       value="${sim_cfg['gaussian_noise']}"/>

File: urdf/sensors/lidars/hokuyo_utm30lx.xacro (robot description, xacro)
@@ -85,4 +85,5 @@
             sim_lidar_hor_res_deg
             sim_lidar_dist_span
+            sim_lidar_dist_res:=0.0
             sim_lidar_gaussian_noise:='0 0'
             namespace:=''
@@ -186,4 +187,5 @@
         hor_res_deg="${sim_lidar_hor_res_deg}"
         dist_span="${sim_lidar_dist_span}"
+        dist_res="${sim_lidar_dist_res}"
         gaussian_noise="${sim_lidar_gaussian_noise}"
         namespace="${namespace}"

File: urdf/sensors/lidars/robosense_airy_macro.xacro (robot description, xacro)
@@ -118,4 +118,5 @@
                        sim_lidar_ver_res_deg
                        sim_lidar_dist_span
+                       sim_lidar_dist_res:=0.0
                        sim_lidar_gaussian_noise:='0 0'
                        sim_imu_enabled:=False
@@ -265,4 +266,5 @@
         ver_res_deg="${sim_lidar_ver_res_deg}"
         dist_span="${sim_lidar_dist_span}"
+        dist_res="${sim_lidar_dist_res}"
         gaussian_noise="${sim_lidar_gaussian_noise}"
         namespace="${namespace}"

File: urdf/sensors/lidars/robosense_helios_16_macro.xacro (robot description, xacro)
@@ -88,4 +88,5 @@
                        sim_ver_res_deg
                        sim_dist_span
+                       sim_dist_res:=0.0
                        sim_gaussian_noise:='0 0'
                        namespace:=''
@@ -194,4 +195,5 @@
         ver_res_deg="${sim_ver_res_deg}"
         dist_span="${sim_dist_span}"
+        dist_res="${sim_dist_res}"
         gaussian_noise="${sim_gaussian_noise}"
         namespace="${namespace}"

File: urdf/sensors/lidars/sick_s300.xacro (robot description, xacro)
@@ -77,4 +77,5 @@
             sim_lidar_hor_res_deg
             sim_lidar_dist_span
+            sim_lidar_dist_res:=0.0
             sim_lidar_gaussian_noise:='0 0'
             namespace:=''
@@ -180,4 +181,5 @@
         hor_res_deg="${sim_lidar_hor_res_deg}"
         dist_span="${sim_lidar_dist_span}"
+        dist_res="${sim_lidar_dist_res}"
         gaussian_noise="${sim_lidar_gaussian_noise}"
         namespace="${namespace}"
