Commit message: fix: make basket colors caller-owned
Remove default visual and Gazebo colors from the new basket macros so robotics_description does not impose presentation choices.

Callers can still pass explicit materials using the existing color_name r g b a contract.
159ce8

File: urdf/extras/basket/basket_macros.xacro (robot description, xacro)
@@ -15,4 +15,5 @@
       joint_parent_fr_basket_fr (S) = 'x y z roll pitch yaw'
   color (S): Optional material in the form '<color_name> r g b a'.
+             If empty, the mesh may use its embedded color.
   -->
   <xacro:macro name="basket_chassis_macro"
@@ -20,5 +21,5 @@
                        parent
                        joint_parent_fr_basket_fr:='0 0 0 0 0 0'
-                       color:='red_color 1.0 0.0 0.0 1.0'">
+                       color:=''">
     <joint name="${prefix}basket_chassis_joint" type="fixed">
       <axis xyz="0 1 0"/>
@@ -33,5 +34,4 @@
     </link>
     <gazebo reference="${prefix}basket_chassis_link">
-      <material>Gazebo/Red</material>
       <gravity>true</gravity>
     </gazebo>
@@ -42,4 +42,5 @@
       joint_parent_fr_container_fr (S) = 'x y z roll pitch yaw'
   color (S): Optional material in the form '<color_name> r g b a'.
+             If empty, the mesh may use its embedded color.
   -->
   <xacro:macro name="basket_container_macro"
@@ -47,5 +48,5 @@
                        parent
                        joint_parent_fr_container_fr:='-0.068 0 0.013 0 0 0'
-                       color:='alu_color 0.1 0.1 0.1 1.0'">
+                       color:=''">
     <joint name="${prefix}basket_container_joint" type="fixed">
       <axis xyz="0 1 0"/>
@@ -60,5 +61,4 @@
     </link>
     <gazebo reference="${prefix}basket_container_link">
-      <material>Gazebo/Red</material>
       <gravity>true</gravity>
     </gazebo>
@@ -73,6 +73,6 @@
                        joint_parent_fr_basket_fr:='0 0 0 0 0 0'
                        joint_basket_fr_container_fr:='-0.068 0 0.013 0 0 0'
-                       basket_chassis_color:='red_color 1.0 0.0 0.0 1.0'
-                       basket_container_color:='alu_color 0.1 0.1 0.1 1.0'">
+                       basket_chassis_color:=''
+                       basket_container_color:=''">
     <xacro:basket_chassis_macro prefix="${prefix}"
                                 parent="${parent}"

Commit message: fix: use explicit basket origins
Replace the internal origin_element helper in basket macros with direct origin elements validated inside the public macro contract.

Derive Gazebo ambient and diffuse values from the caller-provided RGBA color instead of pinning a Gazebo material name.

File: urdf/extras/basket/basket_macros.xacro (robot description, xacro)
@@ -22,16 +22,32 @@
                        joint_parent_fr_basket_fr:='0 0 0 0 0 0'
                        color:=''">
+    <xacro:property name="joint_parent_fr_basket_fr_items"
+                    value="${joint_parent_fr_basket_fr.split()}"/>
+    <xacro:if value="${len(joint_parent_fr_basket_fr_items) != 6}">
+      ${xacro.fatal("basket_chassis_macro: joint_parent_fr_basket_fr must be 'x y z roll pitch yaw'")}
+    </xacro:if>
     <joint name="${prefix}basket_chassis_joint" type="fixed">
       <axis xyz="0 1 0"/>
-      <xacro:origin_element origin="${joint_parent_fr_basket_fr}"/>
+      <origin xyz="${joint_parent_fr_basket_fr_items[0]} ${joint_parent_fr_basket_fr_items[1]} ${joint_parent_fr_basket_fr_items[2]}"
+              rpy="${joint_parent_fr_basket_fr_items[3]} ${joint_parent_fr_basket_fr_items[4]} ${joint_parent_fr_basket_fr_items[5]}"/>
       <parent link="${parent}"/>
       <child link="${prefix}basket_chassis_link"/>
     </joint>
     <link name="${prefix}basket_chassis_link">
-      <xacro:null_inertia/>
       <xacro:visual_mesh mesh="${basket_chassis_mesh}" color="${color}"/>
       <xacro:collision_mesh mesh="${basket_chassis_mesh}"/>
+      <xacro:null_inertia/>
     </link>
     <gazebo reference="${prefix}basket_chassis_link">
+      <xacro:if value="${color != ''}">
+        <xacro:property name="color_items" value="${color.split()}"/>
+        <xacro:if value="${len(color_items) != 5}">
+          ${xacro.fatal("basket_chassis_macro: color must be 'color_name r g b a'")}
+        </xacro:if>
+        <material>
+          <ambient>${color_items[1]} ${color_items[2]} ${color_items[3]} ${color_items[4]}</ambient>
+          <diffuse>${color_items[1]} ${color_items[2]} ${color_items[3]} ${color_items[4]}</diffuse>
+        </material>
+      </xacro:if>
       <gravity>true</gravity>
     </gazebo>
@@ -49,7 +65,13 @@
                        joint_parent_fr_container_fr:='-0.068 0 0.013 0 0 0'
                        color:=''">
+    <xacro:property name="joint_parent_fr_container_fr_items"
+                    value="${joint_parent_fr_container_fr.split()}"/>
+    <xacro:if value="${len(joint_parent_fr_container_fr_items) != 6}">
+      ${xacro.fatal("basket_container_macro: joint_parent_fr_container_fr must be 'x y z roll pitch yaw'")}
+    </xacro:if>
     <joint name="${prefix}basket_container_joint" type="fixed">
       <axis xyz="0 1 0"/>
-      <xacro:origin_element origin="${joint_parent_fr_container_fr}"/>
+      <origin xyz="${joint_parent_fr_container_fr_items[0]} ${joint_parent_fr_container_fr_items[1]} ${joint_parent_fr_container_fr_items[2]}"
+              rpy="${joint_parent_fr_container_fr_items[3]} ${joint_parent_fr_container_fr_items[4]} ${joint_parent_fr_container_fr_items[5]}"/>
       <parent link="${parent}"/>
       <child link="${prefix}basket_container_link"/>
@@ -61,4 +83,14 @@
     </link>
     <gazebo reference="${prefix}basket_container_link">
+      <xacro:if value="${color != ''}">
+        <xacro:property name="color_items" value="${color.split()}"/>
+        <xacro:if value="${len(color_items) != 5}">
+          ${xacro.fatal("basket_container_macro: color must be 'color_name r g b a'")}
+        </xacro:if>
+        <material>
+          <ambient>${color_items[1]} ${color_items[2]} ${color_items[3]} ${color_items[4]}</ambient>
+          <diffuse>${color_items[1]} ${color_items[2]} ${color_items[3]} ${color_items[4]}</diffuse>
+        </material>
+      </xacro:if>
       <gravity>true</gravity>
     </gazebo>

Commit message: refactor: delegate basket origin validation
Use the shared origin_element helper in basket macros so origin parsing and validation stay owned by the common xacro utilities.

File: urdf/extras/basket/basket_macros.xacro (robot description, xacro)
@@ -22,13 +22,7 @@
                        joint_parent_fr_basket_fr:='0 0 0 0 0 0'
                        color:=''">
-    <xacro:property name="joint_parent_fr_basket_fr_items"
-                    value="${joint_parent_fr_basket_fr.split()}"/>
-    <xacro:if value="${len(joint_parent_fr_basket_fr_items) != 6}">
-      ${xacro.fatal("basket_chassis_macro: joint_parent_fr_basket_fr must be 'x y z roll pitch yaw'")}
-    </xacro:if>
     <joint name="${prefix}basket_chassis_joint" type="fixed">
       <axis xyz="0 1 0"/>
-      <origin xyz="${joint_parent_fr_basket_fr_items[0]} ${joint_parent_fr_basket_fr_items[1]} ${joint_parent_fr_basket_fr_items[2]}"
-              rpy="${joint_parent_fr_basket_fr_items[3]} ${joint_parent_fr_basket_fr_items[4]} ${joint_parent_fr_basket_fr_items[5]}"/>
+      <xacro:origin_element origin="${joint_parent_fr_basket_fr}"/>
       <parent link="${parent}"/>
       <child link="${prefix}basket_chassis_link"/>
@@ -65,13 +59,7 @@
                        joint_parent_fr_container_fr:='-0.068 0 0.013 0 0 0'
                        color:=''">
-    <xacro:property name="joint_parent_fr_container_fr_items"
-                    value="${joint_parent_fr_container_fr.split()}"/>
-    <xacro:if value="${len(joint_parent_fr_container_fr_items) != 6}">
-      ${xacro.fatal("basket_container_macro: joint_parent_fr_container_fr must be 'x y z roll pitch yaw'")}
-    </xacro:if>
     <joint name="${prefix}basket_container_joint" type="fixed">
       <axis xyz="0 1 0"/>
-      <origin xyz="${joint_parent_fr_container_fr_items[0]} ${joint_parent_fr_container_fr_items[1]} ${joint_parent_fr_container_fr_items[2]}"
-              rpy="${joint_parent_fr_container_fr_items[3]} ${joint_parent_fr_container_fr_items[4]} ${joint_parent_fr_container_fr_items[5]}"/>
+      <xacro:origin_element origin="${joint_parent_fr_container_fr}"/>
       <parent link="${parent}"/>
       <child link="${prefix}basket_container_link"/>

Commit message: fix: remove fixed basket joint axes
Drop axis elements from fixed basket joints because fixed joints have no degree of freedom and the unused axis is misleading.

File: urdf/extras/basket/basket_macros.xacro (robot description, xacro)
@@ -23,5 +23,4 @@
                        color:=''">
     <joint name="${prefix}basket_chassis_joint" type="fixed">
-      <axis xyz="0 1 0"/>
       <xacro:origin_element origin="${joint_parent_fr_basket_fr}"/>
       <parent link="${parent}"/>
@@ -60,5 +59,4 @@
                        color:=''">
     <joint name="${prefix}basket_container_joint" type="fixed">
-      <axis xyz="0 1 0"/>
       <xacro:origin_element origin="${joint_parent_fr_container_fr}"/>
       <parent link="${parent}"/>

Commit message: refactor: update basket mesh variants
Replace the legacy basket wrapper with explicit chassis and sensor-mounted variants backed by the new mesh assets.

File: urdf/extras/basket/basket_macros.xacro (robot description, xacro)
@@ -6,99 +6,75 @@
 <robot name="basket_macros" xmlns:xacro="http://www.ros.org/wiki/xacro">
   <xacro:include filename="$(find robotics_description)/urdf/common/all_commons.xacro"/>
-  <xacro:property name="basket_chassis_mesh"
-                  value="robotics_description/meshes/extras/basket/basket_chassis.stl"/>
-  <xacro:property name="basket_container_mesh"
+  <xacro:property name="basket_chassis_visual_mesh"
+                  value="robotics_description/meshes/extras/basket/basket_container.obj"/>
+  <xacro:property name="basket_chassis_collision_mesh"
                   value="robotics_description/meshes/extras/basket/basket_container.stl"/>
+  <xacro:property name="basket_chassis_closed_visual_mesh"
+                  value="robotics_description/meshes/extras/basket/basket_container.obj"/>
+  <xacro:property name="basket_chassis_closed_collision_mesh"
+                  value="robotics_description/meshes/extras/basket/basket_container.stl"/>
+  <xacro:property name="basket_sensors_visual_mesh"
+                  value="robotics_description/meshes/extras/basket/basket_sensors.obj"/>
+  <xacro:property name="basket_sensors_collision_mesh"
+                  value="robotics_description/meshes/extras/basket/basket_sensors.stl"/>
   <!--
-  Macro for the basket chassis only.
+  Macro for the basket chassis.
   joint_parent_fr_basket_fr (S): Basket chassis pose relative to parent.
       joint_parent_fr_basket_fr (S) = 'x y z roll pitch yaw'
-  color (S): Optional material in the form '<color_name> r g b a'.
-             If empty, the mesh may use its embedded color.
   -->
   <xacro:macro name="basket_chassis_macro"
                params="prefix
                        parent
-                       joint_parent_fr_basket_fr:='0 0 0 0 0 0'
-                       color:=''">
+                       joint_parent_fr_basket_fr:='0 0 0 0 0 0'">
     <joint name="${prefix}basket_chassis_joint" type="fixed">
       <xacro:origin_element origin="${joint_parent_fr_basket_fr}"/>
       <parent link="${parent}"/>
-      <child link="${prefix}basket_chassis_link"/>
+      <child link="${prefix}basket_root_link"/>
     </joint>
-    <link name="${prefix}basket_chassis_link">
-      <xacro:visual_mesh mesh="${basket_chassis_mesh}" color="${color}"/>
-      <xacro:collision_mesh mesh="${basket_chassis_mesh}"/>
+    <link name="${prefix}basket_root_link">
+      <xacro:visual_mesh mesh="${basket_chassis_visual_mesh}"/>
+      <xacro:collision_mesh mesh="${basket_chassis_collision_mesh}"/>
       <xacro:null_inertia/>
     </link>
-    <gazebo reference="${prefix}basket_chassis_link">
-      <xacro:if value="${color != ''}">
-        <xacro:property name="color_items" value="${color.split()}"/>
-        <xacro:if value="${len(color_items) != 5}">
-          ${xacro.fatal("basket_chassis_macro: color must be 'color_name r g b a'")}
-        </xacro:if>
-        <material>
-          <ambient>${color_items[1]} ${color_items[2]} ${color_items[3]} ${color_items[4]}</ambient>
-          <diffuse>${color_items[1]} ${color_items[2]} ${color_items[3]} ${color_items[4]}</diffuse>
-        </material>
-      </xacro:if>
-      <gravity>true</gravity>
-    </gazebo>
   </xacro:macro>
   <!--
-  Macro for the basket container only.
-  joint_parent_fr_container_fr (S): Basket container pose relative to parent.
-      joint_parent_fr_container_fr (S) = 'x y z roll pitch yaw'
-  color (S): Optional material in the form '<color_name> r g b a'.
-             If empty, the mesh may use its embedded color.
+  Macro for the closed basket chassis.
+  joint_parent_fr_basket_fr (S): Basket chassis pose relative to parent.
+      joint_parent_fr_basket_fr (S) = 'x y z roll pitch yaw'
   -->
-  <xacro:macro name="basket_container_macro"
+  <xacro:macro name="basket_chassis_closed_macro"
                params="prefix
                        parent
-                       joint_parent_fr_container_fr:='-0.068 0 0.013 0 0 0'
-                       color:=''">
-    <joint name="${prefix}basket_container_joint" type="fixed">
-      <xacro:origin_element origin="${joint_parent_fr_container_fr}"/>
+                       joint_parent_fr_basket_fr:='0 0 0 0 0 0'">
+    <joint name="${prefix}basket_chassis_closed_joint" type="fixed">
+      <xacro:origin_element origin="${joint_parent_fr_basket_fr}"/>
       <parent link="${parent}"/>
-      <child link="${prefix}basket_container_link"/>
+      <child link="${prefix}basket_root_link"/>
     </joint>
-    <link name="${prefix}basket_container_link">
+    <link name="${prefix}basket_root_link">
+      <xacro:visual_mesh mesh="${basket_chassis_closed_visual_mesh}"/>
+      <xacro:collision_mesh mesh="${basket_chassis_closed_collision_mesh}"/>
       <xacro:null_inertia/>
-      <xacro:visual_mesh mesh="${basket_container_mesh}" color="${color}"/>
-      <xacro:collision_mesh mesh="${basket_container_mesh}"/>
     </link>
-    <gazebo reference="${prefix}basket_container_link">
-      <xacro:if value="${color != ''}">
-        <xacro:property name="color_items" value="${color.split()}"/>
-        <xacro:if value="${len(color_items) != 5}">
-          ${xacro.fatal("basket_container_macro: color must be 'color_name r g b a'")}
-        </xacro:if>
-        <material>
-          <ambient>${color_items[1]} ${color_items[2]} ${color_items[3]} ${color_items[4]}</ambient>
-          <diffuse>${color_items[1]} ${color_items[2]} ${color_items[3]} ${color_items[4]}</diffuse>
-        </material>
-      </xacro:if>
-      <gravity>true</gravity>
-    </gazebo>
   </xacro:macro>
   <!--
-  Macro for the complete basket assembly.
-  The container offset stays explicit until the container STL frame is normalized.
+  Macro for the closed basket chassis with sensor mounts.
+  joint_parent_fr_basket_fr (S): Basket chassis pose relative to parent.
+      joint_parent_fr_basket_fr (S) = 'x y z roll pitch yaw'
   -->
-  <xacro:macro name="basket_full_macro"
+  <xacro:macro name="basket_sensors"
                params="prefix
                        parent
-                       joint_parent_fr_basket_fr:='0 0 0 0 0 0'
-                       joint_basket_fr_container_fr:='-0.068 0 0.013 0 0 0'
-                       basket_chassis_color:=''
-                       basket_container_color:=''">
-    <xacro:basket_chassis_macro prefix="${prefix}"
-                                parent="${parent}"
-                                joint_parent_fr_basket_fr="${joint_parent_fr_basket_fr}"
-                                color="${basket_chassis_color}"/>
-    <xacro:basket_container_macro prefix="${prefix}"
-                                  parent="${prefix}basket_chassis_link"
-                                  joint_parent_fr_container_fr="${joint_basket_fr_container_fr}"
-                                  color="${basket_container_color}"/>
+                       joint_parent_fr_basket_fr:='0 0 0 0 0 0'">
+    <joint name="${prefix}basket_chassis_closed_livox_supports_joint" type="fixed">
+      <xacro:origin_element origin="${joint_parent_fr_basket_fr}"/>
+      <parent link="${parent}"/>
+      <child link="${prefix}basket_root_link"/>
+    </joint>
+    <link name="${prefix}basket_root_link">
+      <xacro:visual_mesh mesh="${basket_sensors_visual_mesh}"/>
+      <xacro:collision_mesh mesh="${basket_sensors_collision_mesh}"/>
+      <xacro:null_inertia/>
+    </link>
   </xacro:macro>
 </robot>
